File: Wireless modbus/Wireless slave/wireless_Slave/LoRa_sch.kicad_sch (KiCad schematic)
At the start: 5 parts, among them IC1 LoRa-E5, J2 2337019-1

Commit message: ændringer
Parts:
- removed R1: R, symbol Device:R
- added C2: NC, symbol Device:C
- added C3: 4,7uF, symbol Device:C
- added J1: Conn_02x09_Odd_Even, symbol Connector_Generic:Conn_02x09_Odd_Even
- C1: value C -> NC
- L1: value L -> 0R
Connections:
- net at C1.1: now also IC1.15 (RFIO), L1.1
- net GND: now reaches C1.2
- net GND: now also IC1.14 (GND_2), IC1.16 (GND_3), IC1.2 (GND_1), IC1.22 (GND_4), J2.2 (GND), J2.3 (GND_2), C2.2, C3.2
- net VCC: now reaches IC1.1 (VCC)
- net VCC: now also C3.1
- net RXD: now reaches IC1.10 (PB6)
- net PB5: now reaches IC1.11 (PB5)
- net PB5: now also J1.13 (Pin_13)
- net PC1: now reaches IC1.12 (PC1)
- net PC1: now also J1.15 (Pin_15)
- net PC0: now reaches IC1.13 (PC0)
- net PC0: now also J1.17 (Pin_17)
- net Reset: now reaches IC1.17 (RST)
- net PA3: now reaches IC1.18 (PA3)
- net PA3: now also J1.18 (Pin_18)
- net PA2: now reaches IC1.19 (PA2)
- net PA2: now also J1.16 (Pin_16)
- net PB10: now reaches IC1.20 (PB10)
- net PB10: now also J1.14 (Pin_14)
- net PA9: now reaches IC1.21 (PA9)
- net PA9: now also J1.12 (Pin_12)
- net PA0: now reaches IC1.23 (PA0)
- net PA0: now also J1.10 (Pin_10)
- net Boot: now reaches IC1.24 (PB13)
- net PB9: now reaches IC1.25 (PB9)
- net PB9: now also J1.8 (Pin_8)
- net PB14: now reaches IC1.26 (PB14)
- net PB14: now also J1.6 (Pin_6)
- net PA10: now reaches IC1.27 (PA10)
- net PA10: now also J1.4 (Pin_4)
- net PB0: now reaches IC1.28 (PB0)
- net PB0: now also J1.2 (Pin_2)
- net PA13: now reaches IC1.3 (PA13)
- net PA13: now also J1.1 (Pin_1)
- net PA14: now reaches IC1.4 (PA14)
- net PA14: now also J1.3 (Pin_3)
- net PB15: now reaches IC1.5 (PB15)
- net PB15: now also J1.5 (Pin_5)
- net PA15: now reaches IC1.6 (PA15)
- net PA15: now also J1.7 (Pin_7)
- net PB4: now reaches IC1.7 (PB4)
- net PB4: now also J1.9 (Pin_9)
- net PB3: now reaches IC1.8 (PB3)
- net PB3: now also J1.11 (Pin_11)
- net TXD: now reaches IC1.9 (PB7)
- net at J2.1 (SIGNAL): now also L1.2, C2.1
Other:
- moved on the sheet: C1, J2, L1
