File: Wireless modbus/Wireless slave/wireless_Slave/LoRa_sch.kicad_sch (KiCad schematic)
At the start: 7 parts, among them IC1 LoRa-E5, J1 Conn_02x09_Odd_Even, J2 2337019-1

Commit message: wup wup
Parts:
- renumbered C3 to C15, C1 to C16, C2 to C17, J2 to J3, J1 to J4
Changed lines of the file:
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@@
   (symbol (lib_id "power:GND") (at 201.93 92.075 0) (unit 1)
     (in_bom yes) (on_board yes) (dnp no) (fields_autoplaced)
-    (property "Reference" "#PWR01" (at 201.93 98.425 0)
+    (property "Reference" "#PWR030" (at 201.93 98.425 0)
       (effects (font (size 1.27 1.27)) hide)
     )
@@
       (project "wireless_Slave"
         (path "/0e0a1f86-1a9d-413b-96af-bc4dca868b1d/652affe9-0d80-4167-b21e-3f1d9d20c33e"
-          (reference "#PWR01") (unit 1)
+          (reference "#PWR030") (unit 1)
         )
       )
@@
   (symbol (lib_id "power:GND") (at 180.34 88.9 0) (unit 1)
     (in_bom yes) (on_board yes) (dnp no) (fields_autoplaced)
-    (property "Reference" "#PWR03" (at 180.34 95.25 0)
+    (property "Reference" "#PWR029" (at 180.34 95.25 0)
       (effects (font (size 1.27 1.27)) hide)
     )
@@
       (project "wireless_Slave"
         (path "/0e0a1f86-1a9d-413b-96af-bc4dca868b1d/652affe9-0d80-4167-b21e-3f1d9d20c33e"
-          (reference "#PWR03") (unit 1)
+          (reference "#PWR029") (unit 1)
         )
       )
@@
   (symbol (lib_id "Device:C") (at 171.45 85.09 0) (unit 1)
     (in_bom yes) (on_board yes) (dnp no) (fields_autoplaced)
-    (property "Reference" "C1" (at 175.26 83.82 0)
+    (property "Reference" "C16" (at 175.26 83.82 0)
       (effects (font (size 1.27 1.27)) (justify left))
     )
@@
       (project "wireless_Slave"
         (path "/0e0a1f86-1a9d-413b-96af-bc4dca868b1d/652affe9-0d80-4167-b21e-3f1d9d20c33e"
-          (reference "C1") (unit 1)
+          (reference "C16") (unit 1)
         )
       )
@@
   (symbol (lib_id "power:GND") (at 160.02 99.06 0) (unit 1)
     (in_bom yes) (on_board yes) (dnp no) (fields_autoplaced)
-    (property "Reference" "#PWR07" (at 160.02 105.41 0)
+    (property "Reference" "#PWR027" (at 160.02 105.41 0)
       (effects (font (size 1.27 1.27)) hide)
     )
@@
       (project "wireless_Slave"
         (path "/0e0a1f86-1a9d-413b-96af-bc4dca868b1d/652affe9-0d80-4167-b21e-3f1d9d20c33e"
-          (reference "#PWR07") (unit 1)
+          (reference "#PWR027") (unit 1)
         )
       )
@@
   (symbol (lib_id "power:GND") (at 167.64 78.74 90) (unit 1)
     (in_bom yes) (on_board yes) (dnp no) (fields_autoplaced)
-    (property "Reference" "#PWR02" (at 173.99 78.74 0)
+    (property "Reference" "#PWR028" (at 173.99 78.74 0)
       (effects (font (size 1.27 1.27)) hide)
     )
@@
       (project "wireless_Slave"
         (path "/0e0a1f86-1a9d-413b-96af-bc4dca868b1d/652affe9-0d80-4167-b21e-3f1d9d20c33e"
-          (reference "#PWR02") (unit 1)
+          (reference "#PWR028") (unit 1)
         )
       )
@@
   (symbol (lib_id "power:GND") (at 160.02 48.26 180) (unit 1)
     (in_bom yes) (on_board yes) (dnp no) (fields_autoplaced)
-    (property "Reference" "#PWR06" (at 160.02 41.91 0)
+    (property "Reference" "#PWR026" (at 160.02 41.91 0)
       (effects (font (size 1.27 1.27)) hide)
     )
@@
       (project "wireless_Slave"
         (path "/0e0a1f86-1a9d-413b-96af-bc4dca868b1d/652affe9-0d80-4167-b21e-3f1d9d20c33e"
-          (reference "#PWR06") (unit 1)
+          (reference "#PWR026") (unit 1)
         )
       )
@@
   (symbol (lib_id "Connector_Generic:Conn_02x09_Odd_Even") (at 212.09 52.07 0) (unit 1)
     (in_bom yes) (on_board yes) (dnp no) (fields_autoplaced)
-    (property "Reference" "J1" (at 213.36 36.195 0)
+    (property "Reference" "J4" (at 213.36 36.195 0)
       (effects (font (size 1.27 1.27)))
     )
@@
       (project "wireless_Slave"
         (path "/0e0a1f86-1a9d-413b-96af-bc4dca868b1d/652affe9-0d80-4167-b21e-3f1d9d20c33e"
-          (reference "J1") (unit 1)
+          (reference "J4") (unit 1)
         )
       )
@@
         )
         (path "/0e0a1f86-1a9d-413b-96af-bc4dca868b1d/652affe9-0d80-4167-b21e-3f1d9d20c33e"
-          (reference "IC1") (unit 1)
+          (reference "IC2") (unit 1)
         )
       )
@@
   (symbol (lib_name "2337019-1_1") (lib_id "SamacSys_Parts:2337019-1") (at 173.99 85.09 0) (unit 1)
     (in_bom yes) (on_board yes) (dnp no) (fields_autoplaced)
-    (property "Reference" "J2" (at 208.28 80.0277 0)
+    (property "Reference" "J3" (at 208.28 80.0277 0)
       (effects (font (size 1.27 1.27)) (justify left))
     )
@@
       (project "wireless_Slave"
         (path "/0e0a1f86-1a9d-413b-96af-bc4dca868b1d/652affe9-0d80-4167-b21e-3f1d9d20c33e"
-          (reference "J2") (unit 1)
+          (reference "J3") (unit 1)
         )
       )
@@
   (symbol (lib_id "Device:C") (at 124.46 60.96 0) (unit 1)
     (in_bom yes) (on_board yes) (dnp no) (fields_autoplaced)
-    (property "Reference" "C3" (at 128.27 59.69 0)
+    (property "Reference" "C15" (at 128.27 59.69 0)
       (effects (font (size 1.27 1.27)) (justify left))
     )
@@
       (project "wireless_Slave"
         (path "/0e0a1f86-1a9d-413b-96af-bc4dca868b1d/652affe9-0d80-4167-b21e-3f1d9d20c33e"
-          (reference "C3") (unit 1)
+          (reference "C15") (unit 1)
         )
       )
@@
   (symbol (lib_id "power:GND") (at 137.16 68.58 270) (unit 1)
     (in_bom yes) (on_board yes) (dnp no) (fields_autoplaced)
-    (property "Reference" "#PWR05" (at 130.81 68.58 0)
+    (property "Reference" "#PWR025" (at 130.81 68.58 0)
       (effects (font (size 1.27 1.27)) hide)
     )
@@
       (project "wireless_Slave"
         (path "/0e0a1f86-1a9d-413b-96af-bc4dca868b1d/652affe9-0d80-4167-b21e-3f1d9d20c33e"
-          (reference "#PWR05") (unit 1)
+          (reference "#PWR025") (unit 1)
         )
       )
@@
   (symbol (lib_id "power:GND") (at 124.46 64.77 0) (unit 1)
     (in_bom yes) (on_board yes) (dnp no) (fields_autoplaced)
-    (property "Reference" "#PWR04" (at 124.46 71.12 0)
+    (property "Reference" "#PWR024" (at 124.46 71.12 0)
       (effects (font (size 1.27 1.27)) hide)
     )
@@
       (project "wireless_Slave"
         (path "/0e0a1f86-1a9d-413b-96af-bc4dca868b1d/652affe9-0d80-4167-b21e-3f1d9d20c33e"
-          (reference "#PWR04") (unit 1)
+          (reference "#PWR024") (unit 1)
         )
       )
@@
   (symbol (lib_id "Device:C") (at 186.69 85.09 0) (unit 1)
     (in_bom yes) (on_board yes) (dnp no) (fields_autoplaced)
-    (property "Reference" "C2" (at 190.5 83.82 0)
+    (property "Reference" "C17" (at 190.5 83.82 0)
       (effects (font (size 1.27 1.27)) (justify left))
     )
@@
       (project "wireless_Slave"
         (path "/0e0a1f86-1a9d-413b-96af-bc4dca868b1d/652affe9-0d80-4167-b21e-3f1d9d20c33e"
-          (reference "C2") (unit 1)
-        )
-      )
+          (reference "C17") (unit 1)
+        )
+      )

Commit message: wup
Parts:
- added TP1: Antenne, TestPoint:TestPoint_Pad_D2.5mm, symbol Connector:TestPoint
- C16: renamed from C15; value 4,7uF -> 4,7uf; footprint (none) -> Capacitor_SMD:C_0402_1005Metric
- C17: renamed from C16; footprint (none) -> Capacitor_SMD:C_0402_1005Metric
- J4: footprint (none) -> Connector_PinHeader_2.54mm:PinHeader_2x09_P2.54mm_Vertical
- L1: footprint Capacitor_SMD:C_0402_1005Metric -> Resistor_SMD:R_0402_1005Metric
- renumbered C17 to C18
Connections:
- net PA10: now also J4.16 (Pin_16); no longer J4.4 (Pin_4)
- net PA13: now also J4.17 (Pin_17); no longer J4.1 (Pin_1)
- net PA14: now also J4.15 (Pin_15); no longer J4.3 (Pin_3)
- net PA15: now also J4.11 (Pin_11); no longer J4.7 (Pin_7)
- net PA2: now also J4.4 (Pin_4); no longer J4.16 (Pin_16)
- net PA3: now also J4.6 (Pin_6); no longer J4.18 (Pin_18)
- net PA9: now also J4.8 (Pin_8); no longer J4.12 (Pin_12)
- net PB0: now also J4.18 (Pin_18); no longer J4.2 (Pin_2)
- net PB10: now also J4.2 (Pin_2); no longer J4.14 (Pin_14)
- net PB14: now also J4.14 (Pin_14); no longer J4.6 (Pin_6)
- net PB15: now also J4.13 (Pin_13); no longer J4.5 (Pin_5)
- net PB3: now also J4.1 (Pin_1); no longer J4.11 (Pin_11)
- net PB5: now also J4.3 (Pin_3); no longer J4.13 (Pin_13)
- net PB9: now also J4.12 (Pin_12); no longer J4.8 (Pin_8)
- net PC0: now also J4.7 (Pin_7); no longer J4.17 (Pin_17)
- net PC1: now also J4.5 (Pin_5); no longer J4.15 (Pin_15)
- net at C18.1, J3.1 (SIGNAL), L1.2: now also TP1.1

Commit message: wupwup
Parts:
- added AE1: Antenna, SELF_MADE:Event_alarm_antenna, symbol Device:Antenna
Connections:
- net at C18.1, J3.1 (SIGNAL), L1.2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: now also AE1.1 (A)
Changed lines of the file:
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@@
   (junction (at 180.34 88.9) (diameter 0) (color 0 0 0 0)
+  )
+  (junction (at 182.88 81.28) (diameter 0) (color 0 0 0 0)
   )
   (wire (pts (xy 167.64 68.58) (xy 172.72 68.58))
@@
         )
       )
+    )
+  )
+  (symbol (lib_id "Device:Antenna") (at 182.88 76.2 0) (unit 1)
+    (in_bom yes) (on_board yes) (dnp no)
+    (property "Reference" "AE1" (at 180.34 69.85 0)
+      (effects (font (size 1.27 1.27)) (justify left))
+    )
+    (property "Value" "Antenna" (at 180.34 72.39 0)
+      (effects (font (size 1.27 1.27)) (justify left))
+    )
+    (property "Footprint" "SELF_MADE:Event_alarm_antenna" (at 182.88 76.2 0)
+      (effects (font (size 1.27 1.27)) hide)
+    )
+    (property "Datasheet" "~" (at 182.88 76.2 0)
+      (effects (font (size 1.27 1.27)) hide)
+    )
+    (pin "1")
+    (instances
+      (project "wireless_Slave"
+        (path "/0e0a1f86-1a9d-413b-96af-bc4dca868b1d/58bbf317-6f19-4695-b4b3-bbbe360cf741"
+          (reference "AE1") (unit 1)
+        )
+        (path "/0e0a1f86-1a9d-413b-96af-bc4dca868b1d/652affe9-0d80-4167-b21e-3f1d9d20c33e"
+          (reference "AE1") (unit 1)
+        )
+      )

Commit message: jaaaaaaaaaaaaa
Parts:
- removed J4: Conn_02x09_Odd_Even, Connector_PinHeader_2.54mm:PinHeader_2x09_P2.54mm_Vertical, symbol Connector_Generic:Conn_02x09_Odd_Even
- added J2: Conn_01x18, Connector_PinHeader_2.54mm:PinHeader_1x18_P2.54mm_Vertical, symbol Connector_Generic:Conn_01x18
Connections:
- net PA0: now also J2.14 (Pin_14)
- net PA10: now also J2.11 (Pin_11)
- net PA13: now also J2.9 (Pin_9)
- net PA14: now also J2.8 (Pin_8)
- net PA15: now also J2.6 (Pin_6)
- net PA2: now also J2.17 (Pin_17)
- net PA3: now also J2.18 (Pin_18)
- net PA9: now also J2.15 (Pin_15)
- net PB0: now also J2.10 (Pin_10)
- net PB10: now also J2.16 (Pin_16)
- net PB14: now also J2.12 (Pin_12)
- net PB15: now also J2.7 (Pin_7)
- net PB3: now also J2.4 (Pin_4)
- net PB4: now also J2.5 (Pin_5)
- net PB5: now also J2.3 (Pin_3)
- net PB9: now also J2.13 (Pin_13)
- net PC0: now also J2.1 (Pin_1)
- net PC1: now also J2.2 (Pin_2)
Changed lines of the file:
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@@
     (stroke (width 0) (type default))
   )
-  (wire (pts (xy 207.01 46.99) (xy 201.93 46.99))
+  (wire (pts (xy 241.3 42.545) (xy 236.22 42.545))
     (stroke (width 0) (type default))
   )
@@
     (stroke (width 0) (type default))
   )
-  (wire (pts (xy 207.01 44.45) (xy 201.93 44.45))
+  (wire (pts (xy 241.3 47.625) (xy 236.22 47.625))
     (stroke (width 0) (type default))
   )
@@
     (stroke (width 0) (type default))
   )
-  (wire (pts (xy 219.71 41.91) (xy 224.79 41.91))
+  (wire (pts (xy 241.3 78.105) (xy 236.22 78.105))
     (stroke (width 0) (type default))
   )
@@
     (stroke (width 0) (type default))
   )
-  (wire (pts (xy 224.79 52.07) (xy 219.71 52.07))
+  (wire (pts (xy 236.22 73.025) (xy 241.3 73.025))
     (stroke (width 0) (type default))
   )
@@
     (stroke (width 0) (type default))
   )
-  (wire (pts (xy 201.93 57.15) (xy 207.01 57.15))
+  (wire (pts (xy 236.22 55.245) (xy 241.3 55.245))
     (stroke (width 0) (type default))
   )
@@
     (stroke (width 0) (type default))
   )
-  (wire (pts (xy 224.79 54.61) (xy 219.71 54.61))
-    (stroke (width 0) (type default))
-  )
-  (wire (pts (xy 201.93 54.61) (xy 207.01 54.61))
-    (stroke (width 0) (type default))
-  )
-  (wire (pts (xy 224.79 59.69) (xy 219.71 59.69))
-    (stroke (width 0) (type default))
-  )
-  (wire (pts (xy 219.71 46.99) (xy 224.79 46.99))
+  (wire (pts (xy 236.22 70.485) (xy 241.3 70.485))
+    (stroke (width 0) (type default))
+  )
+  (wire (pts (xy 236.22 52.705) (xy 241.3 52.705))
+    (stroke (width 0) (type default))
+  )
+  (wire (pts (xy 236.22 65.405) (xy 241.3 65.405))
+    (stroke (width 0) (type default))
+  )
+  (wire (pts (xy 241.3 83.185) (xy 236.22 83.185))
     (stroke (width 0) (type default))
   )
@@
     (stroke (width 0) (type default))
   )
-  (wire (pts (xy 201.93 52.07) (xy 207.01 52.07))
+  (wire (pts (xy 236.22 50.165) (xy 241.3 50.165))
     (stroke (width 0) (type default))
   )
@@
     (stroke (width 0) (type default))
   )
-  (wire (pts (xy 219.71 49.53) (xy 224.79 49.53))
-    (stroke (width 0) (type default))
-  )
-  (wire (pts (xy 224.79 57.15) (xy 219.71 57.15))
+  (wire (pts (xy 241.3 75.565) (xy 236.22 75.565))
+    (stroke (width 0) (type default))
+  )
+  (wire (pts (xy 236.22 67.945) (xy 241.3 67.945))
     (stroke (width 0) (type default))
   )
@@
     (stroke (width 0) (type default))
   )
-  (wire (pts (xy 201.93 62.23) (xy 207.01 62.23))
+  (wire (pts (xy 236.22 60.325) (xy 241.3 60.325))
     (stroke (width 0) (type default))
   )
@@
     (stroke (width 0) (type default))
   )
-  (wire (pts (xy 224.79 62.23) (xy 219.71 62.23))
-    (stroke (width 0) (type default))
-  )
-  (wire (pts (xy 207.01 41.91) (xy 201.93 41.91))
-    (stroke (width 0) (type default))
-  )
-  (wire (pts (xy 207.01 49.53) (xy 201.93 49.53))
-    (stroke (width 0) (type default))
-  )
-  (wire (pts (xy 219.71 44.45) (xy 224.79 44.45))
-    (stroke (width 0) (type default))
-  )
-  (wire (pts (xy 201.93 59.69) (xy 207.01 59.69))
-    (stroke (width 0) (type default))
-  )
-  (label "PC0" (at 201.93 49.53 0) (fields_autoplaced)
-    (effects (font (size 1.27 1.27)) (justify left bottom))
-  )
-  (label "PB3" (at 201.93 41.91 0) (fields_autoplaced)
+  (wire (pts (xy 236.22 62.865) (xy 241.3 62.865))
+    (stroke (width 0) (type default))
+  )
+  (wire (pts (xy 241.3 45.085) (xy 236.22 45.085))
+    (stroke (width 0) (type default))
+  )
+  (wire (pts (xy 241.3 40.005) (xy 236.22 40.005))
+    (stroke (width 0) (type default))
+  )
+  (wire (pts (xy 241.3 80.645) (xy 236.22 80.645))
+    (stroke (width 0) (type default))
+  )
+  (wire (pts (xy 236.22 57.785) (xy 241.3 57.785))
+    (stroke (width 0) (type default))
+  )
+  (label "PC0" (at 236.22 40.005 0) (fields_autoplaced)
+    (effects (font (size 1.27 1.27)) (justify left bottom))
+  )
+  (label "PB3" (at 236.22 47.625 0) (fields_autoplaced)
     (effects (font (size 1.27 1.27)) (justify left bottom))
   )
@@
     (effects (font (size 1.27 1.27)) (justify left bottom))
   )
-  (label "PA15" (at 201.93 54.61 0) (fields_autoplaced)
-    (effects (font (size 1.27 1.27)) (justify left bottom))
-  )
-  (label "PA10" (at 224.79 59.69 180) (fields_autoplaced)
-    (effects (font (size 1.27 1.27)) (justify right bottom))
-  )
-  (label "PA2" (at 224.79 44.45 180) (fields_autoplaced)
-    (effects (font (size 1.27 1.27)) (justify right bottom))
-  )
-  (label "PA14" (at 201.93 59.69 0) (fields_autoplaced)
+  (label "PA15" (at 236.22 52.705 0) (fields_autoplaced)
+    (effects (font (size 1.27 1.27)) (justify left bottom))
+  )
+  (label "PA10" (at 236.22 65.405 0) (fields_autoplaced)
+    (effects (font (size 1.27 1.27)) (justify left bottom))
+  )
+  (label "PA2" (at 236.22 80.645 0) (fields_autoplaced)
+    (effects (font (size 1.27 1.27)) (justify left bottom))
+  )
+  (label "PA14" (at 236.22 57.785 0) (fields_autoplaced)
     (effects (font (size 1.27 1.27)) (justify left bottom))
   )
@@
     (effects (font (size 1.27 1.27)) (justify left bottom))
   )
-  (label "PB10" (at 224.79 41.91 180) (fields_autoplaced)
-    (effects (font (size 1.27 1.27)) (justify right bottom))
-  )
-  (label "PA9" (at 224.79 49.53 180) (fields_autoplaced)
-    (effects (font (size 1.27 1.27)) (justify right bottom))
-  )
-  (label "PB9" (at 224.79 54.61 180) (fields_autoplaced)
-    (effects (font (size 1.27 1.27)) (justify right bottom))
+  (label "PB10" (at 236.22 78.105 0) (fields_autoplaced)
+    (effects (font (size 1.27 1.27)) (justify left bottom))
+  )
+  (label "PA9" (at 236.22 75.565 0) (fields_autoplaced)
+    (effects (font (size 1.27 1.27)) (justify left bottom))
+  )
+  (label "PB9" (at 236.22 70.485 0) (fields_autoplaced)
+    (effects (font (size 1.27 1.27)) (justify left bottom))
   )
   (label "PA9" (at 172.72 66.04 180) (fields_autoplaced)
     (effects (font (size 1.27 1.27)) (justify right bottom))
   )
-  (label "PA0" (at 224.79 52.07 180) (fields_autoplaced)
-    (effects (font (size 1.27 1.27)) (justify right bottom))
+  (label "PA0" (at 236.22 73.025 0) (fields_autoplaced)
+    (effects (font (size 1.27 1.27)) (justify left bottom))
   )
   (label "PA15" (at 132.08 78.74 0) (fields_autoplaced)
     (effects (font (size 1.27 1.27)) (justify left bottom))
   )
-  (label "PB15" (at 201.93 57.15 0) (fields_autoplaced)
+  (label "PB15" (at 236.22 55.245 0) (fields_autoplaced)
     (effects (font (size 1.27 1.27)) (justify left bottom))
   )
@@
     (effects (font (size 1.27 1.27)) (justify right bottom))
   )
-  (label "PB0" (at 224.79 62.23 180) (fields_autoplaced)
-    (effects (font (size 1.27 1.27)) (justify right bottom))
-  )
-  (label "PB14" (at 224.79 57.15 180) (fields_autoplaced)
-    (effects (font (size 1.27 1.27)) (justify right bottom))
+  (label "PB0" (at 236.22 62.865 0) (fields_autoplaced)
+    (effects (font (size 1.27 1.27)) (justify left bottom))
+  )
+  (label "PB14" (at 236.22 67.945 0) (fields_autoplaced)
+    (effects (font (size 1.27 1.27)) (justify left bottom))
   )
   (label "PB3" (at 144.78 104.14 90) (fields_autoplaced)
     (effects (font (size 1.27 1.27)) (justify left bottom))
   )
-  (label "PB4" (at 201.93 52.07 0) (fields_autoplaced)
-    (effects (font (size 1.27 1.27)) (justify left bottom))
-  )
-  (label "PA3" (at 224.79 46.99 180) (fields_autoplaced)
-    (effects (font (size 1.27 1.27)) (justify right bottom))
-  )
-  (label "PA13" (at 201.93 62.23 0) (fields_autoplaced)
-    (effects (font (size 1.27 1.27)) (justify left bottom))
-  )
-  (label "PB5" (at 201.93 44.45 0) (fields_autoplaced)
+  (label "PB4" (at 236.22 50.165 0) (fields_autoplaced)
+    (effects (font (size 1.27 1.27)) (justify left bottom))
+  )
+  (label "PA3" (at 236.22 83.185 0) (fields_autoplaced)
+    (effects (font (size 1.27 1.27)) (justify left bottom))
+  )
+  (label "PA13" (at 236.22 60.325 0) (fields_autoplaced)
+    (effects (font (size 1.27 1.27)) (justify left bottom))
+  )
+  (label "PB5" (at 236.22 45.085 0) (fields_autoplaced)
     (effects (font (size 1.27 1.27)) (justify left bottom))
   )
@@
     (effects (font (size 1.27 1.27)) (justify right bottom))
   )
-  (label "PC1" (at 201.93 46.99 0) (fields_autoplaced)
+  (label "PC1" (at 236.22 42.545 0) (fields_autoplaced)
     (effects (font (size 1.27 1.27)) (justify left bottom))
   )
@@
     )
   )
-  (symbol (lib_id "Connector_Generic:Conn_02x09_Odd_Even") (at 212.09 52.07 0) (unit 1)
-    (in_bom yes) (on_board yes) (dnp no) (fields_autoplaced)
-    (property "Reference" "J4" (at 213.36 36.195 0)
-      (effects (font (size 1.27 1.27)))
-    )
-    (property "Value" "Conn_02x09_Odd_Even" (at 213.36 38.735 0)
-      (effects (font (size 1.27 1.27)))
-    )
-    (property "Footprint" "Connector_PinHeader_2.54mm:PinHeader_2x09_P2.54mm_Vertical" (at 212.09 52.07 0)
-      (effects (font (size 1.27 1.27)) hide)
-    )
-    (property "Datasheet" "~" (at 212.09 52.07 0)
+  (symbol (lib_id "Connector_Generic:Conn_01x18") (at 246.38 60.325 0) (unit 1)
+    (in_bom yes) (on_board yes) (dnp no) (fields_autoplaced)
+    (property "Reference" "J2" (at 248.92 60.325 0)
+      (effects (font (size 1.27 1.27)) (justify left))
+    )
+    (property "Value" "Conn_01x18" (at 248.92 62.865 0)
+      (effects (font (size 1.27 1.27)) (justify left))
+    )
+    (property "Footprint" "Connector_PinHeader_2.54mm:PinHeader_1x18_P2.54mm_Vertical" (at 246.38 60.325 0)
+      (effects (font (size 1.27 1.27)) hide)
+    )
+    (property "Datasheet" "~" (at 246.38 60.325 0)
       (effects (font (size 1.27 1.27)) hide)
     )
@@
       (project "wireless_Slave"
         (path "/0e0a1f86-1a9d-413b-96af-bc4dca868b1d/652affe9-0d80-4167-b21e-3f1d9d20c33e"
-          (reference "J4") (unit 1)
-        )
-      )
+          (reference "J2") (unit 1)
+        )
+      )
