File: Wireless modbus/Wireless slave/wireless_Slave/LoRa_sch.kicad_sch (KiCad schematic)
At the start: 9 parts, among them IC1 LoRa-E5, J2 Conn_01x18, J3 2337019-1

Commit message: test
Parts:
- removed J2: Conn_01x18, Connector_PinHeader_2.54mm:PinHeader_1x18_P2.54mm_Vertical, symbol Connector_Generic:Conn_01x18
Changed lines of the file:
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@@
-    (stroke (width 0) (type default))
-  )
-  (wire (pts (xy 241.3 42.545) (xy 236.22 42.545))
     (stroke (width 0) (type default))
   )
@@
     (stroke (width 0) (type default))
   )
-  (wire (pts (xy 241.3 47.625) (xy 236.22 47.625))
-    (stroke (width 0) (type default))
-  )
   (wire (pts (xy 157.48 99.06) (xy 157.48 104.14))
     (stroke (width 0) (type default))
@@
     (stroke (width 0) (type default))
   )
-  (wire (pts (xy 241.3 78.105) (xy 236.22 78.105))
-    (stroke (width 0) (type default))
-  )
   (wire (pts (xy 167.64 81.28) (xy 171.45 81.28))
     (stroke (width 0) (type default))
   )
-  (wire (pts (xy 236.22 73.025) (xy 241.3 73.025))
-    (stroke (width 0) (type default))
-  )
   (wire (pts (xy 167.64 66.04) (xy 172.72 66.04))
     (stroke (width 0) (type default))
   )
-  (wire (pts (xy 236.22 55.245) (xy 241.3 55.245))
-    (stroke (width 0) (type default))
-  )
   (wire (pts (xy 132.08 78.74) (xy 137.16 78.74))
     (stroke (width 0) (type default))
@@
     (stroke (width 0) (type default))
   )
-  (wire (pts (xy 236.22 70.485) (xy 241.3 70.485))
-    (stroke (width 0) (type default))
-  )
-  (wire (pts (xy 236.22 52.705) (xy 241.3 52.705))
-    (stroke (width 0) (type default))
-  )
-  (wire (pts (xy 236.22 65.405) (xy 241.3 65.405))
-    (stroke (width 0) (type default))
-  )
-  (wire (pts (xy 241.3 83.185) (xy 236.22 83.185))
-    (stroke (width 0) (type default))
-  )
   (wire (pts (xy 132.08 73.66) (xy 137.16 73.66))
     (stroke (width 0) (type default))
@@
     (stroke (width 0) (type default))
   )
-  (wire (pts (xy 236.22 50.165) (xy 241.3 50.165))
-    (stroke (width 0) (type default))
-  )
   (wire (pts (xy 152.4 43.18) (xy 152.4 48.26))
     (stroke (width 0) (type default))
@@
     (stroke (width 0) (type default))
   )
-  (wire (pts (xy 241.3 75.565) (xy 236.22 75.565))
-    (stroke (width 0) (type default))
-  )
-  (wire (pts (xy 236.22 67.945) (xy 241.3 67.945))
-    (stroke (width 0) (type default))
-  )
   (wire (pts (xy 132.08 76.2) (xy 137.16 76.2))
     (stroke (width 0) (type default))
@@
     (stroke (width 0) (type default))
   )
-  (wire (pts (xy 236.22 60.325) (xy 241.3 60.325))
-    (stroke (width 0) (type default))
-  )
   (wire (pts (xy 182.88 81.28) (xy 186.69 81.28))
     (stroke (width 0) (type default))
@@
     (stroke (width 0) (type default))
   )
-  (wire (pts (xy 236.22 62.865) (xy 241.3 62.865))
-    (stroke (width 0) (type default))
-  )
-  (wire (pts (xy 241.3 45.085) (xy 236.22 45.085))
-    (stroke (width 0) (type default))
-  )
-  (wire (pts (xy 241.3 40.005) (xy 236.22 40.005))
-    (stroke (width 0) (type default))
-  )
-  (wire (pts (xy 241.3 80.645) (xy 236.22 80.645))
-    (stroke (width 0) (type default))
-  )
-  (wire (pts (xy 236.22 57.785) (xy 241.3 57.785))
-    (stroke (width 0) (type default))
-  )
-  (label "PC0" (at 236.22 40.005 0) (fields_autoplaced)
-    (effects (font (size 1.27 1.27)) (justify left bottom))
-  )
-  (label "PB3" (at 236.22 47.625 0) (fields_autoplaced)
-    (effects (font (size 1.27 1.27)) (justify left bottom))
-  )
   (label "PC1" (at 154.94 104.14 90) (fields_autoplaced)
     (effects (font (size 1.27 1.27)) (justify left bottom))
@@
     (effects (font (size 1.27 1.27)) (justify left bottom))
   )
-  (label "PA15" (at 236.22 52.705 0) (fields_autoplaced)
-    (effects (font (size 1.27 1.27)) (justify left bottom))
-  )
-  (label "PA10" (at 236.22 65.405 0) (fields_autoplaced)
-    (effects (font (size 1.27 1.27)) (justify left bottom))
-  )
-  (label "PA2" (at 236.22 80.645 0) (fields_autoplaced)
-    (effects (font (size 1.27 1.27)) (justify left bottom))
-  )
-  (label "PA14" (at 236.22 57.785 0) (fields_autoplaced)
-    (effects (font (size 1.27 1.27)) (justify left bottom))
-  )
   (label "PA14" (at 132.08 73.66 0) (fields_autoplaced)
     (effects (font (size 1.27 1.27)) (justify left bottom))
@@
     (effects (font (size 1.27 1.27)) (justify left bottom))
   )
-  (label "PB10" (at 236.22 78.105 0) (fields_autoplaced)
-    (effects (font (size 1.27 1.27)) (justify left bottom))
-  )
-  (label "PA9" (at 236.22 75.565 0) (fields_autoplaced)
-    (effects (font (size 1.27 1.27)) (justify left bottom))
-  )
-  (label "PB9" (at 236.22 70.485 0) (fields_autoplaced)
-    (effects (font (size 1.27 1.27)) (justify left bottom))
-  )
   (label "PA9" (at 172.72 66.04 180) (fields_autoplaced)
     (effects (font (size 1.27 1.27)) (justify right bottom))
   )
-  (label "PA0" (at 236.22 73.025 0) (fields_autoplaced)
-    (effects (font (size 1.27 1.27)) (justify left bottom))
-  )
   (label "PA15" (at 132.08 78.74 0) (fields_autoplaced)
     (effects (font (size 1.27 1.27)) (justify left bottom))
   )
-  (label "PB15" (at 236.22 55.245 0) (fields_autoplaced)
-    (effects (font (size 1.27 1.27)) (justify left bottom))
-  )
   (label "PA13" (at 132.08 71.12 0) (fields_autoplaced)
     (effects (font (size 1.27 1.27)) (justify left bottom))
@@
     (effects (font (size 1.27 1.27)) (justify right bottom))
   )
-  (label "PB0" (at 236.22 62.865 0) (fields_autoplaced)
-    (effects (font (size 1.27 1.27)) (justify left bottom))
-  )
-  (label "PB14" (at 236.22 67.945 0) (fields_autoplaced)
-    (effects (font (size 1.27 1.27)) (justify left bottom))
-  )
   (label "PB3" (at 144.78 104.14 90) (fields_autoplaced)
     (effects (font (size 1.27 1.27)) (justify left bottom))
   )
-  (label "PB4" (at 236.22 50.165 0) (fields_autoplaced)
-    (effects (font (size 1.27 1.27)) (justify left bottom))
-  )
-  (label "PA3" (at 236.22 83.185 0) (fields_autoplaced)
-    (effects (font (size 1.27 1.27)) (justify left bottom))
-  )
-  (label "PA13" (at 236.22 60.325 0) (fields_autoplaced)
-    (effects (font (size 1.27 1.27)) (justify left bottom))
-  )
-  (label "PB5" (at 236.22 45.085 0) (fields_autoplaced)
-    (effects (font (size 1.27 1.27)) (justify left bottom))
-  )
   (label "PB10" (at 172.72 68.58 180) (fields_autoplaced)
     (effects (font (size 1.27 1.27)) (justify right bottom))
-  )
-  (label "PC1" (at 236.22 42.545 0) (fields_autoplaced)
-    (effects (font (size 1.27 1.27)) (justify left bottom))
   )
   (label "PB0" (at 144.78 43.18 270) (fields_autoplaced)
@@
         )
       )
-    )
-  )
-  (symbol (lib_id "Connector_Generic:Conn_01x18") (at 246.38 60.325 0) (unit 1)
-    (in_bom yes) (on_board yes) (dnp no) (fields_autoplaced)
-    (property "Reference" "J2" (at 248.92 60.325 0)
-      (effects (font (size 1.27 1.27)) (justify left))
-    )
-    (property "Value" "Conn_01x18" (at 248.92 62.865 0)
-      (effects (font (size 1.27 1.27)) (justify left))
-    )
-    (property "Footprint" "Connector_PinHeader_2.54mm:PinHeader_1x18_P2.54mm_Vertical" (at 246.38 60.325 0)
-      (effects (font (size 1.27 1.27)) hide)
-    )
-    (property "Datasheet" "~" (at 246.38 60.325 0)
-      (effects (font (size 1.27 1.27)) hide)
-    )
-    (pin "1")
-    (pin "10")
-    (pin "11")
-    (pin "12")
-    (pin "13")
-    (pin "14")
-    (pin "15")
-    (pin "16")
-    (pin "17")
-    (pin "18")
-    (pin "2")
-    (pin "3")
-    (pin "4")
-    (pin "5")
-    (pin "6")
-    (pin "7")
-    (pin "8")
-    (pin "9")
-    (instances
-      (project "wireless_Slave"
-        (path "/0e0a1f86-1a9d-413b-96af-bc4dca868b1d/652affe9-0d80-4167-b21e-3f1d9d20c33e"
-          (reference "J2") (unit 1)
-        )
-      )

Commit message: TJEK
Parts:
- renumbered TP1 to Antenna1, C16 to C19, C17 to C20, C18 to C21, J3 to J6
Changed lines of the file:
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@@
   (symbol (lib_id "power:GND") (at 201.93 92.075 0) (unit 1)
     (in_bom yes) (on_board yes) (dnp no) (fields_autoplaced)
-    (property "Reference" "#PWR030" (at 201.93 98.425 0)
+    (property "Reference" "#PWR056" (at 201.93 98.425 0)
       (effects (font (size 1.27 1.27)) hide)
     )
@@
       (project "wireless_Slave"
         (path "/0e0a1f86-1a9d-413b-96af-bc4dca868b1d/652affe9-0d80-4167-b21e-3f1d9d20c33e"
-          (reference "#PWR030") (unit 1)
+          (reference "#PWR056") (unit 1)
         )
       )
@@
   (symbol (lib_id "power:GND") (at 180.34 88.9 0) (unit 1)
     (in_bom yes) (on_board yes) (dnp no) (fields_autoplaced)
-    (property "Reference" "#PWR029" (at 180.34 95.25 0)
+    (property "Reference" "#PWR055" (at 180.34 95.25 0)
       (effects (font (size 1.27 1.27)) hide)
     )
@@
       (project "wireless_Slave"
         (path "/0e0a1f86-1a9d-413b-96af-bc4dca868b1d/652affe9-0d80-4167-b21e-3f1d9d20c33e"
-          (reference "#PWR029") (unit 1)
+          (reference "#PWR055") (unit 1)
         )
       )
@@
   (symbol (lib_id "Device:C") (at 171.45 85.09 0) (unit 1)
     (in_bom yes) (on_board yes) (dnp no) (fields_autoplaced)
-    (property "Reference" "C17" (at 175.26 83.82 0)
+    (property "Reference" "C20" (at 175.26 83.82 0)
       (effects (font (size 1.27 1.27)) (justify left))
     )
@@
       (project "wireless_Slave"
         (path "/0e0a1f86-1a9d-413b-96af-bc4dca868b1d/652affe9-0d80-4167-b21e-3f1d9d20c33e"
-          (reference "C17") (unit 1)
+          (reference "C20") (unit 1)
         )
       )
@@
   (symbol (lib_id "Connector:TestPoint") (at 186.69 81.28 0) (unit 1)
     (in_bom yes) (on_board yes) (dnp no)
-    (property "Reference" "TP1" (at 189.23 76.708 0)
+    (property "Reference" "Antenna1" (at 189.23 76.708 0)
       (effects (font (size 1.27 1.27)) (justify left))
     )
@@
       (project "wireless_Slave"
         (path "/0e0a1f86-1a9d-413b-96af-bc4dca868b1d/652affe9-0d80-4167-b21e-3f1d9d20c33e"
-          (reference "TP1") (unit 1)
+          (reference "Antenna1") (unit 1)
         )
       )
@@
   (symbol (lib_id "power:GND") (at 160.02 99.06 0) (unit 1)
     (in_bom yes) (on_board yes) (dnp no) (fields_autoplaced)
-    (property "Reference" "#PWR027" (at 160.02 105.41 0)
+    (property "Reference" "#PWR057" (at 160.02 105.41 0)
       (effects (font (size 1.27 1.27)) hide)
     )
@@
       (project "wireless_Slave"
         (path "/0e0a1f86-1a9d-413b-96af-bc4dca868b1d/652affe9-0d80-4167-b21e-3f1d9d20c33e"
-          (reference "#PWR027") (unit 1)
+          (reference "#PWR057") (unit 1)
         )
       )
@@
   (symbol (lib_id "power:GND") (at 167.64 78.74 90) (unit 1)
     (in_bom yes) (on_board yes) (dnp no) (fields_autoplaced)
-    (property "Reference" "#PWR028" (at 173.99 78.74 0)
+    (property "Reference" "#PWR054" (at 173.99 78.74 0)
       (effects (font (size 1.27 1.27)) hide)
     )
@@
       (project "wireless_Slave"
         (path "/0e0a1f86-1a9d-413b-96af-bc4dca868b1d/652affe9-0d80-4167-b21e-3f1d9d20c33e"
-          (reference "#PWR028") (unit 1)
+          (reference "#PWR054") (unit 1)
         )
       )
@@
   (symbol (lib_id "power:GND") (at 160.02 48.26 180) (unit 1)
     (in_bom yes) (on_board yes) (dnp no) (fields_autoplaced)
-    (property "Reference" "#PWR026" (at 160.02 41.91 0)
+    (property "Reference" "#PWR051" (at 160.02 41.91 0)
       (effects (font (size 1.27 1.27)) hide)
     )
@@
       (project "wireless_Slave"
         (path "/0e0a1f86-1a9d-413b-96af-bc4dca868b1d/652affe9-0d80-4167-b21e-3f1d9d20c33e"
-          (reference "#PWR026") (unit 1)
+          (reference "#PWR051") (unit 1)
         )
       )
@@
         )
         (path "/0e0a1f86-1a9d-413b-96af-bc4dca868b1d/652affe9-0d80-4167-b21e-3f1d9d20c33e"
-          (reference "IC2") (unit 1)
+          (reference "IC5") (unit 1)
         )
       )
@@
   (symbol (lib_name "2337019-1_1") (lib_id "SamacSys_Parts:2337019-1") (at 173.99 85.09 0) (unit 1)
     (in_bom yes) (on_board yes) (dnp no) (fields_autoplaced)
-    (property "Reference" "J3" (at 208.28 80.0277 0)
+    (property "Reference" "J6" (at 208.28 80.0277 0)
       (effects (font (size 1.27 1.27)) (justify left))
     )
@@
       (project "wireless_Slave"
         (path "/0e0a1f86-1a9d-413b-96af-bc4dca868b1d/652affe9-0d80-4167-b21e-3f1d9d20c33e"
-          (reference "J3") (unit 1)
+          (reference "J6") (unit 1)
         )
       )
@@
   (symbol (lib_id "Device:C") (at 124.46 60.96 0) (unit 1)
     (in_bom yes) (on_board yes) (dnp no) (fields_autoplaced)
-    (property "Reference" "C16" (at 128.27 59.69 0)
+    (property "Reference" "C19" (at 128.27 59.69 0)
       (effects (font (size 1.27 1.27)) (justify left))
     )
@@
       (project "wireless_Slave"
         (path "/0e0a1f86-1a9d-413b-96af-bc4dca868b1d/652affe9-0d80-4167-b21e-3f1d9d20c33e"
-          (reference "C16") (unit 1)
+          (reference "C19") (unit 1)
         )
       )
@@
   (symbol (lib_id "power:GND") (at 137.16 68.58 270) (unit 1)
     (in_bom yes) (on_board yes) (dnp no) (fields_autoplaced)
-    (property "Reference" "#PWR025" (at 130.81 68.58 0)
+    (property "Reference" "#PWR053" (at 130.81 68.58 0)
       (effects (font (size 1.27 1.27)) hide)
     )
@@
       (project "wireless_Slave"
         (path "/0e0a1f86-1a9d-413b-96af-bc4dca868b1d/652affe9-0d80-4167-b21e-3f1d9d20c33e"
-          (reference "#PWR025") (unit 1)
+          (reference "#PWR053") (unit 1)
         )
       )
@@
   (symbol (lib_id "power:GND") (at 124.46 64.77 0) (unit 1)
     (in_bom yes) (on_board yes) (dnp no) (fields_autoplaced)
-    (property "Reference" "#PWR024" (at 124.46 71.12 0)
+    (property "Reference" "#PWR052" (at 124.46 71.12 0)
       (effects (font (size 1.27 1.27)) hide)
     )
@@
       (project "wireless_Slave"
         (path "/0e0a1f86-1a9d-413b-96af-bc4dca868b1d/652affe9-0d80-4167-b21e-3f1d9d20c33e"
-          (reference "#PWR024") (unit 1)
+          (reference "#PWR052") (unit 1)
         )
       )
@@
   (symbol (lib_id "Device:C") (at 186.69 85.09 0) (unit 1)
     (in_bom yes) (on_board yes) (dnp no) (fields_autoplaced)
-    (property "Reference" "C18" (at 190.5 83.82 0)
+    (property "Reference" "C21" (at 190.5 83.82 0)
       (effects (font (size 1.27 1.27)) (justify left))
     )
@@
       (project "wireless_Slave"
         (path "/0e0a1f86-1a9d-413b-96af-bc4dca868b1d/652affe9-0d80-4167-b21e-3f1d9d20c33e"
-          (reference "C18") (unit 1)
-        )
-      )
+          (reference "C21") (unit 1)
+        )
+      )
