File: Wireless modbus/Wireless slave/wireless_Slave/wireless_Slave.kicad_sch (KiCad schematic)
At the start: 1 part, among them IC1 LoRa-E5

Commit message: ændringer
Parts:
- added U1: RP2040, Package_DFN_QFN:QFN-56-1EP_7x7mm_P0.4mm_EP3.2x3.2mm, symbol MCU_RaspberryPi:RP2040
Connections:
- new net: U1.1 (IOVDD), U1.10 (IOVDD), U1.22 (IOVDD), U1.33 (IOVDD), U1.42 (IOVDD), U1.49 (IOVDD)
- new net: U1.23 (DVDD), U1.50 (DVDD)
Changed lines of the file:
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@@
 (kicad_sch (version 20230121) (generator eeschema)
   (paper "A4")
+  (symbol (lib_id "MCU_RaspberryPi:RP2040") (at 74.93 92.71 0) (unit 1)
+    (in_bom yes) (on_board yes) (dnp no) (fields_autoplaced)
+    (property "Reference" "U1" (at 77.1241 137.16 0)
+      (effects (font (size 1.27 1.27)) (justify left))
+    )
+    (property "Value" "RP2040" (at 77.1241 139.7 0)
+      (effects (font (size 1.27 1.27)) (justify left))
+    )
+    (property "Footprint" "Package_DFN_QFN:QFN-56-1EP_7x7mm_P0.4mm_EP3.2x3.2mm" (at 74.93 92.71 0)
+      (effects (font (size 1.27 1.27)) hide)
+    )
+    (property "Datasheet" "https://datasheets.raspberrypi.com/rp2040/rp2040-datasheet.pdf" (at 74.93 92.71 0)
+      (effects (font (size 1.27 1.27)) hide)
+    )
+    (pin "1")
+    (pin "10")
+    (pin "11")
+    (pin "12")
+    (pin "13")
+    (pin "14")
+    (pin "15")
+    (pin "16")
+    (pin "17")
+    (pin "18")
+    (pin "19")
+    (pin "2")
+    (pin "20")
+    (pin "21")
+    (pin "22")
+    (pin "23")
+    (pin "24")
+    (pin "25")
+    (pin "26")
+    (pin "27")
+    (pin "28")
+    (pin "29")
+    (pin "3")
+    (pin "30")
+    (pin "31")
+    (pin "32")
+    (pin "33")
+    (pin "34")
+    (pin "35")
+    (pin "36")
+    (pin "37")
+    (pin "38")
+    (pin "39")
+    (pin "4")
+    (pin "40")
+    (pin "41")
+    (pin "42")
+    (pin "43")
+    (pin "44")
+    (pin "45")
+    (pin "46")
+    (pin "47")
+    (pin "48")
+    (pin "49")
+    (pin "5")
+    (pin "50")
+    (pin "51")
+    (pin "52")
+    (pin "53")
+    (pin "54")
+    (pin "55")
+    (pin "56")
+    (pin "57")
+    (pin "6")
+    (pin "7")
+    (pin "8")
+    (pin "9")
+    (instances
+      (project "wireless_Slave"
+        (path "/0e0a1f86-1a9d-413b-96af-bc4dca868b1d"
+          (reference "U1") (unit 1)
+        )
+      )
+    )
+  )
   (symbol (lib_id "SamacSys_Parts:LoRa-E5") (at 137.16 80.01 0) (unit 1)
     (in_bom yes) (on_board yes) (dnp no) (fields_autoplaced)

Commit message: Slave
Parts:
- removed IC1: LoRa-E5, LoRaE5, symbol SamacSys_Parts:LoRa-E5
- removed U1: RP2040, Package_DFN_QFN:QFN-56-1EP_7x7mm_P0.4mm_EP3.2x3.2mm, symbol MCU_RaspberryPi:RP2040
Other:
- added sheet LoRa (LoRa_sch.kicad_sch)
- added sheet RPI2040_main (RPI2040_main_sch.kicad_sch)
Changed lines of the file:
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@@
 (kicad_sch (version 20230121) (generator eeschema)
   (paper "A4")
-  (symbol (lib_id "MCU_RaspberryPi:RP2040") (at 74.93 92.71 0) (unit 1)
-    (in_bom yes) (on_board yes) (dnp no) (fields_autoplaced)
-    (property "Reference" "U1" (at 77.1241 137.16 0)
-      (effects (font (size 1.27 1.27)) (justify left))
+  (sheet (at 152.4 63.5) (size 25.4 38.1) (fields_autoplaced)
+    (stroke (width 0.1524) (type solid))
+    (fill (color 0 0 0 0.0000))
+    (property "Sheetname" "RPI2040_main" (at 152.4 62.7884 0)
+      (effects (font (size 1.27 1.27)) (justify left bottom))
     )
-    (property "Value" "RP2040" (at 77.1241 139.7 0)
-      (effects (font (size 1.27 1.27)) (justify left))
+    (property "Sheetfile" "RPI2040_main_sch.kicad_sch" (at 152.4 102.1846 0)
+      (effects (font (size 1.27 1.27)) (justify left top))
     )
-    (property "Footprint" "Package_DFN_QFN:QFN-56-1EP_7x7mm_P0.4mm_EP3.2x3.2mm" (at 74.93 92.71 0)
-      (effects (font (size 1.27 1.27)) hide)
-    )
-    (property "Datasheet" "https://datasheets.raspberrypi.com/rp2040/rp2040-datasheet.pdf" (at 74.93 92.71 0)
-      (effects (font (size 1.27 1.27)) hide)
-    )
-    (pin "1")
-    (pin "10")
-    (pin "11")
-    (pin "12")
-    (pin "13")
-    (pin "14")
-    (pin "15")
-    (pin "16")
-    (pin "17")
-    (pin "18")
-    (pin "19")
-    (pin "2")
-    (pin "20")
-    (pin "21")
-    (pin "22")
-    (pin "23")
-    (pin "24")
-    (pin "25")
-    (pin "26")
-    (pin "27")
-    (pin "28")
-    (pin "29")
-    (pin "3")
-    (pin "30")
-    (pin "31")
-    (pin "32")
-    (pin "33")
-    (pin "34")
-    (pin "35")
-    (pin "36")
-    (pin "37")
-    (pin "38")
-    (pin "39")
-    (pin "4")
-    (pin "40")
-    (pin "41")
-    (pin "42")
-    (pin "43")
-    (pin "44")
-    (pin "45")
-    (pin "46")
-    (pin "47")
-    (pin "48")
-    (pin "49")
-    (pin "5")
-    (pin "50")
-    (pin "51")
-    (pin "52")
-    (pin "53")
-    (pin "54")
-    (pin "55")
-    (pin "56")
-    (pin "57")
-    (pin "6")
-    (pin "7")
-    (pin "8")
-    (pin "9")
     (instances
       (project "wireless_Slave"
-        (path "/0e0a1f86-1a9d-413b-96af-bc4dca868b1d"
-          (reference "U1") (unit 1)
-        )
+        (path "/0e0a1f86-1a9d-413b-96af-bc4dca868b1d" (page "2"))
       )
     )
   )
-  (symbol (lib_id "SamacSys_Parts:LoRa-E5") (at 137.16 80.01 0) (unit 1)
-    (in_bom yes) (on_board yes) (dnp no) (fields_autoplaced)
-    (property "Reference" "IC1" (at 168.91 73.0819 0)
-      (effects (font (size 1.27 1.27)))
+  (sheet (at 223.52 41.91) (size 22.86 13.97) (fields_autoplaced)
+    (stroke (width 0.1524) (type solid))
+    (fill (color 0 0 0 0.0000))
+    (property "Sheetname" "LoRa" (at 223.52 41.1984 0)
+      (effects (font (size 1.27 1.27)) (justify left bottom))
     )
-    (property "Value" "LoRa-E5" (at 168.91 75.6219 0)
-      (effects (font (size 1.27 1.27)))
+    (property "Sheetfile" "LoRa_sch.kicad_sch" (at 223.52 56.4646 0)
+      (effects (font (size 1.27 1.27)) (justify left top))
     )
-    (property "Footprint" "LoRaE5" (at 163.83 164.77 0)
-      (effects (font (size 1.27 1.27)) (justify left top) hide)
-    )
-    (property "Datasheet" "https://no.mouser.com/datasheet/2/744/LoRa_E5_module_datasheet_V1_0-2488126.pdf" (at 163.83 264.77 0)
-      (effects (font (size 1.27 1.27)) (justify left top) hide)
-    )
-    (property "Height" "2.5" (at 163.83 464.77 0)
-      (effects (font (size 1.27 1.27)) (justify left top) hide)
-    )
-    (property "Manufacturer_Name" "Seeed Studio" (at 163.83 564.77 0)
-      (effects (font (size 1.27 1.27)) (justify left top) hide)
-    )
-    (property "Manufacturer_Part_Number" "LoRa-E5" (at 163.83 664.77 0)
-      (effects (font (size 1.27 1.27)) (justify left top) hide)
-    )
-    (property "Mouser Part Number" "" (at 163.83 764.77 0)
-      (effects (font (size 1.27 1.27)) (justify left top) hide)
-    )
-    (property "Mouser Price/Stock" "" (at 163.83 864.77 0)
-      (effects (font (size 1.27 1.27)) (justify left top) hide)
-    )
-    (property "Arrow Part Number" "" (at 163.83 964.77 0)
-      (effects (font (size 1.27 1.27)) (justify left top) hide)
-    )
-    (property "Arrow Price/Stock" "" (at 163.83 1064.77 0)
-      (effects (font (size 1.27 1.27)) (justify left top) hide)
-    )
-    (pin "1")
-    (pin "10")
-    (pin "11")
-    (pin "12")
-    (pin "13")
-    (pin "14")
-    (pin "15")
-    (pin "16")
-    (pin "17")
-    (pin "18")
-    (pin "19")
-    (pin "2")
-    (pin "20")
-    (pin "21")
-    (pin "22")
-    (pin "23")
-    (pin "24")
-    (pin "25")
-    (pin "26")
-    (pin "27")
-    (pin "28")
-    (pin "3")
-    (pin "4")
-    (pin "5")
-    (pin "6")
-    (pin "7")
-    (pin "8")
-    (pin "9")
     (instances
       (project "wireless_Slave"
-        (path "/0e0a1f86-1a9d-413b-96af-bc4dca868b1d"
-          (reference "IC1") (unit 1)
-        )
+        (path "/0e0a1f86-1a9d-413b-96af-bc4dca868b1d" (page "3"))
       )
     )

Commit message: ændringer
Other:
- sheet LoRa ports: added Boot, RXD, Reset, TXD; removed none
Changed lines of the file:
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@@
     )
   )
-  (sheet (at 223.52 41.91) (size 22.86 13.97) (fields_autoplaced)
+  (sheet (at 199.39 68.58) (size 22.86 31.75) (fields_autoplaced)
     (stroke (width 0.1524) (type solid))
     (fill (color 0 0 0 0.0000))
-    (property "Sheetname" "LoRa" (at 223.52 41.1984 0)
+    (property "Sheetname" "LoRa" (at 199.39 67.8684 0)
       (effects (font (size 1.27 1.27)) (justify left bottom))
     )
-    (property "Sheetfile" "LoRa_sch.kicad_sch" (at 223.52 56.4646 0)
+    (property "Sheetfile" "LoRa_sch.kicad_sch" (at 199.39 100.9146 0)
       (effects (font (size 1.27 1.27)) (justify left top))
     )
+    (pin "Boot" input (at 199.39 73.66 180)
+      (effects (font (size 1.27 1.27)) (justify left))
+    )
+    (pin "Reset" input (at 199.39 76.2 180)
+      (effects (font (size 1.27 1.27)) (justify left))
+    )
+    (pin "RXD" input (at 199.39 80.01 180)
+      (effects (font (size 1.27 1.27)) (justify left))
+    )
+    (pin "TXD" input (at 199.39 82.55 180)
+      (effects (font (size 1.27 1.27)) (justify left))
+    )
     (instances

Commit message: ændringer
Other:
- added sheet Temp+Hum (Temp+Hum.kicad_sch)
Changed lines of the file:
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@@
+    )
+  )
+  (sheet (at 71.12 74.93) (size 27.94 26.67) (fields_autoplaced)
+    (stroke (width 0.1524) (type solid))
+    (fill (color 0 0 0 0.0000))
+    (property "Sheetname" "Temp+Hum" (at 71.12 74.2184 0)
+      (effects (font (size 1.27 1.27)) (justify left bottom))
+    )
+    (property "Sheetfile" "Temp+Hum.kicad_sch" (at 71.12 102.1846 0)
+      (effects (font (size 1.27 1.27)) (justify left top))
+    )
+    (instances
+      (project "wireless_Slave"
+        (path "/0e0a1f86-1a9d-413b-96af-bc4dca868b1d" (page "4"))
+      )
     )
   )

Commit message: bæ
Other:
- removed sheet Temp+Hum
- sheet RPI2040_main ports: added LoRa_BOO, LoRa_RES, RXD, TXD; removed none
Changed lines of the file:
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@@
 (kicad_sch (version 20230121) (generator eeschema)
   (paper "A4")
+  (wire (pts (xy 177.8 73.66) (xy 199.39 73.66))
+    (stroke (width 0) (type default))
+  )
+  (wire (pts (xy 177.8 80.01) (xy 199.39 80.01))
+    (stroke (width 0) (type default))
+  )
+  (wire (pts (xy 177.8 76.2) (xy 199.39 76.2))
+    (stroke (width 0) (type default))
+  )
+  (wire (pts (xy 177.8 82.55) (xy 199.39 82.55))
+    (stroke (width 0) (type default))
+  )
   (sheet (at 152.4 63.5) (size 25.4 38.1) (fields_autoplaced)
     (stroke (width 0.1524) (type solid))
@@
     (property "Sheetfile" "RPI2040_main_sch.kicad_sch" (at 152.4 102.1846 0)
       (effects (font (size 1.27 1.27)) (justify left top))
+    )
+    (pin "RXD" input (at 177.8 80.01 0)
+      (effects (font (size 1.27 1.27)) (justify right))
+    )
+    (pin "TXD" output (at 177.8 82.55 0)
+      (effects (font (size 1.27 1.27)) (justify right))
+    )
+    (pin "LoRa_BOO" input (at 177.8 73.66 0)
+      (effects (font (size 1.27 1.27)) (justify right))
+    )
+    (pin "LoRa_RES" input (at 177.8 76.2 0)
+      (effects (font (size 1.27 1.27)) (justify right))
     )
     (instances
@@
       )
     )
-  )
-  (sheet (at 71.12 74.93) (size 27.94 26.67) (fields_autoplaced)
-    (stroke (width 0.1524) (type solid))
-    (fill (color 0 0 0 0.0000))
-    (property "Sheetname" "Temp+Hum" (at 71.12 74.2184 0)
-      (effects (font (size 1.27 1.27)) (justify left bottom))
-    )
-    (property "Sheetfile" "Temp+Hum.kicad_sch" (at 71.12 102.1846 0)
-      (effects (font (size 1.27 1.27)) (justify left top))
-    )
-    (instances
-      (project "wireless_Slave"
-        (path "/0e0a1f86-1a9d-413b-96af-bc4dca868b1d" (page "4"))
-      )
-    )

Commit message: Ændring
Changed lines of the file:
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@@
 (kicad_sch (version 20230121) (generator eeschema)
   (paper "A4")
-  (wire (pts (xy 177.8 73.66) (xy 199.39 73.66))
+  (wire (pts (xy 97.79 42.545) (xy 119.38 42.545))
     (stroke (width 0) (type default))
   )
-  (wire (pts (xy 177.8 80.01) (xy 199.39 80.01))
+  (wire (pts (xy 97.79 48.895) (xy 119.38 48.895))
     (stroke (width 0) (type default))
   )
-  (wire (pts (xy 177.8 76.2) (xy 199.39 76.2))
+  (wire (pts (xy 97.79 45.085) (xy 119.38 45.085))
     (stroke (width 0) (type default))
   )
-  (wire (pts (xy 177.8 82.55) (xy 199.39 82.55))
+  (wire (pts (xy 97.79 51.435) (xy 119.38 51.435))
     (stroke (width 0) (type default))
   )
-  (sheet (at 152.4 63.5) (size 25.4 38.1) (fields_autoplaced)
+  (sheet (at 72.39 32.385) (size 25.4 38.1) (fields_autoplaced)
     (stroke (width 0.1524) (type solid))
     (fill (color 0 0 0 0.0000))
-    (property "Sheetname" "RPI2040_main" (at 152.4 62.7884 0)
+    (property "Sheetname" "RPI2040_main" (at 72.39 31.6734 0)
       (effects (font (size 1.27 1.27)) (justify left bottom))
     )
-    (property "Sheetfile" "RPI2040_main_sch.kicad_sch" (at 152.4 102.1846 0)
+    (property "Sheetfile" "RPI2040_main_sch.kicad_sch" (at 72.39 71.0696 0)
       (effects (font (size 1.27 1.27)) (justify left top))
     )
-    (pin "RXD" input (at 177.8 80.01 0)
+    (pin "RXD" input (at 97.79 48.895 0)
       (effects (font (size 1.27 1.27)) (justify right))
     )
-    (pin "TXD" output (at 177.8 82.55 0)
+    (pin "TXD" output (at 97.79 51.435 0)
       (effects (font (size 1.27 1.27)) (justify right))
     )
-    (pin "LoRa_BOO" input (at 177.8 73.66 0)
+    (pin "LoRa_BOO" input (at 97.79 42.545 0)
       (effects (font (size 1.27 1.27)) (justify right))
     )
-    (pin "LoRa_RES" input (at 177.8 76.2 0)
+    (pin "LoRa_RES" input (at 97.79 45.085 0)
       (effects (font (size 1.27 1.27)) (justify right))
     )
@@
     )
   )
-  (sheet (at 199.39 68.58) (size 22.86 31.75) (fields_autoplaced)
+  (sheet (at 119.38 37.465) (size 22.86 31.75) (fields_autoplaced)
     (stroke (width 0.1524) (type solid))
     (fill (color 0 0 0 0.0000))
-    (property "Sheetname" "LoRa" (at 199.39 67.8684 0)
+    (property "Sheetname" "LoRa" (at 119.38 36.7534 0)
       (effects (font (size 1.27 1.27)) (justify left bottom))
     )
-    (property "Sheetfile" "LoRa_sch.kicad_sch" (at 199.39 100.9146 0)
+    (property "Sheetfile" "LoRa_sch.kicad_sch" (at 119.38 69.7996 0)
       (effects (font (size 1.27 1.27)) (justify left top))
     )
-    (pin "Boot" input (at 199.39 73.66 180)
+    (pin "Boot" input (at 119.38 42.545 180)
       (effects (font (size 1.27 1.27)) (justify left))
     )
-    (pin "Reset" input (at 199.39 76.2 180)
+    (pin "Reset" input (at 119.38 45.085 180)
       (effects (font (size 1.27 1.27)) (justify left))
     )
-    (pin "RXD" input (at 199.39 80.01 180)
+    (pin "RXD" input (at 119.38 48.895 180)
       (effects (font (size 1.27 1.27)) (justify left))
     )
-    (pin "TXD" input (at 199.39 82.55 180)
+    (pin "TXD" input (at 119.38 51.435 180)
       (effects (font (size 1.27 1.27)) (justify left))
     )
