File: Wireless modbus/Wireless slave/wireless_Slave/wireless_Slave.kicad_sch (KiCad schematic)
At the start: 0 parts

Commit message: test
Other:
- sheet RPI2040_main ports: added LoRa_RXD, LoRa_TXD; removed RXD, TXD
Changed lines of the file:
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@@
       (effects (font (size 1.27 1.27)) (justify left top))
-    )
-    (pin "RXD" input (at 177.8 80.01 0)
-      (effects (font (size 1.27 1.27)) (justify right))
-    )
-    (pin "TXD" output (at 177.8 82.55 0)
-      (effects (font (size 1.27 1.27)) (justify right))
     )
     (pin "LoRa_BOO" input (at 177.8 73.66 0)
@@
       (effects (font (size 1.27 1.27)) (justify right))
     )
+    (pin "LoRa_RXD" input (at 177.8 80.01 0)
+      (effects (font (size 1.27 1.27)) (justify right))
+    )
+    (pin "LoRa_TXD" output (at 177.8 82.55 0)
+      (effects (font (size 1.27 1.27)) (justify right))
+    )

Commit message: tjek
Other:
- removed sheet LoRa
- sheet RPI2040_main ports: added none; removed LoRa_BOO, LoRa_RES, LoRa_RXD, LoRa_TXD
Changed lines of the file:
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@@
 (kicad_sch (version 20230121) (generator eeschema)
   (paper "A4")
-  (wire (pts (xy 177.8 73.66) (xy 199.39 73.66))
-    (stroke (width 0) (type default))
-  )
-  (wire (pts (xy 177.8 80.01) (xy 199.39 80.01))
-    (stroke (width 0) (type default))
-  )
-  (wire (pts (xy 177.8 76.2) (xy 199.39 76.2))
-    (stroke (width 0) (type default))
-  )
-  (wire (pts (xy 177.8 82.55) (xy 199.39 82.55))
-    (stroke (width 0) (type default))
-  )
   (sheet (at 152.4 63.5) (size 25.4 38.1) (fields_autoplaced)
     (stroke (width 0.1524) (type solid))
@@
       (effects (font (size 1.27 1.27)) (justify left top))
     )
-    (pin "LoRa_BOO" input (at 177.8 73.66 0)
-      (effects (font (size 1.27 1.27)) (justify right))
-    )
-    (pin "LoRa_RES" input (at 177.8 76.2 0)
-      (effects (font (size 1.27 1.27)) (justify right))
-    )
-    (pin "LoRa_RXD" input (at 177.8 80.01 0)
-      (effects (font (size 1.27 1.27)) (justify right))
-    )
-    (pin "LoRa_TXD" output (at 177.8 82.55 0)
-      (effects (font (size 1.27 1.27)) (justify right))
-    )
     (instances
       (project "wireless_Slave"
@@
       )
     )
-  )
-  (sheet (at 199.39 68.58) (size 22.86 31.75) (fields_autoplaced)
-    (stroke (width 0.1524) (type solid))
-    (fill (color 0 0 0 0.0000))
-    (property "Sheetname" "LoRa" (at 199.39 67.8684 0)
-      (effects (font (size 1.27 1.27)) (justify left bottom))
-    )
-    (property "Sheetfile" "LoRa_sch.kicad_sch" (at 199.39 100.9146 0)
-      (effects (font (size 1.27 1.27)) (justify left top))
-    )
-    (pin "Boot" input (at 199.39 73.66 180)
-      (effects (font (size 1.27 1.27)) (justify left))
-    )
-    (pin "Reset" input (at 199.39 76.2 180)
-      (effects (font (size 1.27 1.27)) (justify left))
-    )
-    (pin "RXD" input (at 199.39 80.01 180)
-      (effects (font (size 1.27 1.27)) (justify left))
-    )
-    (pin "TXD" input (at 199.39 82.55 180)
-      (effects (font (size 1.27 1.27)) (justify left))
-    )
-    (instances
-      (project "wireless_Slave"
-        (path "/0e0a1f86-1a9d-413b-96af-bc4dca868b1d" (page "3"))
-      )
-    )
