File: Wireless modbus/Wireless slave/wireless_Slave/RPI2040_main_sch.kicad_sch (KiCad schematic)
At the start: 1 part, among them U1 RP2040

Commit message: ændringer
Parts:
- added C4: C, symbol Device:C
- added J3: Conn_01x02, symbol Connector_Generic:Conn_01x02
- added R1: R, symbol Device:R
- added U2: W25Q128JVS, Package_SO:SOIC-8_5.23x5.23mm_P1.27mm, symbol Memory_Flash:W25Q128JVS
- added Y1: Crystal, symbol Device:Crystal
Changed lines of the file:
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@@
 (kicad_sch (version 20230121) (generator eeschema)
   (paper "A4")
+  (symbol (lib_id "Device:R") (at 120.65 154.94 0) (unit 1)
+    (in_bom yes) (on_board yes) (dnp no) (fields_autoplaced)
+    (property "Reference" "R1" (at 123.19 153.67 0)
+      (effects (font (size 1.27 1.27)) (justify left))
+    )
+    (property "Value" "R" (at 123.19 156.21 0)
+      (effects (font (size 1.27 1.27)) (justify left))
+    )
+    (property "Footprint" "" (at 118.872 154.94 90)
+      (effects (font (size 1.27 1.27)) hide)
+    )
+    (property "Datasheet" "~" (at 120.65 154.94 0)
+      (effects (font (size 1.27 1.27)) hide)
+    )
+    (pin "1")
+    (pin "2")
+    (instances
+      (project "wireless_Slave"
+        (path "/0e0a1f86-1a9d-413b-96af-bc4dca868b1d/58bbf317-6f19-4695-b4b3-bbbe360cf741"
+          (reference "R1") (unit 1)
+        )
+      )
+    )
+  )
+  (symbol (lib_id "Device:Crystal") (at 80.01 156.21 0) (unit 1)
+    (in_bom yes) (on_board yes) (dnp no) (fields_autoplaced)
+    (property "Reference" "Y1" (at 80.01 148.59 0)
+      (effects (font (size 1.27 1.27)))
+    )
+    (property "Value" "Crystal" (at 80.01 151.13 0)
+      (effects (font (size 1.27 1.27)))
+    )
+    (property "Footprint" "" (at 80.01 156.21 0)
+      (effects (font (size 1.27 1.27)) hide)
+    )
+    (property "Datasheet" "~" (at 80.01 156.21 0)
+      (effects (font (size 1.27 1.27)) hide)
+    )
+    (pin "1")
+    (pin "2")
+    (instances
+      (project "wireless_Slave"
+        (path "/0e0a1f86-1a9d-413b-96af-bc4dca868b1d/58bbf317-6f19-4695-b4b3-bbbe360cf741"
+          (reference "Y1") (unit 1)
+        )
+      )
+    )
+  )
+  (symbol (lib_id "Connector_Generic:Conn_01x02") (at 39.37 113.03 0) (unit 1)
+    (in_bom yes) (on_board yes) (dnp no) (fields_autoplaced)
+    (property "Reference" "J3" (at 41.91 113.03 0)
+      (effects (font (size 1.27 1.27)) (justify left))
+    )
+    (property "Value" "Conn_01x02" (at 41.91 115.57 0)
+      (effects (font (size 1.27 1.27)) (justify left))
+    )
+    (property "Footprint" "" (at 39.37 113.03 0)
+      (effects (font (size 1.27 1.27)) hide)
+    )
+    (property "Datasheet" "~" (at 39.37 113.03 0)
+      (effects (font (size 1.27 1.27)) hide)
+    )
+    (pin "1")
+    (pin "2")
+    (instances
+      (project "wireless_Slave"
+        (path "/0e0a1f86-1a9d-413b-96af-bc4dca868b1d/58bbf317-6f19-4695-b4b3-bbbe360cf741"
+          (reference "J3") (unit 1)
+        )
+      )
+    )
+  )
+  (symbol (lib_id "Memory_Flash:W25Q128JVS") (at 71.12 111.76 0) (unit 1)
+    (in_bom yes) (on_board yes) (dnp no) (fields_autoplaced)
+    (property "Reference" "U2" (at 80.01 110.49 0)
+      (effects (font (size 1.27 1.27)) (justify left))
+    )
+    (property "Value" "W25Q128JVS" (at 80.01 113.03 0)
+      (effects (font (size 1.27 1.27)) (justify left))
+    )
+    (property "Footprint" "Package_SO:SOIC-8_5.23x5.23mm_P1.27mm" (at 71.12 111.76 0)
+      (effects (font (size 1.27 1.27)) hide)
+    )
+    (property "Datasheet" "http://www.winbond.com/resource-files/w25q128jv_dtr%20revc%2003272018%20plus.pdf" (at 71.12 111.76 0)
+      (effects (font (size 1.27 1.27)) hide)
+    )
+    (pin "1")
+    (pin "2")
+    (pin "3")
+    (pin "4")
+    (pin "5")
+    (pin "6")
+    (pin "7")
+    (pin "8")
+    (instances
+      (project "wireless_Slave"
+        (path "/0e0a1f86-1a9d-413b-96af-bc4dca868b1d/58bbf317-6f19-4695-b4b3-bbbe360cf741"
+          (reference "U2") (unit 1)
+        )
+      )
+    )
+  )
   (symbol (lib_id "MCU_RaspberryPi:RP2040") (at 133.35 88.9 0) (unit 1)
     (in_bom yes) (on_board yes) (dnp no) (fields_autoplaced)
@@
         )
       )
+    )
+  )
+  (symbol (lib_id "Device:C") (at 101.6 151.13 0) (unit 1)
+    (in_bom yes) (on_board yes) (dnp no) (fields_autoplaced)
+    (property "Reference" "C4" (at 105.41 149.86 0)
+      (effects (font (size 1.27 1.27)) (justify left))
+    )
+    (property "Value" "C" (at 105.41 152.4 0)
+      (effects (font (size 1.27 1.27)) (justify left))
+    )
+    (property "Footprint" "" (at 102.5652 154.94 0)
+      (effects (font (size 1.27 1.27)) hide)
+    )
+    (property "Datasheet" "~" (at 101.6 151.13 0)
+      (effects (font (size 1.27 1.27)) hide)
+    )
+    (pin "1")
+    (pin "2")
+    (instances
+      (project "wireless_Slave"
+        (path "/0e0a1f86-1a9d-413b-96af-bc4dca868b1d/58bbf317-6f19-4695-b4b3-bbbe360cf741"
+          (reference "C4") (unit 1)
+        )
+      )

Commit message: ændringer
Parts:
- added C10, C11, C12, C13, C14, C5, C7, C8, C9: 100n, symbol Device:C
- added C15, C16: 1u, symbol Device:C
- added C6: 27p, symbol Device:C
- added J4: USB, symbol Connector_Generic:Conn_01x02
- added R10, R11, R4, R5, R6, R7, R8, R9: 10K, symbol Device:R
- added R2: 1K, symbol Device:R
- added R3: 27, symbol Device:R
- added S1: 219-8MSTR, 2198MSTR, symbol SamacSys_Parts:219-8MSTR
- added Ul: MCP9700Ax-ETT, Package_TO_SOT_SMD:SOT-23, symbol Sensor_Temperature:MCP9700Ax-ETT
- C4: value C -> 27p
- R1: value R -> 27
- U1: JLCPCB (none) -> C2040
- U2: JLCPCB (none) -> C97521
- Y1: value Crystal -> 12.000MHz
Connections:
- net at R1.1: now also J4.2 (Pin_2)
- net D+: now reaches R1.2
- net D+: now also U1.47 (USB_DP)
- net at Y1.1: now also C4.2, U1.21 (XOUT)
- net at Y1.2: now also U1.20 (XIN), C6.2
- net GND: now reaches J3.1 (Pin_1)
- net GND: now also C4.1, U1.19 (TESTEN), U1.57 (GND), U2.4 (GND), C10.2, C11.2, C12.2, C13.2, C14.2, C15.2, C16.2, C5.2, C6.1, C7.2, C8.2, C9.2, R10.1, R11.1, R4.1, R5.1, R6.1, R7.1, R8.1, R9.1, Ul.3 (GND)
- net at J3.2 (Pin_2): now also R2.1
- net QSPI_SS: now reaches U2.1 (~{CS})
- net QSPI_SS: now also U1.56 (QSPI_SS), R2.2
- net QSPI_SD1: now reaches U2.2 (DO(IO1))
- net QSPI_SD1: now also U1.55 (QSPI_SD1)
- net QSPI_SD2: now reaches U2.3 (IO2)
- net QSPI_SD2: now also U1.54 (QSPI_SD2)
- net QSPI_SD0: now reaches U2.5 (DI(IO0))
- net QSPI_SD0: now also U1.53 (QSPI_SD0)
- net QSPI_SCLK: now reaches U2.6 (CLK)
- net QSPI_SCLK: now also U1.52 (QSPI_SCLK)
- net QSPI_SD3: now reaches U2.7 (IO3)
- net QSPI_SD3: now also U1.51 (QSPI_SD3)
- net +3.3V: now reaches U2.8 (VCC)
- net +3.3V: now also U1.1 (IOVDD), U1.10 (IOVDD), U1.22 (IOVDD), U1.33 (IOVDD), U1.42 (IOVDD), U1.43 (ADC_AVDD), U1.44 (VREG_IN), U1.48 (USB_VDD), U1.49 (IOVDD), C10.1, C11.1, C12.1, C13.1, C14.1, C16.1, C5.1, C9.1, S1.1, S1.11, S1.13, S1.15, S1.3, S1.5, S1.7, S1.9, Ul.1 (V_{DD})
- net GPIO8: now reaches U1.11 (GPIO8)
- net GPIO9: now reaches U1.12 (GPIO9)
- net GPIO10: now reaches U1.13 (GPIO10)
- net GPIO11: now reaches U1.14 (GPIO11)
- net GPIO12: now reaches U1.15 (GPIO12)
- net GPIO13: now reaches U1.16 (GPIO13)
- net GPIO14: now reaches U1.17 (GPIO14)
- net GPIO15: now reaches U1.18 (GPIO15)
- net GPIO0: now reaches U1.2 (GPIO0)
- net +1V1: now reaches U1.23 (DVDD), U1.50 (DVDD)
- net +1V1: now also U1.45 (VREG_VOUT), C15.1, C7.1, C8.1
- net SWCLK: now reaches U1.24 (SWCLK)
- net SWD: now reaches U1.25 (SWD)
- net RUN: now reaches U1.26 (RUN)
- net GPIO16: now reaches U1.27 (GPIO16)
- net GPIO17: now reaches U1.28 (GPIO17)
- net GPIO18: now reaches U1.29 (GPIO18)
- net GPIO18: now also R11.2, S1.2
- net GPIO1: now reaches U1.3 (GPIO1)
- net GPIO19: now reaches U1.30 (GPIO19)
- net GPIO19: now also R10.2, S1.4
- net GPIO20: now reaches U1.31 (GPIO20)
- net GPIO20: now also R9.2, S1.6
- net GPIO21: now reaches U1.32 (GPIO21)
- net GPIO21: now also R8.2, S1.8
- net GPIO22: now reaches U1.34 (GPIO22)
- net GPIO22: now also R7.2, S1.10
- net GPIO23: now reaches U1.35 (GPIO23)
- net GPIO23: now also R6.2, S1.12
- net GPIO24: now reaches U1.36 (GPIO24)
- net GPIO24: now also R5.2, S1.14
- net GPIO25: now reaches U1.37 (GPIO25)
- net GPIO25: now also R4.2, S1.16
- net ADC0: now reaches U1.38 (GPIO26_ADC0)
- net ADC1: now reaches U1.39 (GPIO27_ADC1)
- net GPIO2: now reaches U1.4 (GPIO2)
- net ADC2: now reaches U1.40 (GPIO28_ADC2)
- net ADC3: now reaches U1.41 (GPIO29_ADC3)
- net ADC3: now also Ul.2 (V_{OUT})
- net D-: now reaches U1.46 (USB_DM)
- net D-: now also R3.2
- net GPIO3: now reaches U1.5 (GPIO3)
- net GPIO4: now reaches U1.6 (GPIO4)
- net GPIO5: now reaches U1.7 (GPIO5)
- net GPIO6: now reaches U1.8 (GPIO6)
- net GPIO7: now reaches U1.9 (GPIO7)
- new net: J4.1 (Pin_1), R3.1
Other:
- note added: "C15 og C16 sættes så tæt på 2040 som muligt"
- note added: "R1 og R2 sættes så tæt på 2040 som muligt"
- moved on the sheet: C4, J3, U1, U2, Y1

Commit message: ændringer
Parts:
- removed Ul: MCP9700Ax-ETT, Package_TO_SOT_SMD:SOT-23, symbol Sensor_Temperature:MCP9700Ax-ETT
- added C17: 100n, symbol Device:C
- added IC2: SHT30-DIS-B10KS, SON50P250X250X100-9N-D, symbol SamacSys_Parts:SHT30-DIS-B10KS
Connections:
- net +3.3V: now also C17.1, IC2.5 (VDD)
- net GND: now also C17.2, IC2.2 (ADDR), IC2.7 (R), IC2.8 (VSS), IC2.9 (EP)
- net GPIO2: now also IC2.1 (SDA)
- net GPIO3: now also IC2.4 (SCL)
- net GPIO0 renamed TXD
- net GPIO1 renamed RXD
- no-connect marks 0 -> 2
Other:
- moved on the sheet: C5, J3, R10, R11, R2, R4, R5, R6, R7, R8, R9, U2

Commit message: bæ
Connections:
- net GPIO16 renamed LoRa_RES
- net GPIO17 renamed LoRa_BOO
Changed lines of the file:
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@@
-    (stroke (width 0) (type default))
-  )
-  (wire (pts (xy 177.8 104.14) (xy 185.42 104.14))
     (stroke (width 0) (type default))
   )
@@
     (stroke (width 0) (type default))
   )
+  (wire (pts (xy 187.96 105.41) (xy 187.96 106.68))
+    (stroke (width 0) (type default))
+  )
+  (wire (pts (xy 177.8 106.68) (xy 187.96 106.68))
+    (stroke (width 0) (type default))
+  )
   (wire (pts (xy 196.85 39.37) (xy 185.42 39.37))
     (stroke (width 0) (type default))
@@
     (stroke (width 0) (type default))
   )
+  (wire (pts (xy 190.5 104.14) (xy 190.5 102.87))
+    (stroke (width 0) (type default))
+  )
   (wire (pts (xy 185.42 46.99) (xy 191.77 46.99))
     (stroke (width 0) (type default))
@@
     (stroke (width 0) (type default))
   )
-  (wire (pts (xy 177.8 106.68) (xy 185.42 106.68))
-    (stroke (width 0) (type default))
-  )
   (wire (pts (xy 177.8 66.04) (xy 185.42 66.04))
     (stroke (width 0) (type default))
@@
     (stroke (width 0) (type default))
   )
+  (wire (pts (xy 190.5 105.41) (xy 187.96 105.41))
+    (stroke (width 0) (type default))
+  )
   (wire (pts (xy 208.28 46.99) (xy 219.71 46.99))
     (stroke (width 0) (type default))
@@
     (stroke (width 0) (type default))
   )
+  (wire (pts (xy 177.8 104.14) (xy 190.5 104.14))
+    (stroke (width 0) (type default))
+  )
   (wire (pts (xy 177.8 81.28) (xy 185.42 81.28))
     (stroke (width 0) (type default))
@@
   (label "QSPI_SD0" (at 115.57 86.36 0) (fields_autoplaced)
     (effects (font (size 1.27 1.27)) (justify left bottom))
+  )
+  (hierarchical_label "LoRa_BOO" (shape input) (at 190.5 105.41 0) (fields_autoplaced)
+    (effects (font (size 1.27 1.27)) (justify left))
   )
   (hierarchical_label "RXD" (shape input) (at 185.42 66.04 0) (fields_autoplaced)
     (effects (font (size 1.27 1.27)) (justify left))
   )
+  (hierarchical_label "LoRa_RES" (shape input) (at 190.5 102.87 0) (fields_autoplaced)
+    (effects (font (size 1.27 1.27)) (justify left))
+  )

Commit message: næ
Parts:
- added R12: 10K, symbol Device:R
- added R13: R_Photo, symbol Device:R_Photo
Connections:
- net +3.3V: now also R13.1
- net GND: now also R12.1
- net ADC1 renamed LUX
- net LUX: now also R12.2, R13.2
Changed lines of the file:
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@@
   (junction (at 157.48 55.88) (diameter 0) (color 0 0 0 0)
+  )
+  (junction (at 273.05 151.13) (diameter 0) (color 0 0 0 0)
   )
   (junction (at 264.16 123.19) (diameter 0) (color 0 0 0 0)
@@
     (stroke (width 0) (type default))
   )
+  (wire (pts (xy 267.97 151.13) (xy 273.05 151.13))
+    (stroke (width 0) (type default))
+  )
   (wire (pts (xy 190.5 104.14) (xy 190.5 102.87))
     (stroke (width 0) (type default))
@@
     (stroke (width 0) (type default))
   )
+  (wire (pts (xy 273.05 149.86) (xy 273.05 151.13))
+    (stroke (width 0) (type default))
+  )
   (wire (pts (xy 234.95 115.57) (xy 241.3 115.57))
     (stroke (width 0) (type default))
@@
     (stroke (width 0) (type default))
   )
+  (wire (pts (xy 273.05 151.13) (xy 273.05 152.4))
+    (stroke (width 0) (type default))
+  )
   (wire (pts (xy 264.16 123.19) (xy 271.78 123.19))
     (stroke (width 0) (type default))
@@
     (stroke (width 0) (type default))
   )
+  (rectangle (start 266.7 134.62) (end 284.48 165.1)
+    (stroke (width 0) (type default))
+    (fill (type none))
+  )
   (rectangle (start 24.13 60.96) (end 95.25 109.22)
     (stroke (width 0) (type default))
@@
     (effects (font (size 1.27 1.27)) (justify left bottom))
   )
-  (label "ADC1" (at 185.42 134.62 180) (fields_autoplaced)
-    (effects (font (size 1.27 1.27)) (justify right bottom))
-  )
   (label "GPIO21" (at 185.42 116.84 180) (fields_autoplaced)
     (effects (font (size 1.27 1.27)) (justify right bottom))
@@
     (effects (font (size 1.27 1.27)) (justify left bottom))
   )
+  (label "LUX" (at 185.42 134.62 180) (fields_autoplaced)
+    (effects (font (size 1.27 1.27)) (justify right bottom))
+  )
   (label "QSPI_SD2" (at 115.57 91.44 0) (fields_autoplaced)
     (effects (font (size 1.27 1.27)) (justify left bottom))
@@
   )
   (label "QSPI_SD2" (at 49.53 92.71 0) (fields_autoplaced)
+    (effects (font (size 1.27 1.27)) (justify left bottom))
+  )
+  (label "LUX" (at 267.97 151.13 0) (fields_autoplaced)
     (effects (font (size 1.27 1.27)) (justify left bottom))
   )
@@
     )
   )
+  (symbol (lib_id "Device:R_Photo") (at 273.05 146.05 0) (unit 1)
+    (in_bom yes) (on_board yes) (dnp no) (fields_autoplaced)
+    (property "Reference" "R13" (at 275.59 144.78 0)
+      (effects (font (size 1.27 1.27)) (justify left))
+    )
+    (property "Value" "R_Photo" (at 275.59 147.32 0)
+      (effects (font (size 1.27 1.27)) (justify left))
+    )
+    (property "Footprint" "" (at 274.32 152.4 90)
+      (effects (font (size 1.27 1.27)) (justify left) hide)
+    )
+    (property "Datasheet" "~" (at 273.05 147.32 0)
+      (effects (font (size 1.27 1.27)) hide)
+    )
+    (pin "1")
+    (pin "2")
+    (instances
+      (project "wireless_Slave"
+        (path "/0e0a1f86-1a9d-413b-96af-bc4dca868b1d/58bbf317-6f19-4695-b4b3-bbbe360cf741"
+          (reference "R13") (unit 1)
+        )
+      )
+    )
+  )
   (symbol (lib_id "Connector_Generic:Conn_01x02") (at 109.22 73.66 180) (unit 1)
     (in_bom yes) (on_board yes) (dnp no)
@@
     )
   )
+  (symbol (lib_id "Device:R") (at 273.05 156.21 180) (unit 1)
+    (in_bom yes) (on_board yes) (dnp no) (fields_autoplaced)
+    (property "Reference" "R12" (at 275.59 154.94 0)
+      (effects (font (size 1.27 1.27)) (justify right))
+    )
+    (property "Value" "10K" (at 275.59 157.48 0)
+      (effects (font (size 1.27 1.27)) (justify right))
+    )
+    (property "Footprint" "" (at 274.828 156.21 90)
+      (effects (font (size 1.27 1.27)) hide)
+    )
+    (property "Datasheet" "~" (at 273.05 156.21 0)
+      (effects (font (size 1.27 1.27)) hide)
+    )
+    (pin "1")
+    (pin "2")
+    (instances
+      (project "wireless_Slave"
+        (path "/0e0a1f86-1a9d-413b-96af-bc4dca868b1d/58bbf317-6f19-4695-b4b3-bbbe360cf741"
+          (reference "R12") (unit 1)
+        )
+      )
+    )
+  )
   (symbol (lib_id "power:GND") (at 127 139.7 270) (unit 1)
     (in_bom yes) (on_board yes) (dnp no) (fields_autoplaced)
@@
         (path "/0e0a1f86-1a9d-413b-96af-bc4dca868b1d/58bbf317-6f19-4695-b4b3-bbbe360cf741"
           (reference "R10") (unit 1)
+        )
+      )
+    )
+  )
+  (symbol (lib_id "power:GND") (at 273.05 160.02 0) (unit 1)
+    (in_bom yes) (on_board yes) (dnp no)
+    (property "Reference" "#PWR026" (at 273.05 166.37 0)
+      (effects (font (size 1.27 1.27)) hide)
+    )
+    (property "Value" "GND" (at 273.05 163.83 0)
+      (effects (font (size 1.27 1.27)))
+    )
+    (property "Footprint" "" (at 273.05 160.02 0)
+      (effects (font (size 1.27 1.27)) hide)
+    )
+    (property "Datasheet" "" (at 273.05 160.02 0)
+      (effects (font (size 1.27 1.27)) hide)
+    )
+    (pin "1")
+    (instances
+      (project "wireless_Slave"
+        (path "/0e0a1f86-1a9d-413b-96af-bc4dca868b1d/58bbf317-6f19-4695-b4b3-bbbe360cf741"
+          (reference "#PWR026") (unit 1)
         )
       )
@@
         )
       )
+    )
+  )
+  (symbol (lib_id "power:+3.3V") (at 273.05 142.24 0) (unit 1)
+    (in_bom yes) (on_board yes) (dnp no) (fields_autoplaced)
+    (property "Reference" "#PWR027" (at 273.05 146.05 0)
+      (effects (font (size 1.27 1.27)) hide)
+    )
+    (property "Value" "+3.3V" (at 273.05 137.16 0)
+      (effects (font (size 1.27 1.27)))
+    )
+    (property "Footprint" "" (at 273.05 142.24 0)
+      (effects (font (size 1.27 1.27)) hide)
+    )
+    (property "Datasheet" "" (at 273.05 142.24 0)
+      (effects (font (size 1.27 1.27)) hide)
+    )
+    (pin "1")
+    (instances
+      (project "wireless_Slave"
+        (path "/0e0a1f86-1a9d-413b-96af-bc4dca868b1d/58bbf317-6f19-4695-b4b3-bbbe360cf741"
+          (reference "#PWR027") (unit 1)
+        )
+      )

Commit message: Ændring
Parts:
- added R14: 10K, symbol Device:R
- added U3: EKMB1107111, EKMB1107111, symbol SamacSys_Parts:EKMB1107111
Connections:
- net +3.3V: now also U3.1 (VDD)
- net GND: now also R14.1, U3.3 (GND)
- net GPIO4: now also R14.2, U3.2 (OUT)
Other:
- note added: "PIR sensor"

Commit message: wup wup
Parts:
- added C21: 100n, symbol Device:C
- renumbered C5 to C1, C11 to C10, C12 to C11, C13 to C12, C14 to C13, C17 to C14, C6 to C2, C4 to C3, C7 to C4, C8 to C5, C15 to C6, C16 to C7, C9 to C8, C10 to C9, IC2 to IC1, J3 to J1, J4 to J2, R14 to R1, R9 to R10, R10 to R11, R11 to R12, R12 to R14, R1 to R3, R3 to R4, R4 to R5, R5 to R6, R6 to R7, R7 to R8, R8 to R9, U3 to U1
Connections:
- net +3.3V: now also C21.1
- net GND: now also C21.2

Commit message: wup
Parts:
- removed S1: 219-8MSTR, 2198MSTR, symbol SamacSys_Parts:219-8MSTR
- removed Y1: 12.000MHz, symbol Device:Crystal
- added BT1: Battery_Cell, SamacSys_Parts3:BHAA-3, symbol Device:Battery_Cell
- added IC3: ZMOD4410AI1R, ZMOD4410AI1R, symbol SamacSys_Parts2:ZMOD4410AI1R
- added R18, R19, R20, R21, R22, R23, R24, R25: 10K, Resistor_SMD:R_0402_1005Metric, symbol Device:R
- added SW1: SW_DIP_x12, SamacSys_Parts3:21912LPST, symbol Switch:SW_DIP_x12
- added SW2: SW_DIP_x06, SamacSys_Parts3:2195MSTR, symbol Switch:SW_DIP_x06
- added Y3: 12MHz, SamacSys_Parts2:X322512MSB4SI, symbol Device:Crystal_GND24
- C1: renamed from C21; value 100n -> 100nf; footprint (none) -> Capacitor_SMD:C_0402_1005Metric
- C10: renamed from C9; value 100n -> 100nf; footprint (none) -> Capacitor_SMD:C_0402_1005Metric
- C11: renamed from C10; value 100n -> 100nf; footprint (none) -> Capacitor_SMD:C_0402_1005Metric
- C12: renamed from C11; value 100n -> 100nf; footprint (none) -> Capacitor_SMD:C_0402_1005Metric
- C13: renamed from C12; value 100n -> 100nf; footprint (none) -> Capacitor_SMD:C_0402_1005Metric
- C14: renamed from C13; value 100n -> 100nf; footprint (none) -> Capacitor_SMD:C_0402_1005Metric
- C15: renamed from C14; value 100n -> 100nf; footprint (none) -> Capacitor_SMD:C_0402_1005Metric
- C2: renamed from C1; value 100n -> 100nf; footprint (none) -> Capacitor_SMD:C_0402_1005Metric
- C3: renamed from C2; value 27p -> 27pf; footprint (none) -> Capacitor_SMD:C_0402_1005Metric
- C4: renamed from C3; value 27p -> 27pf; footprint (none) -> Capacitor_SMD:C_0402_1005Metric
- C5: renamed from C4; value 100n -> 100nf; footprint (none) -> Capacitor_SMD:C_0402_1005Metric
- C6: renamed from C5; value 100n -> 100nf; footprint (none) -> Capacitor_SMD:C_0402_1005Metric
- C7: renamed from C6; value 1u -> 1uf; footprint (none) -> Capacitor_SMD:C_0603_1608Metric
- C8: renamed from C7; value 1u -> 1uf; footprint (none) -> Capacitor_SMD:C_0603_1608Metric
- C9: renamed from C8; value 100n -> 100nf; footprint (none) -> Capacitor_SMD:C_0402_1005Metric
- J1, J2: footprint (none) -> Connector_PinHeader_2.54mm:PinHeader_1x02_P2.54mm_Vertical
- R1, R10, R11, R12, R14, R2, R3, R4, R5, R6, R7, R8, R9: footprint (none) -> Resistor_SMD:R_0402_1005Metric
- R13: footprint (none) -> SamacSys_Parts:02LDR1
Connections:
- net GPIO7 is gone; now on net LoRa_RES: U1.9 (GPIO7)
- net GPIO8 is gone; now on net LoRa_BOO: U1.11 (GPIO8)
- net +3.3V: now also BT1.1 (+), IC3.10 (VDDH), IC3.12 (VDDIO), IC3.5 (VDD)
- net GND: now also BT1.2 (-), IC3.6 (VSS_1), IC3.7 (VSS_2), IC3.9 (VSS_3), R18.1, R19.1, R20.1, R21.1, R22.1, R23.1, R24.1, R25.1, Y3.2, Y3.4
- net GPIO10: now also R25.2
- net GPIO11: now also R24.2
- net GPIO12: now also R12.2
- net GPIO13: now also R11.2
- net GPIO14: now also R10.2
- net GPIO15: now also R9.2
- net GPIO18: now also R6.2; no longer R12.2
- net GPIO19: now also R5.2; no longer R11.2
- net GPIO20: now also R23.2, SW2.1; no longer R10.2
- net GPIO21: now also R22.2, SW2.2; no longer R9.2
- net GPIO22: now also R21.2, SW2.3; no longer R8.2
- net GPIO23: now also R20.2, SW2.4; no longer R7.2
- net GPIO24: now also R19.2, SW2.5; no longer R6.2
- net GPIO25: now also R18.2, SW2.6; no longer R5.2
- net LoRa_BOO: no longer U1.28 (GPIO17)
- net LoRa_RES: no longer U1.27 (GPIO16)
- net at C3.2, U1.20 (XIN): now also Y3.3
- net at C4.2, U1.21 (XOUT): now also Y3.1
- net GPIO2 renamed SDA
- net SDA: now also IC3.2 (SDA)
- net GPIO3 renamed SCL
- net SCL: now also IC3.1 (SCL)
- net GPIO4 renamed PIR
- net GPIO5 renamed AIR_INT
- net AIR_INT: now also IC3.3 (INT)
- net GPIO6 renamed AIR_RES
- net AIR_RES: now also IC3.11 (RES_N)
- new net: SW2.10, SW2.11, SW2.12, SW2.7, SW2.8, SW2.9
- new net GPIO16: R8.2
- new net GPIO17: R7.2
- no-connect marks 2 -> 4
Other:
- note added: "Air quality sensor"
- note added: "DIP"
- note added: "Flash"
- note added: "LUX"
- note added: "Power"
- note added: "Temp/fugt sensor"
- moved on the sheet: R10, R11, R12, R5, R6, R7, R8, R9
