File: Wireless modbus/Wireless slave/wireless_Slave/RPI2040_main_sch.kicad_sch (KiCad schematic)
At the start: 62 parts, among them IC1 SHT30-DIS-B10KS, IC3 ZMOD4410AI1R, IC4 ADP5587ACPZ-R7, J1 Conn_01x02, J5 USB, J6 ON/OFF, J7 Digital_in, J8 I2C, SW1 SW_DIP_x12, SW2 SW_DIP_x06, U1 EKMB1107111, U1 RP2040, U2 W25Q128JVS, Y3 12MHz

Commit message: jaaaaaaaaaaaaa
Parts:
- SW2: footprint SamacSys_Parts3:2195MSTR -> SamacSys_Parts3:2196LPST
Connections:
- net +3.3V: now also S1.1, SW1.B1, SW1.B10, SW1.B11, SW1.B12, SW1.B2, SW1.B3, SW1.B4, SW1.B5, SW1.B6, SW1.B7, SW1.B8, SW1.B9; no longer SW1.A1, SW1.A10, SW1.A11, SW1.A12, SW1.A2, SW1.A3, SW1.A4, SW1.A5, SW1.A6, SW1.A7, SW1.A8, SW1.A9
- net C0: now also SW1.A9; no longer SW1.B9
- net C1: now also SW1.A10; no longer SW1.B10
- net C2: now also SW1.A11; no longer SW1.B11
- net C3: now also SW1.A12; no longer SW1.B12
- net C4: now also R23.2, SW2.A1; no longer R18.2, SW2.A6
- net C5: now also R22.2, SW2.A2; no longer R19.2, SW2.A5
- net C6: now also R21.2, SW2.A3; no longer R20.2, SW2.A4
- net C7: now also R20.2, SW2.A4; no longer R21.2, SW2.A3
- net C8: now also R19.2, SW2.A5; no longer R22.2, SW2.A2
- net C9: now also R18.2, SW2.A6; no longer R23.2, SW2.A1
- net R0: now also SW1.A8; no longer SW1.B8
- net R1: now also SW1.A7; no longer SW1.B7
- net R2: now also SW1.A6; no longer SW1.B6
- net R3: now also SW1.A5; no longer SW1.B5
- net R4: now also SW1.A4; no longer SW1.B4
- net R5: now also SW1.A3; no longer SW1.B3
- net R6: now also SW1.A2; no longer SW1.B2
- net R7: now also SW1.A1; no longer SW1.B1
Other:
- moved on the sheet: R18, R19, R20, R21, R22, R23
Changed lines of the file:
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@@
   (junction (at 104.775 227.965) (diameter 0) (color 0 0 0 0)
   )
-  (junction (at 95.25 197.485) (diameter 0) (color 0 0 0 0)
-  )
   (junction (at 212.09 72.39) (diameter 0) (color 0 0 0 0)
   )
@@
   (junction (at 21.59 210.185) (diameter 0) (color 0 0 0 0)
   )
+  (junction (at 95.25 200.025) (diameter 0) (color 0 0 0 0)
+  )
   (junction (at 382.27 180.34) (diameter 0) (color 0 0 0 0)
   )
@@
   (junction (at 21.59 200.025) (diameter 0) (color 0 0 0 0)
   )
-  (junction (at 95.25 200.025) (diameter 0) (color 0 0 0 0)
-  )
   (junction (at 95.25 207.645) (diameter 0) (color 0 0 0 0)
   )
@@
   (junction (at 76.835 247.015) (diameter 0) (color 0 0 0 0)
   )
+  (junction (at 95.25 197.485) (diameter 0) (color 0 0 0 0)
+  )
   (junction (at 21.59 217.805) (diameter 0) (color 0 0 0 0)
   )
@@
     (stroke (width 0) (type default))
   )
+  (wire (pts (xy 95.25 197.485) (xy 95.25 200.025))
+    (stroke (width 0) (type default))
+  )
   (wire (pts (xy 20.32 239.395) (xy 23.495 239.395))
     (stroke (width 0) (type default))
@@
     (stroke (width 0) (type default))
   )
-  (wire (pts (xy 95.25 197.485) (xy 95.25 200.025))
+  (wire (pts (xy 95.25 196.215) (xy 95.25 197.485))
     (stroke (width 0) (type default))
   )
@@
     (stroke (width 0) (type default))
   )
-  (wire (pts (xy 95.25 196.215) (xy 95.25 197.485))
-    (stroke (width 0) (type default))
-  )
   (wire (pts (xy 257.81 80.01) (xy 269.24 80.01))
     (stroke (width 0) (type default))
@@
     )
   )
-  (symbol (lib_id "Switch:SW_DIP_x12") (at 29.21 212.725 0) (unit 1)
-    (in_bom yes) (on_board yes) (dnp no) (fields_autoplaced)
+  (symbol (lib_id "Switch:SW_DIP_x12") (at 29.21 212.725 0) (mirror y) (unit 1)
+    (in_bom yes) (on_board yes) (dnp no)
     (property "Reference" "SW1" (at 29.21 189.865 0)
       (effects (font (size 1.27 1.27)))
@@
     )
   )
+  (symbol (lib_id "power:+3.3V") (at 384.175 177.8 0) (unit 1)
+    (in_bom yes) (on_board yes) (dnp no)
+    (property "Reference" "#PWR060" (at 384.175 181.61 0)
+      (effects (font (size 1.27 1.27)) hide)
+    )
+    (property "Value" "+3.3V" (at 381 175.26 0)
+      (effects (font (size 1.27 1.27)))
+    )
+    (property "Footprint" "" (at 384.175 177.8 0)
+      (effects (font (size 1.27 1.27)) hide)
+    )
+    (property "Datasheet" "" (at 384.175 177.8 0)
+      (effects (font (size 1.27 1.27)) hide)
+    )
+    (pin "1")
+    (instances
+      (project "wireless_Slave"
+        (path "/0e0a1f86-1a9d-413b-96af-bc4dca868b1d/58bbf317-6f19-4695-b4b3-bbbe360cf741"
+          (reference "#PWR060") (unit 1)
+        )
+      )
+    )
+  )
   (symbol (lib_id "power:+3.3V") (at 212.09 72.39 0) (unit 1)
     (in_bom yes) (on_board yes) (dnp no) (fields_autoplaced)
@@
     )
   )
-  (symbol (lib_id "Device:R") (at 89.535 224.155 180) (unit 1)
+  (symbol (lib_id "Device:R") (at 97.155 224.155 0) (mirror x) (unit 1)
     (in_bom yes) (on_board yes) (dnp no) (fields_autoplaced)
-    (property "Reference" "R20" (at 92.075 222.885 0)
+    (property "Reference" "R20" (at 94.615 222.885 0)
       (effects (font (size 1.27 1.27)) (justify right))
     )
-    (property "Value" "10K" (at 92.075 225.425 0)
+    (property "Value" "10K" (at 94.615 225.425 0)
       (effects (font (size 1.27 1.27)) (justify right))
     )
-    (property "Footprint" "Resistor_SMD:R_0402_1005Metric" (at 91.313 224.155 90)
+    (property "Footprint" "Resistor_SMD:R_0402_1005Metric" (at 95.377 224.155 90)
       (effects (font (size 1.27 1.27)) hide)
     )
-    (property "Datasheet" "~" (at 89.535 224.155 0)
+    (property "Datasheet" "~" (at 97.155 224.155 0)
       (effects (font (size 1.27 1.27)) hide)
     )
@@
     )
   )
-  (symbol (lib_id "Device:R") (at 104.775 224.155 180) (unit 1)
+  (symbol (lib_id "Device:R") (at 81.915 224.155 0) (mirror x) (unit 1)
     (in_bom yes) (on_board yes) (dnp no) (fields_autoplaced)
-    (property "Reference" "R22" (at 107.315 222.885 0)
+    (property "Reference" "R22" (at 79.375 222.885 0)
       (effects (font (size 1.27 1.27)) (justify right))
     )
-    (property "Value" "10K" (at 107.315 225.425 0)
+    (property "Value" "10K" (at 79.375 225.425 0)
       (effects (font (size 1.27 1.27)) (justify right))
     )
-    (property "Footprint" "Resistor_SMD:R_0402_1005Metric" (at 106.553 224.155 90)
+    (property "Footprint" "Resistor_SMD:R_0402_1005Metric" (at 80.137 224.155 90)
       (effects (font (size 1.27 1.27)) hide)
     )
-    (property "Datasheet" "~" (at 104.775 224.155 0)
+    (property "Datasheet" "~" (at 81.915 224.155 0)
       (effects (font (size 1.27 1.27)) hide)
     )
@@
     )
   )
-  (symbol (lib_id "Device:R") (at 81.915 224.155 180) (unit 1)
+  (symbol (lib_id "Device:R") (at 104.775 224.155 0) (mirror x) (unit 1)
     (in_bom yes) (on_board yes) (dnp no) (fields_autoplaced)
-    (property "Reference" "R19" (at 84.455 222.885 0)
+    (property "Reference" "R19" (at 102.235 222.885 0)
       (effects (font (size 1.27 1.27)) (justify right))
     )
-    (property "Value" "10K" (at 84.455 225.425 0)
+    (property "Value" "10K" (at 102.235 225.425 0)
       (effects (font (size 1.27 1.27)) (justify right))
     )
-    (property "Footprint" "Resistor_SMD:R_0402_1005Metric" (at 83.693 224.155 90)
+    (property "Footprint" "Resistor_SMD:R_0402_1005Metric" (at 102.997 224.155 90)
       (effects (font (size 1.27 1.27)) hide)
     )
-    (property "Datasheet" "~" (at 81.915 224.155 0)
+    (property "Datasheet" "~" (at 104.775 224.155 0)
       (effects (font (size 1.27 1.27)) hide)
     )
@@
     )
   )
-  (symbol (lib_id "Device:R") (at 97.155 224.155 180) (unit 1)
+  (symbol (lib_id "Device:R") (at 89.535 224.155 0) (mirror x) (unit 1)
     (in_bom yes) (on_board yes) (dnp no) (fields_autoplaced)
-    (property "Reference" "R21" (at 99.695 222.885 0)
+    (property "Reference" "R21" (at 86.995 222.885 0)
       (effects (font (size 1.27 1.27)) (justify right))
     )
-    (property "Value" "10K" (at 99.695 225.425 0)
+    (property "Value" "10K" (at 86.995 225.425 0)
       (effects (font (size 1.27 1.27)) (justify right))
     )
-    (property "Footprint" "Resistor_SMD:R_0402_1005Metric" (at 98.933 224.155 90)
+    (property "Footprint" "Resistor_SMD:R_0402_1005Metric" (at 87.757 224.155 90)
       (effects (font (size 1.27 1.27)) hide)
     )
-    (property "Datasheet" "~" (at 97.155 224.155 0)
+    (property "Datasheet" "~" (at 89.535 224.155 0)
       (effects (font (size 1.27 1.27)) hide)
     )
@@
     )
   )
-  (symbol (lib_id "Switch:SW_DIP_x06") (at 87.63 205.105 0) (unit 1)
+  (symbol (lib_id "Switch:SW_DIP_x06") (at 87.63 202.565 0) (mirror x) (unit 1)
     (in_bom yes) (on_board yes) (dnp no)
-    (property "Reference" "SW2" (at 87.63 213.995 0)
+    (property "Reference" "SW2" (at 87.63 193.675 0)
       (effects (font (size 1.27 1.27)))
     )
-    (property "Value" "SW_DIP_x06" (at 87.63 216.535 0)
+    (property "Value" "SW_DIP_x06" (at 87.63 191.135 0)
       (effects (font (size 1.27 1.27)))
     )
-    (property "Footprint" "SamacSys_Parts3:2195MSTR" (at 85.725 190.5 0)
+    (property "Footprint" "SamacSys_Parts3:2196LPST" (at 85.725 217.17 0)
       (effects (font (size 1.27 1.27)) hide)
     )
-    (property "Datasheet" "~" (at 87.63 205.105 0)
+    (property "Datasheet" "~" (at 87.63 202.565 0)
       (effects (font (size 1.27 1.27)) hide)
     )
@@
     )
   )
-  (symbol (lib_id "Device:R") (at 74.295 224.155 180) (unit 1)
+  (symbol (lib_id "Device:R") (at 112.395 224.155 0) (mirror x) (unit 1)
     (in_bom yes) (on_board yes) (dnp no) (fields_autoplaced)
-    (property "Reference" "R18" (at 76.835 222.885 0)
+    (property "Reference" "R18" (at 109.855 222.885 0)
       (effects (font (size 1.27 1.27)) (justify right))
     )
-    (property "Value" "10K" (at 76.835 225.425 0)
+    (property "Value" "10K" (at 109.855 225.425 0)
       (effects (font (size 1.27 1.27)) (justify right))
     )
-    (property "Footprint" "Resistor_SMD:R_0402_1005Metric" (at 76.073 224.155 90)
+    (property "Footprint" "Resistor_SMD:R_0402_1005Metric" (at 110.617 224.155 90)
       (effects (font (size 1.27 1.27)) hide)
     )
-    (property "Datasheet" "~" (at 74.295 224.155 0)
+    (property "Datasheet" "~" (at 112.395 224.155 0)
       (effects (font (size 1.27 1.27)) hide)
     )
@@
     )
   )
-  (symbol (lib_id "Device:R") (at 112.395 224.155 180) (unit 1)
+  (symbol (lib_id "Device:R") (at 74.295 224.155 0) (mirror x) (unit 1)
     (in_bom yes) (on_board yes) (dnp no)
-    (property "Reference" "R23" (at 114.935 222.885 0)
+    (property "Reference" "R23" (at 71.755 222.885 0)
       (effects (font (size 1.27 1.27)) (justify right))
     )
-    (property "Value" "10K" (at 114.935 225.425 0)
+    (property "Value" "10K" (at 71.755 225.425 0)
       (effects (font (size 1.27 1.27)) (justify right))
     )
-    (property "Footprint" "Resistor_SMD:R_0402_1005Metric" (at 114.173 224.155 90)
+    (property "Footprint" "Resistor_SMD:R_0402_1005Metric" (at 72.517 224.155 90)
       (effects (font (size 1.27 1.27)) hide)
     )
-    (property "Datasheet" "~" (at 112.395 224.155 0)
+    (property "Datasheet" "~" (at 74.295 224.155 0)
       (effects (font (size 1.27 1.27)) hide)
     )

Commit message: test
Parts:
- removed J5: USB, Connector_PinHeader_2.54mm:PinHeader_1x03_P2.54mm_Vertical, symbol Connector_Generic:Conn_01x03
- added C19, C20: 10uf, Capacitor_SMD:C_0805_2012Metric, symbol Device:C
- added IC5: NCP1117IDT33T4G, NCP1117IDT33T4G, symbol SamacSys_Parts2:NCP1117IDT33T4G
- added J4: 10118192-0002LF, 101181920002LF, symbol SamacSys_Parts2:10118192-0002LF
- added USB_Power: Jumper_2_Open, Jumper:SolderJumper-2_P1.3mm_Open_RoundedPad1.0x1.5mm, symbol Jumper:Jumper_2_Open
Connections:
- net GPIO11 is gone; now on net Vibration: U1.14 (GPIO11)
- net GPIO16 is gone; now on net LoRa_TXD: U1.27 (GPIO16)
- net GPIO17 is gone; now on net LoRa_RXD: U1.28 (GPIO17)
- net GPIO18 is gone; now on net LoRa_RES: U1.29 (GPIO18)
- net GPIO19 is gone; now on net LoRa_BOO: U1.30 (GPIO19)
- net +3.3V: now also C20.1, IC5.3 (INPUT)
- net AIR_INT: now also U1.6 (GPIO4); no longer U1.7 (GPIO5)
- net AIR_RES: now also U1.5 (GPIO3); no longer U1.8 (GPIO6)
- net D+: now also R3.1, J4.3
- net D-: now also R4.1, J4.2
- net Digital_in: now also U1.4 (GPIO2); no longer U1.12 (GPIO9)
- net GND: now also C19.2, C20.2, IC5.1 (ADJUST/GROUND), J4.5
- net LoRa_BOO: no longer U1.11 (GPIO8)
- net LoRa_RES: no longer U1.9 (GPIO7)
- net LoRa_RXD: no longer U1.3 (GPIO1)
- net LoRa_TXD: no longer U1.2 (GPIO0)
- net PIR: now also U1.13 (GPIO10); no longer U1.6 (GPIO4)
- net SCL: now also U1.9 (GPIO7); no longer U1.5 (GPIO3)
- net SCL0: now also U1.3 (GPIO1); no longer U1.16 (GPIO13)
- net SDA: now also U1.8 (GPIO6); no longer U1.4 (GPIO2)
- net SDA0: now also U1.2 (GPIO0); no longer U1.15 (GPIO12)
- net Vibration: no longer U1.13 (GPIO10)
- net GPIO25: no longer names the net of U1.37 (GPIO25)
- new net: J4.1, USB_Power.1 (A)
- new net: C19.1, IC5.2 (OUTPUT), USB_Power.2 (B)
- no-connect marks 4 -> 11
Other:
- moved on the sheet: R32, R33

Commit message: TJEK
Parts:
- added H1, H2, H3: MountingHole, MountingHole:MountingHole_3.2mm_M3, symbol Mechanical:MountingHole
- renumbered C11 to C10, C12 to C11, C13 to C12, C14 to C13, C2 to C14, C3 to C16, C4 to C17, C22 to C18, C19 to C2, C20 to C3, C5 to C4, C6 to C5, C7 to C6, C8 to C7, C9 to C8, C10 to C9, IC5 to IC1, IC3 to IC2, IC1 to IC3, J6 to J1, J4 to J2, J1 to J3, J8 to J4, J7 to J5, R29 to R10, R28 to R11, R31 to R12, R23 to R13, R22 to R14, R21 to R15, R20 to R16, R19 to R17, R26 to R19, R3 to R2, R27 to R20, R5 to R21, R6 to R22, R7 to R23, R8 to R24, R9 to R25, R10 to R26, R11 to R27, R12 to R28, R24 to R29, R4 to R3, R25 to R30, R32 to R4, R33 to R5, R13 to R6, R14 to R7, R2 to R8, R30 to R9, SW2 to SW1, SW1 to SW2, U2 to U3, USB_Power to USB_Power1, Y3 to Y1
Other:
- moved on the sheet: C2, C3, IC1, J2, R13, R14, R15, R16, R17, R18, USB_Power1

Commit message: tjek
Parts:
- added AE1: Antenna, SELF_MADE:Event_alarm_antenna, symbol Device:Antenna
- added Antenna1: Antenne, TestPoint:TestPoint_Pad_D2.5mm, symbol Connector:TestPoint
- added C19: 4,7uf, Capacitor_SMD:C_0402_1005Metric, symbol Device:C
- added C20, C21: NC, Capacitor_SMD:C_0402_1005Metric, symbol Device:C
- added C22: 100nf, Capacitor_SMD:C_0402_1005Metric, symbol Device:C
- added C23, C24, C25, C26: 10uf, Capacitor_SMD:C_0805_2012Metric, symbol Device:C
- added D1: LED, symbol Device:LED
- added IC1: LoRa-E5, LoRaE5, symbol SamacSys_Parts:LoRa-E5
- added J6: 2337019-1, 23370191, symbol SamacSys_Parts:2337019-1
- added J7: FAN, symbol Connector_Generic:Conn_01x02
- added L1: 0Ω, Resistor_SMD:R_0402_1005Metric, symbol Device:L
- added Q1: 2N2219, Package_TO_SOT_THT:TO-39-3, symbol Transistor_BJT:2N2219
- added R31, R32: 10KΩ, Resistor_SMD:R_0402_1005Metric, symbol Device:R
- added R33, R34: 100Ω, Resistor_SMD:R_0402_1005Metric, symbol Device:R
- C1, C10, C11, C12, C13, C14, C15, C4, C5, C8, C9: JLCPCB (none) -> C1525
- C16, C17: JLCPCB (none) -> C1557
- C18, C6, C7: JLCPCB (none) -> C1592
- C2, C3: JLCPCB C2972784 -> C15850
- IC1: JLCPCB (none) -> C2902115
- IC2: JLCPCB (none) -> C5342493
- IC4: JLCPCB (none) -> C579262
- R1, R10, R11, R12, R13, R14, R15, R16, R17, R18, R19, R20, R21, R22, R23, R24, R25, R26, R27, R28, R29, R30, R4, R5, R7, R9: value 10K -> 10KΩ; JLCPCB (none) -> C25744
- R2, R3: value 27 -> 27Ω; JLCPCB (none) -> C25100
- R8: value 1K -> 1KΩ; JLCPCB (none) -> C11702
- SW1: JLCPCB (none) -> C2842671
- Y1: JLCPCB (none) -> C9002
Connections:
- net +3.3V: now also C19.1, C22.1, C23.1, C24.1, C25.1, C26.1, IC1.1 (VCC), Q1.3 (C), R31.2, R32.2
- net D+: no longer R2.2, U1.47 (USB_DP)
- net D-: no longer R3.2, U1.46 (USB_DM)
- net GND: now also C19.2, C20.2, C21.2, C22.2, C23.2, C24.2, C25.2, C26.2, IC1.14 (GND_2), IC1.16 (GND_3), IC1.2 (GND_1), IC1.22 (GND_4), J6.2 (GND), J6.3 (GND_2), J7.2 (Pin_2), R33.2
- net LoRa_RXD: now also IC1.10 (PB6)
- net LoRa_TXD: now also IC1.9 (PB7)
- net SCL0: now also R32.1
- net SDA0: now also R31.1
- net GPIO14: no longer names the net of U1.17 (GPIO14)
- net GPIO14: now also D1.2 (A)
- net GPIO15: no longer names the net of U1.18 (GPIO15)
- net GPIO15: now also R34.2
- net LoRa_BOO renamed LoRa_Boot
- net LoRa_Boot: now also IC1.24 (PB13)
- net LoRa_RES renamed LoRa_Reset
- net LoRa_Reset: now also IC1.17 (RST)
- new net: AE1.1 (A), Antenna1.1, C21.1, J6.1 (SIGNAL), L1.2
- new net: C20.1, IC1.15 (RFIO), L1.1
- new net: J7.1 (Pin_1), Q1.1 (E)
- new net: Q1.2 (B), R34.1
- new net: D1.1 (K), R33.1
- new net: R3.2, U1.46 (USB_DM)
- new net: R2.2, U1.47 (USB_DP)
- new net PA0: IC1.23 (PA0)
- no-connect marks 11 -> 28
Other:
- moved on the sheet: C10, C11, C12, C13, C16, C17, C18, C4, C5, C6, C7, C8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
