File: Wireless modbus/Wireless slave/wireless_Slave/RPI2040_main_sch.kicad_sch (KiCad schematic)
At the start: 89 parts, among them IC1 LoRa-E5, IC1 NCP1117IDT33T4G, IC2 ZMOD4410AI1R, IC3 SHT30-DIS-B10KS, IC4 ADP5587ACPZ-R7, J1 ON/OFF, J2 10118192-0002LF, J3 Conn_01x02, J4 I2C, J5 Digital_in, J6 2337019-1, J7 FAN, Q1 2N2219, SW1 SW_DIP_x06, SW2 SW_DIP_x12, U1 EKMB1107111, U1 RP2040, U3 W25Q128JVS, Y1 12MHz

Commit message: håhå
Parts:
- C1, C10, C11, C12, C13, C14, C15, C22, C4, C5, C8, C9: JLC (none) -> C1525
- C16, C17: JLC (none) -> C1557
- C18, C6, C7: JLC (none) -> C1592
- C19: JLC (none) -> C368809
- C2, C23, C24, C25, C26, C3: JLC (none) -> C15850
- IC1: JLCPCB C5334317 -> (none)
- IC1: JLCPCB C2902115 -> (none)
- IC2: JLC (none) -> C5342493
- IC3: JLC (none) -> C2687423
- IC4: JLC (none) -> C579262
- J6: JLC (none) -> C434807
- L1: JLC (none) -> C881335
- R1, R10, R11, R12, R13, R14, R15, R16, R17, R18, R19, R20, R21, R22, R23, R24, R25, R26, R27, R28, R29, R30, R31, R32, R4, R5, R7, R9: JLC (none) -> C25744
- R2, R3: JLC (none) -> C25100
- R8: JLC (none) -> C11702
- SW1: JLC (none) -> C2842671
- U1: JLC (none) -> C2040
- U3: JLC (none) -> C97521
- Y1: JLC (none) -> C9002
Other:
- moved on the sheet: R13, R14, R15, R16, R17, R18

Commit message: siejwi
Parts:
- D1: footprint (none) -> LED_SMD:LED_0805_2012Metric; JLC (none) -> C598370
- J7: footprint (none) -> Connector_PinHeader_2.54mm:PinHeader_1x02_P2.54mm_Vertical
- Q1: value 2N2219 -> BCX56; footprint Package_TO_SOT_THT:TO-39-3 -> Package_TO_SOT_SMD:SOT-89-3; JLC (none) -> C5345980
- R33: value 100Ω -> 70Ω; JLC (none) -> C25133; JLCPCB C25744 -> C25133
- R34: value 100Ω -> 2.4KΩ; footprint Resistor_SMD:R_0402_1005Metric -> Resistor_SMD:R_0603_1608Metric; JLC (none) -> C22940; JLCPCB C25744 -> C22940
Connections:
- net GPIO20 is gone; now on an unnamed net: U1.31 (GPIO20)
- net +3.3V: now also Q1.2 (C); no longer Q1.3 (C)
- net at Q1.1 (B): now also R34.1; no longer J7.1 (Pin_1)
- net at R34.2: no longer U1.18 (GPIO15)
- new net: J7.1 (Pin_1), Q1.3 (E)
Changed lines of the file:
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@@
     (stroke (width 0) (type default))
   )
-  (wire (pts (xy 249.555 83.185) (xy 249.555 92.71))
-    (stroke (width 0) (type default))
-  )
   (wire (pts (xy 349.885 70.485) (xy 354.965 70.485))
     (stroke (width 0) (type default))
@@
     (stroke (width 0) (type default))
   )
-  (wire (pts (xy 226.695 83.185) (xy 249.555 83.185))
-    (stroke (width 0) (type default))
-  )
   (wire (pts (xy 103.505 180.34) (xy 110.49 180.34))
     (stroke (width 0) (type default))
@@
     (stroke (width 0) (type default))
   )
+  (wire (pts (xy 249.555 95.885) (xy 249.555 92.71))
+    (stroke (width 0) (type default))
+  )
   (wire (pts (xy 264.795 62.865) (xy 264.795 44.45))
     (stroke (width 0) (type default))
@@
     (stroke (width 0) (type default))
   )
-  (wire (pts (xy 226.695 95.885) (xy 234.315 95.885))
+  (wire (pts (xy 226.695 95.885) (xy 249.555 95.885))
     (stroke (width 0) (type default))
   )
@@
     (effects (font (size 1.27 1.27)) (justify left bottom))
   )
-  (label "GPIO20" (at 234.315 95.885 180) (fields_autoplaced)
-    (effects (font (size 1.27 1.27)) (justify right bottom))
-  )
   (label "R3" (at 38.1 207.645 0) (fields_autoplaced)
     (effects (font (size 1.27 1.27)) (justify left bottom))
@@
       (effects (font (size 1.27 1.27)) (justify left))
     )
-    (property "Value" "2N2219" (at 267.97 93.98 0)
+    (property "Value" "BCX56" (at 267.97 93.98 0)
       (effects (font (size 1.27 1.27)) (justify left))
     )
-    (property "Footprint" "Package_TO_SOT_THT:TO-39-3" (at 267.335 94.615 0)
+    (property "Footprint" "Package_TO_SOT_SMD:SOT-89-3" (at 267.335 94.615 0)
       (effects (font (size 1.27 1.27) italic) (justify left) hide)
     )
-    (property "Datasheet" "http://www.onsemi.com/pub_link/Collateral/2N2219-D.PDF" (at 262.255 92.71 0)
+    (property "Datasheet" "" (at 262.255 92.71 0)
       (effects (font (size 1.27 1.27)) (justify left) hide)
     )
+    (property "JLC" "C5345980" (at 256.54 88.265 0)
+      (effects (font (size 1.27 1.27)) hide)
+    )
     (pin "1")
     (pin "2")
@@
       (effects (font (size 1.27 1.27)) (justify right))
     )
-    (property "Footprint" "" (at 245.11 80.645 0)
+    (property "Footprint" "LED_SMD:LED_0805_2012Metric" (at 245.11 80.645 0)
       (effects (font (size 1.27 1.27)) hide)
     )
@@
       (effects (font (size 1.27 1.27)) hide)
     )
+    (property "JLC" "C598370" (at 245.11 80.645 0)
+      (effects (font (size 1.27 1.27)) hide)
+    )
     (pin "1")
     (pin "2")
@@
       (effects (font (size 1.27 1.27)) (justify left))
     )
-    (property "Footprint" "" (at 269.875 97.79 0)
+    (property "Footprint" "Connector_PinHeader_2.54mm:PinHeader_1x02_P2.54mm_Vertical" (at 269.875 97.79 0)
       (effects (font (size 1.27 1.27)) hide)
     )
@@
       (effects (font (size 1.27 1.27)) (justify right))
     )
-    (property "Value" "100Ω" (at 251.46 78.74 0)
+    (property "Value" "70Ω" (at 251.46 78.74 0)
       (effects (font (size 1.27 1.27)) (justify right))
     )
@@
       (effects (font (size 1.27 1.27)) hide)
     )
-    (property "JLCPCB" "C25744" (at 252.73 80.645 0)
+    (property "JLCPCB" "C25133" (at 252.73 80.645 0)
+      (effects (font (size 1.27 1.27)) hide)
+    )
+    (property "JLC" "C25133" (at 252.73 80.645 0)
       (effects (font (size 1.27 1.27)) hide)
     )
@@
       (effects (font (size 1.27 1.27)) (justify right))
     )
-    (property "Value" "100Ω" (at 254.635 94.615 0)
+    (property "Value" "2.4KΩ" (at 254.635 94.615 0)
       (effects (font (size 1.27 1.27)) (justify right))
     )
-    (property "Footprint" "Resistor_SMD:R_0402_1005Metric" (at 253.365 94.488 90)
+    (property "Footprint" "Resistor_SMD:R_0603_1608Metric" (at 253.365 94.488 90)
       (effects (font (size 1.27 1.27)) hide)
     )
@@
       (effects (font (size 1.27 1.27)) hide)
     )
-    (property "JLCPCB" "C25744" (at 253.365 92.71 0)
+    (property "JLCPCB" "C22940" (at 253.365 92.71 0)
+      (effects (font (size 1.27 1.27)) hide)
+    )
+    (property "JLC" "C22940" (at 253.365 92.71 0)
       (effects (font (size 1.27 1.27)) hide)
     )

Commit message: km
Other:
- note added: "Konfiguration bits"
- note added: "LoRa"
- note added: "RP2040"
- note removed: "Adressering, Delta, interval, pause"
- moved on the sheet: AE1, Antenna1, BT1, C1, C10, C11, C12, C13, C14, C15, C16, C17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
