File: Wireless modbus/Wireless slave/wireless_Slave/dB_sensor.kicad_sch (KiCad schematic)
At the start: 8 parts

Commit message: wup wup
Parts:
- renumbered C19 to C18, C18 to C19, R14 to R16, R16 to R17

Commit message: wup
Parts:
- C19: renamed from C18; footprint (none) -> Capacitor_SMD:C_0603_1608Metric
- C20: renamed from C19; value 10p -> 10pf; footprint (none) -> Capacitor_SMD:C_0402_1005Metric
- C21: renamed from C20; footprint (none) -> Capacitor_SMD:C_0603_1608Metric
- MK1: footprint (none) -> SamacSys_Parts:CMA4544PFW
- R15, R17: value 10k -> 10K; footprint (none) -> Resistor_SMD:R_0402_1005Metric
- R16: footprint (none) -> Resistor_SMD:R_0402_1005Metric
- RV1: value 1k -> 1K

Commit message: jaaaaaaaaaaaaa
Parts:
- renumbered C19 to #C19, C20 to #C20, C21 to #C21, MK1 to #MK1, R15 to #R15, R16 to #R16, R17 to #R17, RV1 to #RV1
Changed lines of the file:
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@@
   (symbol (lib_id "Device:C_Polarized") (at 160.02 41.275 0) (mirror x) (unit 1)
     (in_bom yes) (on_board yes) (dnp no)
-    (property "Reference" "C21" (at 156.845 41.529 0)
+    (property "Reference" "#C21" (at 156.845 41.529 0)
       (effects (font (size 1.27 1.27)) (justify right))
     )
@@
       (project "wireless_Slave"
         (path "/0e0a1f86-1a9d-413b-96af-bc4dca868b1d/6fc288ee-49ba-4f78-a527-a360a72ed5fc"
-          (reference "C21") (unit 1)
+          (reference "#C21") (unit 1)
         )
       )
@@
   (symbol (lib_id "Device:R") (at 152.4 48.895 270) (unit 1)
     (in_bom yes) (on_board yes) (dnp no)
-    (property "Reference" "R17" (at 152.4 53.975 90)
+    (property "Reference" "#R17" (at 152.4 53.975 90)
       (effects (font (size 1.27 1.27)))
     )
@@
       (project "wireless_Slave"
         (path "/0e0a1f86-1a9d-413b-96af-bc4dca868b1d/6fc288ee-49ba-4f78-a527-a360a72ed5fc"
-          (reference "R17") (unit 1)
+          (reference "#R17") (unit 1)
         )
       )
@@
   (symbol (lib_id "Device:C") (at 118.745 53.975 0) (unit 1)
     (in_bom yes) (on_board yes) (dnp no) (fields_autoplaced)
-    (property "Reference" "C20" (at 121.92 53.34 0)
-      (effects (font (size 1.27 1.27)) (justify left))
-    )
-    (property "Value" "10pf" (at 121.92 55.88 0)
-      (effects (font (size 1.27 1.27)) (justify left))
+    (property "Reference" "#C20" (at 115.57 52.705 0)
+      (effects (font (size 1.27 1.27)) (justify right))
+    )
+    (property "Value" "10pf" (at 115.57 55.245 0)
+      (effects (font (size 1.27 1.27)) (justify right))
     )
     (property "Footprint" "Capacitor_SMD:C_0402_1005Metric" (at 119.7102 57.785 0)
@@
       (project "wireless_Slave"
         (path "/0e0a1f86-1a9d-413b-96af-bc4dca868b1d/6fc288ee-49ba-4f78-a527-a360a72ed5fc"
-          (reference "C20") (unit 1)
+          (reference "#C20") (unit 1)
         )
       )
@@
   (symbol (lib_id "Device:R_Potentiometer") (at 160.02 48.895 180) (unit 1)
     (in_bom yes) (on_board yes) (dnp no) (fields_autoplaced)
-    (property "Reference" "RV1" (at 161.925 48.26 0)
-      (effects (font (size 1.27 1.27)) (justify right))
-    )
-    (property "Value" "1K" (at 161.925 50.8 0)
+    (property "Reference" "#RV1" (at 162.56 47.625 0)
+      (effects (font (size 1.27 1.27)) (justify right))
+    )
+    (property "Value" "1K" (at 162.56 50.165 0)
       (effects (font (size 1.27 1.27)) (justify right))
     )
@@
       (project "wireless_Slave"
         (path "/0e0a1f86-1a9d-413b-96af-bc4dca868b1d/6fc288ee-49ba-4f78-a527-a360a72ed5fc"
-          (reference "RV1") (unit 1)
+          (reference "#RV1") (unit 1)
         )
       )
@@
   (symbol (lib_id "Device:R") (at 92.075 43.815 0) (unit 1)
     (in_bom yes) (on_board yes) (dnp no) (fields_autoplaced)
-    (property "Reference" "R15" (at 93.98 43.18 0)
-      (effects (font (size 1.27 1.27)) (justify left))
-    )
-    (property "Value" "10K" (at 93.98 45.72 0)
-      (effects (font (size 1.27 1.27)) (justify left))
+    (property "Reference" "#R15" (at 90.17 42.545 0)
+      (effects (font (size 1.27 1.27)) (justify right))
+    )
+    (property "Value" "10K" (at 90.17 45.085 0)
+      (effects (font (size 1.27 1.27)) (justify right))
     )
     (property "Footprint" "Resistor_SMD:R_0402_1005Metric" (at 90.297 43.815 90)
@@
       (project "wireless_Slave"
         (path "/0e0a1f86-1a9d-413b-96af-bc4dca868b1d/6fc288ee-49ba-4f78-a527-a360a72ed5fc"
-          (reference "R15") (unit 1)
+          (reference "#R15") (unit 1)
         )
       )
@@
   (symbol (lib_id "Device:R") (at 113.03 50.165 90) (unit 1)
     (in_bom yes) (on_board yes) (dnp no) (fields_autoplaced)
-    (property "Reference" "R16" (at 113.03 45.085 90)
-      (effects (font (size 1.27 1.27)))
-    )
-    (property "Value" "680" (at 113.03 47.625 90)
+    (property "Reference" "#R16" (at 113.03 44.45 90)
+      (effects (font (size 1.27 1.27)))
+    )
+    (property "Value" "680" (at 113.03 46.99 90)
       (effects (font (size 1.27 1.27)))
     )
@@
       (project "wireless_Slave"
         (path "/0e0a1f86-1a9d-413b-96af-bc4dca868b1d/6fc288ee-49ba-4f78-a527-a360a72ed5fc"
-          (reference "R16") (unit 1)
+          (reference "#R16") (unit 1)
         )
       )
@@
   (symbol (lib_id "Device:C_Polarized") (at 106.045 43.815 0) (mirror x) (unit 1)
     (in_bom yes) (on_board yes) (dnp no)
-    (property "Reference" "C19" (at 102.87 44.069 0)
+    (property "Reference" "#C19" (at 102.87 44.069 0)
       (effects (font (size 1.27 1.27)) (justify right))
     )
@@
       (project "wireless_Slave"
         (path "/0e0a1f86-1a9d-413b-96af-bc4dca868b1d/6fc288ee-49ba-4f78-a527-a360a72ed5fc"
-          (reference "C19") (unit 1)
+          (reference "#C19") (unit 1)
         )
       )
@@
   (symbol (lib_id "Device:Microphone") (at 106.045 57.785 0) (mirror y) (unit 1)
     (in_bom yes) (on_board yes) (dnp no)
-    (property "Reference" "MK1" (at 101.6 56.4515 0)
+    (property "Reference" "#MK1" (at 101.6 56.4515 0)
       (effects (font (size 1.27 1.27)) (justify left))
     )
@@
       (project "wireless_Slave"
         (path "/0e0a1f86-1a9d-413b-96af-bc4dca868b1d/6fc288ee-49ba-4f78-a527-a360a72ed5fc"
-          (reference "MK1") (unit 1)
-        )
-      )
+          (reference "#MK1") (unit 1)
+        )
+      )

Commit message: TJEK
Parts:
- renumbered #C21 to #C1, #C19 to #C2, #C20 to #C3, #R15 to #R1, #R17 to #R2, #R16 to #R3
Changed lines of the file:
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@@
   (symbol (lib_id "power:GND") (at 92.075 47.625 0) (unit 1)
     (in_bom yes) (on_board yes) (dnp no) (fields_autoplaced)
-    (property "Reference" "#PWR031" (at 92.075 53.975 0)
+    (property "Reference" "#PWR059" (at 92.075 53.975 0)
       (effects (font (size 1.27 1.27)) hide)
     )
@@
       (project "wireless_Slave"
         (path "/0e0a1f86-1a9d-413b-96af-bc4dca868b1d/6fc288ee-49ba-4f78-a527-a360a72ed5fc"
-          (reference "#PWR031") (unit 1)
+          (reference "#PWR059") (unit 1)
         )
       )
@@
   (symbol (lib_id "Device:C_Polarized") (at 160.02 41.275 0) (mirror x) (unit 1)
     (in_bom yes) (on_board yes) (dnp no)
-    (property "Reference" "#C21" (at 156.845 41.529 0)
+    (property "Reference" "#C1" (at 156.845 41.529 0)
       (effects (font (size 1.27 1.27)) (justify right))
     )
@@
       (project "wireless_Slave"
         (path "/0e0a1f86-1a9d-413b-96af-bc4dca868b1d/6fc288ee-49ba-4f78-a527-a360a72ed5fc"
-          (reference "#C21") (unit 1)
+          (reference "#C1") (unit 1)
         )
       )
@@
   (symbol (lib_id "Device:R") (at 152.4 48.895 270) (unit 1)
     (in_bom yes) (on_board yes) (dnp no)
-    (property "Reference" "#R17" (at 152.4 53.975 90)
+    (property "Reference" "#R2" (at 152.4 53.975 90)
       (effects (font (size 1.27 1.27)))
     )
@@
       (project "wireless_Slave"
         (path "/0e0a1f86-1a9d-413b-96af-bc4dca868b1d/6fc288ee-49ba-4f78-a527-a360a72ed5fc"
-          (reference "#R17") (unit 1)
+          (reference "#R2") (unit 1)
         )
       )
@@
   (symbol (lib_id "power:GND") (at 106.045 62.865 0) (unit 1)
     (in_bom yes) (on_board yes) (dnp no) (fields_autoplaced)
-    (property "Reference" "#PWR032" (at 106.045 69.215 0)
+    (property "Reference" "#PWR062" (at 106.045 69.215 0)
       (effects (font (size 1.27 1.27)) hide)
     )
@@
       (project "wireless_Slave"
         (path "/0e0a1f86-1a9d-413b-96af-bc4dca868b1d/6fc288ee-49ba-4f78-a527-a360a72ed5fc"
-          (reference "#PWR032") (unit 1)
+          (reference "#PWR062") (unit 1)
         )
       )
@@
   (symbol (lib_id "Device:C") (at 118.745 53.975 0) (unit 1)
     (in_bom yes) (on_board yes) (dnp no) (fields_autoplaced)
-    (property "Reference" "#C20" (at 115.57 52.705 0)
+    (property "Reference" "#C3" (at 115.57 52.705 0)
       (effects (font (size 1.27 1.27)) (justify right))
     )
@@
       (project "wireless_Slave"
         (path "/0e0a1f86-1a9d-413b-96af-bc4dca868b1d/6fc288ee-49ba-4f78-a527-a360a72ed5fc"
-          (reference "#C20") (unit 1)
+          (reference "#C3") (unit 1)
         )
       )
@@
   (symbol (lib_id "power:GND") (at 118.745 57.785 0) (unit 1)
     (in_bom yes) (on_board yes) (dnp no) (fields_autoplaced)
-    (property "Reference" "#PWR033" (at 118.745 64.135 0)
+    (property "Reference" "#PWR061" (at 118.745 64.135 0)
       (effects (font (size 1.27 1.27)) hide)
     )
@@
       (project "wireless_Slave"
         (path "/0e0a1f86-1a9d-413b-96af-bc4dca868b1d/6fc288ee-49ba-4f78-a527-a360a72ed5fc"
-          (reference "#PWR033") (unit 1)
+          (reference "#PWR061") (unit 1)
         )
       )
@@
   (symbol (lib_id "power:GND") (at 160.02 52.705 0) (unit 1)
     (in_bom yes) (on_board yes) (dnp no) (fields_autoplaced)
-    (property "Reference" "#PWR035" (at 160.02 59.055 0)
+    (property "Reference" "#PWR060" (at 160.02 59.055 0)
       (effects (font (size 1.27 1.27)) hide)
     )
@@
       (project "wireless_Slave"
         (path "/0e0a1f86-1a9d-413b-96af-bc4dca868b1d/6fc288ee-49ba-4f78-a527-a360a72ed5fc"
-          (reference "#PWR035") (unit 1)
+          (reference "#PWR060") (unit 1)
         )
       )
@@
   (symbol (lib_id "Device:R") (at 92.075 43.815 0) (unit 1)
     (in_bom yes) (on_board yes) (dnp no) (fields_autoplaced)
-    (property "Reference" "#R15" (at 90.17 42.545 0)
+    (property "Reference" "#R1" (at 90.17 42.545 0)
       (effects (font (size 1.27 1.27)) (justify right))
     )
@@
       (project "wireless_Slave"
         (path "/0e0a1f86-1a9d-413b-96af-bc4dca868b1d/6fc288ee-49ba-4f78-a527-a360a72ed5fc"
-          (reference "#R15") (unit 1)
+          (reference "#R1") (unit 1)
         )
       )
@@
   (symbol (lib_id "Device:R") (at 113.03 50.165 90) (unit 1)
     (in_bom yes) (on_board yes) (dnp no) (fields_autoplaced)
-    (property "Reference" "#R16" (at 113.03 44.45 90)
+    (property "Reference" "#R3" (at 113.03 44.45 90)
       (effects (font (size 1.27 1.27)))
     )
@@
       (project "wireless_Slave"
         (path "/0e0a1f86-1a9d-413b-96af-bc4dca868b1d/6fc288ee-49ba-4f78-a527-a360a72ed5fc"
-          (reference "#R16") (unit 1)
+          (reference "#R3") (unit 1)
         )
       )
@@
   (symbol (lib_id "Device:C_Polarized") (at 106.045 43.815 0) (mirror x) (unit 1)
     (in_bom yes) (on_board yes) (dnp no)
-    (property "Reference" "#C19" (at 102.87 44.069 0)
+    (property "Reference" "#C2" (at 102.87 44.069 0)
       (effects (font (size 1.27 1.27)) (justify right))
     )
@@
       (project "wireless_Slave"
         (path "/0e0a1f86-1a9d-413b-96af-bc4dca868b1d/6fc288ee-49ba-4f78-a527-a360a72ed5fc"
-          (reference "#C19") (unit 1)
+          (reference "#C2") (unit 1)
         )
       )
@@
   (symbol (lib_id "power:GND") (at 160.02 37.465 180) (unit 1)
     (in_bom yes) (on_board yes) (dnp no) (fields_autoplaced)
-    (property "Reference" "#PWR034" (at 160.02 31.115 0)
+    (property "Reference" "#PWR058" (at 160.02 31.115 0)
       (effects (font (size 1.27 1.27)) hide)
     )
@@
       (project "wireless_Slave"
         (path "/0e0a1f86-1a9d-413b-96af-bc4dca868b1d/6fc288ee-49ba-4f78-a527-a360a72ed5fc"
-          (reference "#PWR034") (unit 1)
-        )
-      )
+          (reference "#PWR058") (unit 1)
+        )
+      )
