File: Wireless modbus/Wireless slave/wireless_Slave/wireless_Slave.kicad_pcb (KiCad board)
At the start: 2 copper layers, 9 parts, among them IC1 SHT30-DIS-B10KS, IC2 LoRa-E5, J3 2337019-1, U1 EKMB1107111, U2 W25Q128JVS, U3 RP2040

Commit message: wup
Parts:
- removed S1: 219-8MSTR, SamacSys_Parts1:2198MSTR
- added BT1: Battery_Cell, SamacSys_Parts3:BHAA-3, F.Cu at (158.1, 134.5)
- added C1: 100nf, Capacitor_SMD:C_0402_1005Metric, F.Cu at (162.7, 131.6)
- added C10: 100nf, Capacitor_SMD:C_0402_1005Metric, F.Cu at (160.2, 120.1)
- added C11: 100nf, Capacitor_SMD:C_0402_1005Metric, F.Cu at (160.3, 115.4)
- added C12: 100nf, Capacitor_SMD:C_0402_1005Metric, F.Cu at (167.0, 123.9)
- added C13: 100nf, Capacitor_SMD:C_0402_1005Metric, F.Cu at (164.6, 111.8)
- added C14: 100nf, Capacitor_SMD:C_0402_1005Metric, F.Cu at (172.2, 114.8)
- added C15: 100nf, Capacitor_SMD:C_0402_1005Metric, F.Cu at (159.0, 117.8)
- added C16: 4,7uf, Capacitor_SMD:C_0402_1005Metric, F.Cu at (166.7, 94.8)
- added C17: NC, Capacitor_SMD:C_0402_1005Metric, F.Cu at (184.2, 100.4)
- added C19: 1uf, Capacitor_SMD:C_0603_1608Metric, F.Cu at (157.2, 65.6)
- added C2: 100nf, Capacitor_SMD:C_0402_1005Metric, F.Cu at (156.1, 104.8)
- added C20: 10pf, Capacitor_SMD:C_0402_1005Metric, F.Cu at (156.6, 70.3)
- added C21: 2.2uf, Capacitor_SMD:C_0603_1608Metric, F.Cu at (157.2, 68.1)
- added C3: 27pf, Capacitor_SMD:C_0402_1005Metric, F.Cu at (163.6, 124.1)
- added C4: 27pf, Capacitor_SMD:C_0402_1005Metric, F.Cu at (165.5, 124.1)
- added C5: 100nf, Capacitor_SMD:C_0402_1005Metric, F.Cu at (163.6, 111.8)
- added C6: 100nf, Capacitor_SMD:C_0402_1005Metric, F.Cu at (168.0, 123.9)
- added C7: 1uf, Capacitor_SMD:C_0603_1608Metric, F.Cu at (168.7, 113.4)
- added C8: 1uf, Capacitor_SMD:C_0603_1608Metric, F.Cu at (171.0, 114.2)
- added C9: 100nf, Capacitor_SMD:C_0402_1005Metric, F.Cu at (171.1, 119.8)
- added IC3: ZMOD4410AI1R, SamacSys_Parts3:ZMOD4410AI1R, F.Cu at (169.7, 73.5)
- added J1: Conn_01x02, Connector_PinHeader_2.54mm:PinHeader_1x02_P2.54mm_Vertical, F.Cu at (152.7, 108.3)
- added J2: USB, Connector_PinHeader_2.54mm:PinHeader_1x02_P2.54mm_Vertical, F.Cu at (167.4, 109.0)
- added J4: Conn_02x09_Odd_Even, Connector_PinHeader_2.54mm:PinHeader_2x09_P2.54mm_Vertical, F.Cu at (144.1, 94.6)
- added MK1: Microphone, SamacSys_Parts:CMA4544PFW, F.Cu at (150.4, 63.5)
- added R1: 10K, Resistor_SMD:R_0402_1005Metric, F.Cu at (160.7, 131.6)
- added R10: 10K, Resistor_SMD:R_0402_1005Metric, F.Cu at (175.8, 121.5)
- added R11: 10K, Resistor_SMD:R_0402_1005Metric, F.Cu at (175.8, 124.7)
- added R12: 10K, Resistor_SMD:R_0402_1005Metric, F.Cu at (175.8, 126.6)
- added R13: R_Photo, SamacSys_Parts:02LDR1, F.Cu at (170.1, 143.3)
- added R14: 10K, Resistor_SMD:R_0402_1005Metric, F.Cu at (170.6, 137.5)
- added R15: 10K, Resistor_SMD:R_0402_1005Metric, F.Cu at (156.6, 59.3)
- added R16: 680, Resistor_SMD:R_0402_1005Metric, F.Cu at (156.6, 61.3)
- added R17: 10K, Resistor_SMD:R_0402_1005Metric, F.Cu at (156.6, 63.3)
- added R18: 10K, Resistor_SMD:R_0402_1005Metric, F.Cu at (230.7, 120.8)
- added R19: 10K, Resistor_SMD:R_0402_1005Metric, F.Cu at (230.7, 122.8)
- added R2: 1K, Resistor_SMD:R_0402_1005Metric, F.Cu at (155.6, 112.1)
- added R20: 10K, Resistor_SMD:R_0402_1005Metric, F.Cu at (230.7, 124.7)
- added R21: 10K, Resistor_SMD:R_0402_1005Metric, F.Cu at (230.7, 126.7)
- added R22: 10K, Resistor_SMD:R_0402_1005Metric, F.Cu at (230.7, 128.7)
- added R23: 10K, Resistor_SMD:R_0402_1005Metric, F.Cu at (230.7, 130.7)
- added R24: 10K, Resistor_SMD:R_0402_1005Metric, F.Cu at (230.7, 132.7)
- added R25: 10K, Resistor_SMD:R_0402_1005Metric, F.Cu at (230.7, 134.7)
- added R3: 27, Resistor_SMD:R_0402_1005Metric, F.Cu at (165.6, 111.8)
- added R4: 27, Resistor_SMD:R_0402_1005Metric, F.Cu at (166.7, 111.8)
- added R5: 10K, Resistor_SMD:R_0402_1005Metric, F.Cu at (175.8, 109.4)
- added R6: 10K, Resistor_SMD:R_0402_1005Metric, F.Cu at (175.8, 111.4)
- added R7: 10K, Resistor_SMD:R_0402_1005Metric, F.Cu at (175.8, 114.5)
- added R8: 10K, Resistor_SMD:R_0402_1005Metric, F.Cu at (175.8, 116.5)
- added R9: 10K, Resistor_SMD:R_0402_1005Metric, F.Cu at (175.8, 119.6)
- added SW1: SW_DIP_x12, SamacSys_Parts3:21912LPST, F.Cu at (229.5, 112.7)
- added SW2: SW_DIP_x06, SamacSys_Parts3:2195MSTR, F.Cu at (220.6, 126.8)
- added Y3: 12MHz, SamacSys_Parts2:X322512MSB4SI, F.Cu at (164.2, 127.7)
- IC1: footprint SamacSys_Parts1:SON50P250X250X100-9N-D -> SamacSys_Parts:SON50P250X250X100-9N-D
- IC2: footprint SamacSys_Parts1:LoRaE5 -> SamacSys_Parts:LoRaE5
- J3: footprint SamacSys_Parts1:23370191 -> SamacSys_Parts:23370191
- L1: footprint Capacitor_SMD:C_0402_1005Metric -> Resistor_SMD:R_0402_1005Metric
- U1: footprint SamacSys_Parts1:EKMB1107111 -> SamacSys_Parts:EKMB1107111
- moved U1 50.2 mm to (162.8, 138.7), turned to 90 degrees
- moved U3 26.5 mm to (165.0, 118.6)
- moved J3 24.7 mm to (187.8, 102.3), turned to -90 degrees
- moved IC1 23.9 mm to (156.7, 117.5)
- moved U2 22.0 mm to (159.5, 108.5), turned to 90 degrees
- moved C18 20.2 mm to (184.2, 104.2), turned to -90 degrees
- moved IC2 19.3 mm to (175.4, 98.0)
- moved L1 17.5 mm to (184.2, 102.3), turned to -90 degrees
- renumbered C17 to C18
Connections:
- net /RPI2040_main/GPIO2 renamed /RPI2040_main/SDA
- net /RPI2040_main/GPIO3 renamed /RPI2040_main/SCL
- net /RPI2040_main/GPIO4 renamed /RPI2040_main/PIR
- U3 pad 7: /RPI2040_main/GPIO5 -> /RPI2040_main/AIR_INT
- U3 pad 8: /RPI2040_main/GPIO6 -> /RPI2040_main/AIR_RES
Routing:
- net /LoRa/PB10: track 0.00 -> 40.8 mm, vias 0 -> 1
- net /LoRa/PA2: track 0.00 -> 38.3 mm, vias 0 -> 1
- net /RPI2040_main/GPIO17: track 0.00 -> 36.6 mm, vias 0 -> 2
- net /LoRa/PB5: track 0.00 -> 36.0 mm, vias 0 -> 1
- net /LoRa/PA3: track 0.00 -> 35.8 mm, vias 0 -> 1
- net /LoRa/PA9: track 0.00 -> 35.4 mm
- net /LoRa/PC1: track 0.00 -> 34.5 mm, vias 0 -> 1
- net /LoRa/PC0: track 0.00 -> 33.7 mm, vias 0 -> 1
- net /LoRa/PB3: track 0.00 -> 32.6 mm, vias 0 -> 1
- net /RPI2040_main/GPIO16: track 0.00 -> 30.2 mm, vias 0 -> 2
- net +3.3V: track 0.00 -> 28.7 mm
- net /LoRa/PA0: track 0.00 -> 27.4 mm
- net /LoRa/PB9: track 0.00 -> 21.6 mm
- net /LoRa/PB4: track 0.00 -> 18.2 mm
- net /LoRa/PB14: track 0.00 -> 17.5 mm
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- added copper zone on F.Cu, net +3.3V

Commit message: jaaaaaaaaaaaaa
Parts:
- removed C19: 1uf, Capacitor_SMD:C_0603_1608Metric
- removed C20: 10pf, Capacitor_SMD:C_0402_1005Metric
- removed C21: 2.2uf, Capacitor_SMD:C_0603_1608Metric
- removed J4: Conn_02x09_Odd_Even, Connector_PinHeader_2.54mm:PinHeader_2x09_P2.54mm_Vertical
- removed MK1: Microphone, SamacSys_Parts:CMA4544PFW
- removed R15, R17: 10K, Resistor_SMD:R_0402_1005Metric
- removed R16: 680, Resistor_SMD:R_0402_1005Metric
- added AE1: Antenna, SELF_MADE:Event_alarm_antenna, F.Cu at (262.7, 128.1)
- added C22: 1uf, Capacitor_SMD:C_0603_1608Metric, F.Cu at (255.4, 130.2)
- added IC4: ADP5587ACPZ-R7, SamacSys_Parts3:QFN50P400X400X80-25N-D, F.Cu at (251.2, 128.0)
- added J5: USB, Connector_PinHeader_2.54mm:PinHeader_1x03_P2.54mm_Vertical, B.Cu at (218.1, 99.9)
- added J6: ON/OFF, Connector_PinHeader_2.54mm:PinHeader_1x02_P2.54mm_Vertical, B.Cu at (237.7, 128.9)
- added J7: Digital_in, Connector_PinHeader_2.54mm:PinHeader_1x02_P2.54mm_Vertical, F.Cu at (218.9, 145.7)
- added J8: I2C, Connector_PinHeader_2.54mm:PinHeader_1x04_P2.54mm_Vertical, F.Cu at (212.3, 136.1)
- added R26: 10K, Resistor_SMD:R_0402_1005Metric, B.Cu at (263.3, 120.4)
- added R27: 10K, Resistor_SMD:R_0402_1005Metric, B.Cu at (260.8, 120.4)
- added R28: 10K, Resistor_SMD:R_0402_1005Metric, F.Cu at (254.8, 128.9)
- added R29: 10K, Resistor_SMD:R_0402_1005Metric, F.Cu at (254.8, 125.9)
- added R30: 10K, Resistor_SMD:R_0402_1005Metric, F.Cu at (215.9, 142.8)
- added R31: 10K, Resistor_SMD:R_0402_1005Metric, F.Cu at (253.3, 139.3)
- added R32: 10K, Resistor_SMD:R_0402_1005Metric, F.Cu at (228.4, 121.0)
- added R33: 10K, Resistor_SMD:R_0402_1005Metric, F.Cu at (228.4, 119.9)
- added S1: 4081, SamacSys_Parts3:4081, F.Cu at (265.8, 144.4)
- added TP1: Antenne, TestPoint:TestPoint_Pad_D2.5mm, B.Cu at (262.0, 128.1)
- BT1, J1, R10, R11, R12, R18, R19, R20, R21, R22, R23, R24, R25, R5, R6, R7, R8, R9, SW1: moved to B.Cu
- IC1: footprint SamacSys_Parts:SON50P250X250X100-9N-D -> SamacSys_Parts2:SON50P250X250X100-9N-D
- IC2: footprint SamacSys_Parts:LoRaE5 -> SamacSys_Parts2:LoRaE5
- J2: value USB -> Conn_01x18; footprint Connector_PinHeader_2.54mm:PinHeader_1x02_P2.54mm_Vertical -> Connector_PinHeader_2.54mm:PinHeader_1x18_P2.54mm_Vertical; moved to B.Cu
- J3: footprint SamacSys_Parts:23370191 -> SamacSys_Parts2:23370191; moved to B.Cu
- SW2: footprint SamacSys_Parts3:2195MSTR -> SamacSys_Parts3:2196LPST; moved to B.Cu
- U1: footprint SamacSys_Parts:EKMB1107111 -> SamacSys_Parts2:EKMB1107111
- moved IC3 90.7 mm to (226.6, 144.1)
- moved J3 83.3 mm to (267.0, 128.1), turned to 90 degrees
- moved R5 83.2 mm to (258.3, 120.4), turned to 0 degrees
- moved BT1 81.9 mm to (239.9, 139.1), turned to 180 degrees
- moved R6 80.4 mm to (255.7, 120.4), turned to 0 degrees
- moved C18 77.8 mm to (261.1, 116.3)
- moved IC2 77.8 mm to (252.3, 110.1)
- moved C16 77.8 mm to (243.6, 106.8)
- moved C17 77.8 mm to (261.1, 112.5)
- moved L1 77.8 mm to (261.1, 114.4)
- moved R7 77.6 mm to (253.2, 120.4), turned to 0 degrees
- moved C1 75.7 mm to (238.4, 133.8)
- moved R1 75.7 mm to (236.4, 133.8)
- moved R13 75.7 mm to (245.8, 145.5)
- moved R14 75.7 mm to (246.3, 139.7)
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Connections:
- BT1 pad 1: +3.3V -> Net-(BT1-+)
- IC2 pad 10: /RPI2040_main/GPIO1 -> /LoRa/RXD
- IC2 pad 17: /RPI2040_main/GPIO16 -> /LoRa/Reset
- IC2 pad 24: /RPI2040_main/GPIO17 -> /LoRa/Boot
- IC2 pad 9: /RPI2040_main/GPIO0 -> /LoRa/TXD
- J2 pad 1: Net-(J2-Pin_1) -> /LoRa/PC0
- J2 pad 2: Net-(J2-Pin_2) -> /LoRa/PC1
- R10 pad 2: /RPI2040_main/GPIO14 -> /RPI2040_main/R0
- R11 pad 2: /RPI2040_main/GPIO13 -> /RPI2040_main/C0
- R12 pad 2: /RPI2040_main/GPIO12 -> /RPI2040_main/C1
- R18 pad 2: /RPI2040_main/GPIO25 -> /RPI2040_main/C9
- R19 pad 2: /RPI2040_main/GPIO24 -> /RPI2040_main/C8
- R20 pad 2: /RPI2040_main/GPIO23 -> /RPI2040_main/C7
- R21 pad 2: /RPI2040_main/GPIO22 -> /RPI2040_main/C6
- R22 pad 2: /RPI2040_main/GPIO21 -> /RPI2040_main/C5
- R23 pad 2: /RPI2040_main/GPIO20 -> /RPI2040_main/C4
- R24 pad 2: /RPI2040_main/GPIO11 -> /RPI2040_main/C2
- R25 pad 2: /RPI2040_main/GPIO10 -> /RPI2040_main/C3
- R3 pad 1: Net-(J2-Pin_2) -> Net-(J5-Pin_3)
- R4 pad 1: Net-(J2-Pin_1) -> Net-(J5-Pin_2)
- R5 pad 2: /RPI2040_main/GPIO19 -> /RPI2040_main/R5
- R6 pad 2: /RPI2040_main/GPIO18 -> /RPI2040_main/R4
- R7 pad 2: /RPI2040_main/GPIO17 -> /RPI2040_main/R3
- R8 pad 2: /RPI2040_main/GPIO16 -> /RPI2040_main/R2
- R9 pad 2: /RPI2040_main/GPIO15 -> /RPI2040_main/R1
- SW1 pad A1: (no net) -> /RPI2040_main/R7
- SW1 pad A10: (no net) -> /RPI2040_main/C1
- SW1 pad A11: (no net) -> /RPI2040_main/C2
- SW1 pad A12: (no net) -> /RPI2040_main/C3
- SW1 pad A2: (no net) -> /RPI2040_main/R6
- SW1 pad A3: (no net) -> /RPI2040_main/R5
- SW1 pad A4: (no net) -> /RPI2040_main/R4
- SW1 pad A5: (no net) -> /RPI2040_main/R3
- SW1 pad A6: (no net) -> /RPI2040_main/R2
- SW1 pad A7: (no net) -> /RPI2040_main/R1
- SW1 pad A8: (no net) -> /RPI2040_main/R0
- SW1 pad A9: (no net) -> /RPI2040_main/C0
- SW1 pad B1: (no net) -> +3.3V
- SW1 pad B10: (no net) -> +3.3V
- SW1 pad B11: (no net) -> +3.3V
- SW1 pad B12: (no net) -> +3.3V
- SW1 pad B2: (no net) -> +3.3V
- SW1 pad B3: (no net) -> +3.3V
- SW1 pad B4: (no net) -> +3.3V
- SW1 pad B5: (no net) -> +3.3V
- SW1 pad B6: (no net) -> +3.3V
- SW1 pad B7: (no net) -> +3.3V
- SW1 pad B8: (no net) -> +3.3V
- SW1 pad B9: (no net) -> +3.3V
- SW2 pad A1: (no net) -> /RPI2040_main/C4
- SW2 pad A2: (no net) -> /RPI2040_main/C5
- SW2 pad A3: (no net) -> /RPI2040_main/C6
- SW2 pad A4: (no net) -> /RPI2040_main/C7
- SW2 pad A5: (no net) -> /RPI2040_main/C8
- SW2 pad B1: (no net) -> +3.3V
- SW2 pad B2: (no net) -> +3.3V
- SW2 pad B3: (no net) -> +3.3V
- SW2 pad B4: (no net) -> +3.3V
- SW2 pad B5: (no net) -> +3.3V
- U3 pad 11: /RPI2040_main/GPIO8 -> /LoRa/Boot
- U3 pad 12: /RPI2040_main/GPIO9 -> /RPI2040_main/Digital_in
- U3 pad 13: /RPI2040_main/GPIO10 -> /RPI2040_main/Vibration
- U3 pad 15: /RPI2040_main/GPIO12 -> /RPI2040_main/SDA0
- U3 pad 16: /RPI2040_main/GPIO13 -> /RPI2040_main/SCL0
- U3 pad 2: /RPI2040_main/GPIO0 -> /RPI2040_main/LoRa_TXD
- U3 pad 3: /RPI2040_main/GPIO1 -> /RPI2040_main/LoRa_RXD
- U3 pad 9: /RPI2040_main/GPIO7 -> /LoRa/Reset
Routing:
- net +3.3V: track 28.7 -> 149.0 mm
- net /RPI2040_main/C9: track 0.00 -> 47.9 mm, vias 0 -> 1
- net /RPI2040_main/C8: track 0.00 -> 44.3 mm, vias 0 -> 1
- net /RPI2040_main/C7: track 0.00 -> 40.8 mm, vias 0 -> 1
- net /RPI2040_main/C6: track 0.00 -> 37.2 mm, vias 0 -> 1
- net /RPI2040_main/GPIO17: track 36.6 -> 0.00 mm, vias 2 -> 0
- net /LoRa/Reset: track 0.00 -> 35.2 mm, vias 0 -> 2
- net /RPI2040_main/C5: track 0.00 -> 33.6 mm, vias 0 -> 1
- net /LoRa/PB10: track 40.8 -> 9.08 mm, vias 1 -> 0
- net Net-(AE1-A): track 3.23 -> 33.7 mm
- net /RPI2040_main/GPIO16: track 30.2 -> 0.00 mm, vias 2 -> 0
- net /RPI2040_main/C4: track 0.00 -> 29.0 mm, vias 0 -> 1
- net /LoRa/Boot: track 0.00 -> 28.5 mm, vias 0 -> 3
- net /LoRa/PA9: track 35.4 -> 6.82 mm
- net /LoRa/PA2: track 38.3 -> 11.6 mm, vias 1 -> 0
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- added copper zone on B.Cu, net GND
- added copper zone on F.Cu, net GND
- removed copper zone on F.Cu, net +3.3V
Other:
- board outline added: 62 x 52 mm
- board text added: "Address"
- board text added: "Delta"
- board text added: "Interval"
- board text added: "Pause"

Commit message: test
Parts:
- removed J2: Conn_01x18, Connector_PinHeader_2.54mm:PinHeader_1x18_P2.54mm_Vertical
- removed J5: USB, Connector_PinHeader_2.54mm:PinHeader_1x03_P2.54mm_Vertical
- added C19: 10uf, Capacitor_SMD:C_0805_2012Metric, F.Cu at (226.9, 106.8)
- added C20: 10uf, Capacitor_SMD:C_0805_2012Metric, F.Cu at (237.4, 101.1)
- added G***: LOGO, LOGO, F.Cu at (264.0, 100.5)
- added G***: LOGO, LOGO, B.Cu at (263.6, 100.5)
- added IC5: NCP1117IDT33T4G, SamacSys_Parts3:NCP1117IDT33T4G, F.Cu at (227.0, 101.4)
- added J4: 10118192-0002LF, SamacSys_Parts3:101181920002LF, F.Cu at (214.9, 99.7)
- added JP1: Jumper_2_Open, Jumper:SolderJumper-2_P1.3mm_Open_RoundedPad1.0x1.5mm, B.Cu at (219.2, 103.0)
- moved R32 2.11 mm to (228.5, 123.1)
- moved R30 0.73 mm to (215.3, 143.3), turned to 0 degrees
- moved R33 0.63 mm to (229.1, 119.9)
- moved C10 0.17 mm to (229.6, 118.9)
Connections:
- R3 pad 1: Net-(J5-Pin_3) -> /RPI2040_main/D+
- R4 pad 1: Net-(J5-Pin_2) -> /RPI2040_main/D-
- S1 pad 1: unconnected-(S1-Pad1) -> +3.3V
- U3 pad 11: /LoRa/Boot -> unconnected-(U3-GPIO8-Pad11)
- U3 pad 12: /RPI2040_main/Digital_in -> unconnected-(U3-GPIO9-Pad12)
- U3 pad 13: /RPI2040_main/Vibration -> /RPI2040_main/PIR
- U3 pad 14: /RPI2040_main/GPIO11 -> /RPI2040_main/Vibration
- U3 pad 15: /RPI2040_main/SDA0 -> unconnected-(U3-GPIO12-Pad15)
- U3 pad 16: /RPI2040_main/SCL0 -> unconnected-(U3-GPIO13-Pad16)
- U3 pad 2: /RPI2040_main/LoRa_TXD -> /RPI2040_main/SDA0
- U3 pad 27: /RPI2040_main/GPIO16 -> /LoRa/TXD
- U3 pad 28: /RPI2040_main/GPIO17 -> /LoRa/RXD
- U3 pad 29: /RPI2040_main/GPIO18 -> /LoRa/Reset
- U3 pad 3: /RPI2040_main/LoRa_RXD -> /RPI2040_main/SCL0
- U3 pad 30: /RPI2040_main/GPIO19 -> /LoRa/Boot
- U3 pad 37: /RPI2040_main/GPIO25 -> unconnected-(U3-GPIO25-Pad37)
- U3 pad 4: /RPI2040_main/SDA -> /RPI2040_main/Digital_in
- U3 pad 5: /RPI2040_main/SCL -> /RPI2040_main/AIR_RES
- U3 pad 6: /RPI2040_main/PIR -> /RPI2040_main/AIR_INT
- U3 pad 7: /RPI2040_main/AIR_INT -> unconnected-(U3-GPIO5-Pad7)
- U3 pad 8: /RPI2040_main/AIR_RES -> /RPI2040_main/SDA
- U3 pad 9: /LoRa/Reset -> /RPI2040_main/SCL
Routing:
- net +3.3V: track 149.0 -> 349.5 mm, vias 0 -> 10
- net /RPI2040_main/SDA: track 1.99 -> 66.6 mm, vias 1 -> 4
- net /RPI2040_main/SCL: track 1.24 -> 62.4 mm, vias 1 -> 5
- net /LoRa/PC0: track 43.0 -> 0.00 mm
- net /RPI2040_main/LUX: track 2.42 -> 44.1 mm, vias 0 -> 2
- net /LoRa/PC1: track 38.7 -> 0.00 mm
- net /RPI2040_main/Vibration: track 5.10 -> 42.4 mm
- net /LoRa/PB5: track 34.2 -> 0.00 mm
- net /RPI2040_main/Digital_in: track 2.59 -> 32.7 mm
- net GND: track 9.90 -> 39.9 mm, vias 0 -> 75
- net /RPI2040_main/AIR_RES: track 0.00 -> 29.6 mm, vias 0 -> 2
- net /RPI2040_main/AIR_INT: track 0.00 -> 27.9 mm, vias 0 -> 2
- net /LoRa/PB3: track 25.8 -> 0.00 mm
- net /RPI2040_main/SCL0: track 0.00 -> 23.8 mm
- net /LoRa/TXD: track 0.00 -> 23.1 mm, vias 0 -> 2
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Other:
- board text added: "+"
- board text added: "-"
- board text added: "1"
- board text added: "BOOT"
- board text added: "Digital IN"
- board text added: "I2C"
- board text added: "On/Off"

Commit message: TJEK
Parts:
- added H1: MountingHole, MountingHole:MountingHole_3.2mm_M3, F.Cu at (244.9, 100.6)
- added H2: MountingHole, MountingHole:MountingHole_3.2mm_M3, F.Cu at (266.0, 151.0)
- added H3: MountingHole, MountingHole:MountingHole_3.2mm_M3, F.Cu at (217.0, 151.0)
- renumbered TP1 to Antenna1, C11 to C10, C12 to C11, C13 to C12, C14 to C13, C2 to C14, C3 to C16, C4 to C17, C22 to C18, C16 to C19, C19 to C2, C17 to C20, C18 to C21, C20 to C3, C5 to C4, C6 to C5, C7 to C6, C8 to C7, C9 to C8, C10 to C9, IC5 to IC1, IC3 to IC2, IC1 to IC3, IC2 to IC5, J6 to J1, J4 to J2, J1 to J3, J8 to J4, J7 to J5, J3 to J6, R29 to R10, R28 to R11, R31 to R12, R23 to R13, R22 to R14, R21 to R15, R20 to R16, R19 to R17, R26 to R19, R3 to R2, R27 to R20, R5 to R21, R6 to R22, R7 to R23, R8 to R24, R9 to R25, R10 to R26, R11 to R27, R12 to R28, R24 to R29, R4 to R3, R25 to R30, R32 to R4, R33 to R5, R13 to R6, R14 to R7, R2 to R8, R30 to R9, SW2 to SW1, SW1 to SW2, U3 to U2, U2 to U3, JP1 to USB_Power1, Y3 to Y1
Routing:
- net /RPI2040_main/Vibration: track 42.4 -> 41.3 mm
- net GND: vias 75 -> 73
Other:
- board size 62 x 52 mm -> 62 x 57 mm

Commit message: tjek
Parts:
- added C22: 100nf, Capacitor_SMD:C_0402_1005Metric, B.Cu at (223.9, 146.6)
- added C23: 10uf, Capacitor_SMD:C_0805_2012Metric, B.Cu at (267.9, 109.3)
- added C24: 10uf, Capacitor_SMD:C_0805_2012Metric, F.Cu at (240.8, 105.0)
- added C25: 10uf, Capacitor_SMD:C_0805_2012Metric, F.Cu at (211.3, 125.6)
- added C26: 10uf, Capacitor_SMD:C_0805_2012Metric, B.Cu at (211.5, 109.3)
- added R31: 10K, Resistor_SMD:R_0402_1005Metric, F.Cu at (214.7, 130.4)
- added R32: 10K, Resistor_SMD:R_0402_1005Metric, F.Cu at (214.7, 133.4)
- moved U1 2.96 mm to (238.5, 143.9)
Connections:
- net /LoRa/Boot renamed /RPI2040_main/LoRa_Boot
- net /LoRa/PA0 renamed /RPI2040_main/PA0
- net /LoRa/RXD renamed /RPI2040_main/LoRa_RXD
- net /LoRa/Reset renamed /RPI2040_main/LoRa_Reset
- net /LoRa/TXD renamed /RPI2040_main/LoRa_TXD
- C19 pad 1: VCC -> +3.3V
- IC5 pad 1: VCC -> +3.3V
- IC5 pad 11: /LoRa/PB5 -> unconnected-(IC5-PB5-Pad11)
- IC5 pad 12: /LoRa/PC1 -> unconnected-(IC5-PC1-Pad12)
- IC5 pad 13: /LoRa/PC0 -> unconnected-(IC5-PC0-Pad13)
- IC5 pad 18: /LoRa/PA3 -> unconnected-(IC5-PA3-Pad18)
- IC5 pad 19: /LoRa/PA2 -> unconnected-(IC5-PA2-Pad19)
- IC5 pad 20: /LoRa/PB10 -> unconnected-(IC5-PB10-Pad20)
- IC5 pad 21: /LoRa/PA9 -> unconnected-(IC5-PA9-Pad21)
- IC5 pad 25: /LoRa/PB9 -> unconnected-(IC5-PB9-Pad25)
- IC5 pad 26: /LoRa/PB14 -> unconnected-(IC5-PB14-Pad26)
- IC5 pad 27: /LoRa/PA10 -> unconnected-(IC5-PA10-Pad27)
- IC5 pad 28: /LoRa/PB0 -> unconnected-(IC5-PB0-Pad28)
- IC5 pad 3: /LoRa/PA13 -> unconnected-(IC5-PA13-Pad3)
- IC5 pad 4: /LoRa/PA14 -> unconnected-(IC5-PA14-Pad4)
- IC5 pad 5: /LoRa/PB15 -> unconnected-(IC5-PB15-Pad5)
- IC5 pad 6: /LoRa/PA15 -> unconnected-(IC5-PA15-Pad6)
- IC5 pad 7: /LoRa/PB4 -> unconnected-(IC5-PB4-Pad7)
- IC5 pad 8: /LoRa/PB3 -> unconnected-(IC5-PB3-Pad8)
- R2 pad 2: /RPI2040_main/D+ -> Net-(U2-USB_DP)
- R3 pad 2: /RPI2040_main/D- -> Net-(U2-USB_DM)
- U2 pad 46: /RPI2040_main/D- -> Net-(U2-USB_DM)
- U2 pad 47: /RPI2040_main/D+ -> Net-(U2-USB_DP)
Routing:
- net +3.3V: track 349.5 -> 376.1 mm, vias 10 -> 11
- net GND: track 39.9 -> 50.4 mm, vias 73 -> 78
- net /RPI2040_main/PIR: track 23.2 -> 26.9 mm
- net Net-(U2-USB_DP): track 0.00 -> 2.99 mm
- net /RPI2040_main/D+: track 17.4 -> 14.4 mm
- net Net-(U2-USB_DM): track 0.00 -> 2.97 mm
- net /RPI2040_main/D-: track 15.9 -> 13.0 mm
- net VCC: track 2.70 -> 0.00 mm
- net /RPI2040_main/SCL0: track 23.8 -> 22.6 mm

Commit message: siejwi
Parts:
- added D1: LED, LED_SMD:LED_0805_2012Metric, B.Cu at (231.8, 120.8)
- added J7: FAN, Connector_PinHeader_2.54mm:PinHeader_1x02_P2.54mm_Vertical, B.Cu at (250.3, 99.2)
- added Q1: BCX56, Package_TO_SOT_SMD:SOT-89-3, B.Cu at (235.1, 101.0)
- added R33: 70Ω, Resistor_SMD:R_0402_1005Metric, B.Cu at (232.4, 118.8)
- added R34: 2.4KΩ, Resistor_SMD:R_0603_1608Metric, B.Cu at (231.4, 104.0)
- L1: value 0R -> 0Ω
- R1, R10, R11, R12, R13, R14, R15, R16, R17, R18, R19, R20, R21, R22, R23, R24, R25, R26, R27, R28, R29, R30, R31, R32, R4, R5, R7, R9: value 10K -> 10KΩ
- R2, R3: value 27 -> 27Ω
- R8: value 1K -> 1KΩ
Connections:
- U2 pad 17: /RPI2040_main/GPIO14 -> Net-(D1-A)
- U2 pad 18: /RPI2040_main/GPIO15 -> unconnected-(U2-GPIO15-Pad18)
- U2 pad 31: /RPI2040_main/GPIO20 -> Net-(U2-GPIO20)
Routing:
- net Net-(J7-Pin_1): track 0.00 -> 18.2 mm
- net +3.3V: track 376.1 -> 384.4 mm, vias 11 -> 13
- net Net-(U2-GPIO20): track 0.00 -> 6.64 mm, vias 0 -> 1
- net Net-(D1-A): track 0.00 -> 6.10 mm, vias 0 -> 1
- net GND: track 50.4 -> 53.1 mm, vias 78 -> 81
- net Net-(Q1-B): track 0.00 -> 2.01 mm
- net Net-(D1-K): track 0.00 -> 1.64 mm
- net /RPI2040_main/LoRa_Boot: track 29.0 -> 27.7 mm
- net /RPI2040_main/PIR: track 26.9 -> 26.2 mm
