File: Modbus-Master-main/Produktion/Modbus_master.kicad_pcb (KiCad board)
At the start: 2 copper layers, 104 x 129 mm, 82 parts, among them J1 Screw_Terminal_01x03, J2 SIM8066-6-1-14-01-A, J3 Conn_Coaxial, J4 Screw_Terminal_01x04, J5 AVR-ISP-6, J6 Conn_01x04_Pin, Q1 BC847CW, Q2 BC847CW, Q3 BC847CW, Q4 BC847CW, Q5 BC847CW, SW1 TL3305AF260QG, U1 ATmega2560-16A, U2 SP485EN-L/TR, U3 L7805, U4 SIM7080G, U5 LSF0204PW-Q100J, Y1 ABM3B-8.000MHZ-10-1-U-T

Commit message: ændring
Parts:
- added D4: GS1M-LTP, Diode_SMD:D_SMA, F.Cu at (151.6, 82.5)
Connections:
- D8 pad 2: VCC_5 -> Net-(D4-K)
Routing:
- net GND: track 100.0 -> 139.5 mm, vias 26 -> 62
- net VCC_5: track 302.4 -> 297.6 mm
- net Net-(D4-K): track 0.00 -> 4.33 mm
