File: Modbus-Master-main/Produktion/Modbus_master.kicad_sch (KiCad schematic)
At the start: 76 parts, among them J1 Screw_Terminal_01x03, J2 SIM8066-6-1-14-01-A, J3 Conn_Coaxial, J4 Screw_Terminal_01x04, J5 AVR-ISP-6, J6 Conn_01x04_Pin, Q1 BC847CW, Q2 BC847CW, Q3 BC847CW, Q4 BC847CW, Q5 BC847CW, SW1 TL3305AF260QG, U1 ATmega2560-16A, U2 SP485EN-L/TR, U3 L7805, U4 SIM7080G, U5 LSF0204PW-Q100J, Y1 ABM3B-8.000MHZ-10-1-U-T

Commit message: ændringer
Other:
- moved on the sheet: C14, C15, C16, D9, R21, R22, R24, R26, R27, U4, U5

Commit message: ændring
Parts:
- added D4: GS1M-LTP, Diode_SMD:D_SMA, symbol Diode:US1G
Connections:
- net VCC_5: now also D4.2 (A); no longer D8.2 (A)
- new net: D4.1 (K), D8.2 (A)
Other:
- moved on the sheet: D8
Changed lines of the file:
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@@
     (stroke (width 0) (type default))
   )
+  (wire (pts (xy 257.175 242.57) (xy 259.715 242.57))
+    (stroke (width 0) (type default))
+  )
   (wire (pts (xy 196.215 274.32) (xy 196.215 276.86))
     (stroke (width 0) (type default))
@@
     (stroke (width 0) (type default))
   )
-  (wire (pts (xy 262.89 242.57) (xy 271.145 242.57))
+  (wire (pts (xy 267.335 242.57) (xy 271.145 242.57))
     (stroke (width 0) (type default))
   )
@@
     (stroke (width 0) (type default))
   )
-  (wire (pts (xy 246.38 242.57) (xy 255.27 242.57))
+  (wire (pts (xy 246.38 242.57) (xy 249.555 242.57))
     (stroke (width 0) (type default))
   )
@@
     )
   )
+  (symbol (lib_id "Diode:US1G") (at 253.365 242.57 180) (unit 1)
+    (in_bom yes) (on_board yes) (dnp no) (fields_autoplaced)
+    (property "Reference" "D4" (at 253.365 237.49 0)
+      (effects (font (size 1.27 1.27)))
+    )
+    (property "Value" "GS1M-LTP" (at 253.365 240.03 0)
+      (effects (font (size 1.27 1.27)))
+    )
+    (property "Footprint" "Diode_SMD:D_SMA" (at 253.365 238.125 0)
+      (effects (font (size 1.27 1.27)) hide)
+    )
+    (property "Datasheet" "https://www.mouser.dk/datasheet/2/258/GS1A_L_7eGS1M_L_DO_214AC_-2634344.pdf" (at 253.365 242.57 0)
+      (effects (font (size 1.27 1.27)) hide)
+    )
+    (property "Sim.Device" "D" (at 253.365 242.57 0)
+      (effects (font (size 1.27 1.27)) hide)
+    )
+    (property "Sim.Pins" "1=K 2=A" (at 253.365 242.57 0)
+      (effects (font (size 1.27 1.27)) hide)
+    )
+    (property "Manufacturer_Name" "Micro Commercial Components (MCC)" (at 253.365 242.57 0)
+      (effects (font (size 1.27 1.27)) hide)
+    )
+    (property "Manufacturer_Part_Number" "GS1M-LTP" (at 253.365 242.57 0)
+      (effects (font (size 1.27 1.27)) hide)
+    )
+    (property "Mouser Price/Stock" "0,15" (at 253.365 242.57 0)
+      (effects (font (size 1.27 1.27)) hide)
+    )
+    (property "Description" "" (at 253.365 242.57 0)
+      (effects (font (size 1.27 1.27)) hide)
+    )
+    (pin "1")
+    (pin "2")
+    (instances
+      (project "Modbus_master"
+        (path "/7751fb88-c92a-4fc4-933d-a75f17492f83"
+          (reference "D4") (unit 1)
+        )
+      )
+    )
+  )
   (symbol (lib_id "Device:R") (at 168.275 237.49 90) (unit 1)
     (in_bom yes) (on_board yes) (dnp no) (fields_autoplaced)
@@
     )
   )
-  (symbol (lib_id "Diode:US1G") (at 259.08 242.57 180) (unit 1)
+  (symbol (lib_id "Diode:US1G") (at 263.525 242.57 180) (unit 1)
     (in_bom yes) (on_board yes) (dnp no) (fields_autoplaced)
-    (property "Reference" "D8" (at 259.08 237.49 0)
+    (property "Reference" "D8" (at 263.525 237.49 0)
       (effects (font (size 1.27 1.27)))
     )
-    (property "Value" "GS1M-LTP" (at 259.08 240.03 0)
+    (property "Value" "GS1M-LTP" (at 263.525 240.03 0)
       (effects (font (size 1.27 1.27)))
     )
-    (property "Footprint" "Diode_SMD:D_SMA" (at 259.08 238.125 0)
+    (property "Footprint" "Diode_SMD:D_SMA" (at 263.525 238.125 0)
       (effects (font (size 1.27 1.27)) hide)
     )
-    (property "Datasheet" "https://www.mouser.dk/datasheet/2/258/GS1A_L_7eGS1M_L_DO_214AC_-2634344.pdf" (at 259.08 242.57 0)
+    (property "Datasheet" "https://www.mouser.dk/datasheet/2/258/GS1A_L_7eGS1M_L_DO_214AC_-2634344.pdf" (at 263.525 242.57 0)
       (effects (font (size 1.27 1.27)) hide)
     )
-    (property "Sim.Device" "D" (at 259.08 242.57 0)
+    (property "Sim.Device" "D" (at 263.525 242.57 0)
       (effects (font (size 1.27 1.27)) hide)
     )
-    (property "Sim.Pins" "1=K 2=A" (at 259.08 242.57 0)
+    (property "Sim.Pins" "1=K 2=A" (at 263.525 242.57 0)
       (effects (font (size 1.27 1.27)) hide)
     )
-    (property "Manufacturer_Name" "Micro Commercial Components (MCC)" (at 259.08 242.57 0)
+    (property "Manufacturer_Name" "Micro Commercial Components (MCC)" (at 263.525 242.57 0)
       (effects (font (size 1.27 1.27)) hide)
     )
-    (property "Manufacturer_Part_Number" "GS1M-LTP" (at 259.08 242.57 0)
+    (property "Manufacturer_Part_Number" "GS1M-LTP" (at 263.525 242.57 0)
       (effects (font (size 1.27 1.27)) hide)
     )
-    (property "Mouser Price/Stock" "0,15" (at 259.08 242.57 0)
+    (property "Mouser Price/Stock" "0,15" (at 263.525 242.57 0)
       (effects (font (size 1.27 1.27)) hide)
     )
-    (property "Description" "" (at 259.08 242.57 0)
+    (property "Description" "" (at 263.525 242.57 0)
       (effects (font (size 1.27 1.27)) hide)
     )
