File: Wireless modbus/Produktion/Modbus_master.kicad_pcb (KiCad board)
At the start: 2 copper layers, 104 x 129 mm, 82 parts, among them J1 Screw_Terminal_01x03, J2 SIM8066-6-1-14-01-A, J3 Conn_Coaxial, J4 Screw_Terminal_01x04, J5 AVR-ISP-6, J6 Conn_01x04_Pin, Q1 BC847CW, Q2 BC847CW, Q3 BC847CW, Q4 BC847CW, Q5 BC847CW, SW1 TL3305AF260QG, U1 ATmega2560-16A, U2 SP485EN-L/TR, U3 L7805, U4 SIM7080G, U5 LSF0204PW-Q100J, Y1 ABM3B-8.000MHZ-10-1-U-T

Commit message: Ændring i print
Parts:
- removed Q1, Q2, Q3: BC847CW, Package_TO_SOT_SMD:SOT-323_SC-70
- removed R11, R14, R18: 1K, Resistor_SMD:R_0402_1005Metric
- added C17: 1uF, Capacitor_SMD:C_0402_1005Metric, F.Cu at (148.7, 92.4)
- added IC1: LoRa-E5, SamacSys_Parts:LoRaE5, F.Cu at (140.0, 88.2)
- moved R21 29.4 mm to (110.6, 76.5)
- moved R22 26.7 mm to (111.8, 76.5)
- moved R1 20.4 mm to (152.3, 111.6), turned to 0 degrees
- moved D8 15.4 mm to (150.5, 102.2)
- moved U5 14.2 mm to (152.0, 86.3)
- moved R27 14.0 mm to (153.0, 91.2), turned to 180 degrees
- moved R26 13.9 mm to (151.6, 92.4), turned to 180 degrees
- moved C2 13.5 mm to (145.3, 109.0), turned to 90 degrees
- moved D5 13.1 mm to (142.1, 69.1), turned to 0 degrees
- moved C6 11.8 mm to (152.7, 126.2)
- moved C8 11.8 mm to (151.6, 126.2)
- moved C9 11.8 mm to (150.5, 126.2)
- moved J6 11.4 mm to (130.4, 100.3), turned to 90 degrees
- moved J5 10.5 mm to (147.8, 109.2)
- moved Y1 10.2 mm to (138.7, 107.4)
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Connections:
- R15 pad 1: Net-(Q1-C) -> LED_RED
- R16 pad 1: Net-(Q2-C) -> LED_GREEN
- R17 pad 2: Net-(Q3-C) -> LED_BLUE
- U1 pad 51: DTR_E -> unconnected-(U1-PG0-Pad51)
- U1 pad 63: unconnected-(U1-PJ0-Pad63) -> LoraTX
- U1 pad 64: unconnected-(U1-PJ1-Pad64) -> LoraRX
- U4 pad 6: SIM_DTR -> unconnected-(U4-UART1_DTR-Pad6)
- U5 pad 11: DTR_E -> unconnected-(U5-B3-Pad11)
- U5 pad 4: SIM_DTR -> unconnected-(U5-A3-Pad4)
Routing:
- net LoraRX: track 0.00 -> 44.8 mm, vias 0 -> 2
- net LoraTX: track 0.00 -> 42.9 mm, vias 0 -> 2
- net SIM_DTR: track 31.7 -> 0.00 mm, vias 2 -> 0
- net GND: track 100.0 -> 126.6 mm, vias 26 -> 38
- net PWRSTATUS: track 84.6 -> 109.4 mm, vias 2 -> 1
- net VCC_5: track 302.4 -> 277.7 mm, vias 6 -> 4
- net UART1_TXD: track 16.7 -> 35.5 mm
- net VCC_3.6: track 49.6 -> 67.3 mm, vias 2 -> 0
- net DTR_E: track 17.6 -> 0.00 mm
- net VDD_EXT: track 34.9 -> 51.1 mm, vias 2 -> 4
- net SIM_TXD: track 33.0 -> 46.8 mm
- net UART1_RXD: track 20.6 -> 34.3 mm
- net SIM_RXD: track 36.0 -> 49.0 mm
- net UART2_RXD: track 36.4 -> 24.2 mm
- net CD: track 12.9 -> 24.1 mm, vias 0 -> 2
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
Commit message: Ændring
Parts:
- renumbered D3 to D2, D7 to D3, D2 to D4, D8 to D6, D10 to D7, D6 to D8, J6 to J3, J3 to J4, J4 to J5, J5 to J6, Q5 to Q1, Q4 to Q2, R8 to R10, R32 to R11, R5 to R12, R9 to R13, R10 to R14, R30 to R18, R31 to R19, R12 to R20, R13 to R21, R20 to R22, R19 to R24, R21 to R26, R22 to R27, R24 to R28, R26 to R29, R27 to R30, R28 to R5, R29 to R6, R33 to R8, R6 to R9

Commit message: Ændring
Parts:
- added C18: NC, Capacitor_SMD:C_0402_1005Metric, F.Cu at (129.6, 79.0)
- added C19: NC, Capacitor_SMD:C_0402_1005Metric, F.Cu at (132.9, 79.0)
- added L1: 0R, Resistor_SMD:R_0402_1005Metric, F.Cu at (131.2, 78.9)
- C17: value 1uF -> 4.7uF
- D2: value UHD111A-FKA -> NH-B2020RGBA-HF; footprint LED_SMD_RGB:LED_RGB_1_1_mm -> SamacSys_Parts:NHB2020RGBAHF
- D3: value GREEN -> GREEN LED
- D7: value YELLOW -> YELLOW LED
- moved J4 2.18 mm to (131.3, 75.8)
- moved R15 0.94 mm to (135.9, 133.0)
- moved R16 0.94 mm to (137.1, 133.0)
- moved R17 0.94 mm to (138.4, 133.0)
- moved D2 0.71 mm to (137.1, 136.0)
Connections:
- D2 pad 1: Net-(D2-BK) -> Net-(D2-K_RED)
- D2 pad 2: Net-(D2-GK) -> Net-(D2-K_BLUE)
- D2 pad 3: Net-(D2-RK) -> VCC_5
- D2 pad 4: VCC_5 -> Net-(D2-K_GREEN)
- J4 pad 1: RF_ANT -> Net-(J4-In)
- R15 pad 2: Net-(D2-RK) -> Net-(D2-K_RED)
- R16 pad 2: Net-(D2-GK) -> Net-(D2-K_GREEN)
- R17 pad 1: Net-(D2-BK) -> Net-(D2-K_BLUE)
Routing:
- net VCC_3.6: track 67.3 -> 74.7 mm
- net GND: track 126.6 -> 133.1 mm
- net Net-(D2-K_GREEN): track 0.00 -> 3.83 mm
- net Net-(J4-In): track 0.00 -> 3.39 mm
- net VCC_5: track 277.7 -> 281.1 mm
- net Net-(D2-BK): track 2.73 -> 0.00 mm
- net Net-(D2-K_BLUE): track 0.00 -> 2.16 mm
- net Net-(D2-K_RED): track 0.00 -> 2.11 mm
- net Net-(D2-RK): track 1.71 -> 0.00 mm
- net RF_ANT: track 10.5 -> 12.2 mm
- net Net-(D2-GK): track 1.46 -> 0.00 mm
- net LED_BLUE: track 7.15 -> 6.10 mm
- net LED_GREEN: track 6.53 -> 5.56 mm
- net LED_RED: track 8.27 -> 7.39 mm

Commit message: Ændring
Parts:
- J2: value SIM8066-6-1-14-01-A -> XKNANO-113
Connections:
- U1 pad 19: SS -> unconnected-(U1-PB0-Pad19)

Commit message: Ændring
Parts:
- added D10: GS1M-LTP, Diode_SMD:D_SMA, F.Cu at (144.5, 100.8)
- moved R30 0.74 mm to (153.3, 91.9)
- moved R29 0.67 mm to (151.2, 92.9)
- moved R1 0.33 mm to (151.9, 111.6)
Connections:
- C14 pad 1: VCC_3.6 -> +3.3V
- C15 pad 1: VCC_3.6 -> +3.3V
- C16 pad 1: VCC_3.6 -> +3.3V
- C17 pad 2: VCC_3.6 -> +3.3V
- D6 pad 1: VCC_3.6 -> Net-(D10-A)
- D9 pad 1: VCC_3.6 -> +3.3V
- IC1 pad 1: VCC_3.6 -> +3.3V
- U4 pad 34: VCC_3.6 -> +3.3V
- U4 pad 35: VCC_3.6 -> +3.3V
Routing:
- net VCC_3.6: track 74.7 -> 0.00 mm
- net +3.3V: track 0.00 -> 70.9 mm
- net GND: track 133.1 -> 189.2 mm, vias 38 -> 65
- net Net-(D10-A): track 0.00 -> 4.22 mm
- net VCC_5: track 281.1 -> 285.1 mm
- net SIM_RXD: track 49.0 -> 51.5 mm
- net RESET: track 13.6 -> 15.1 mm
- net UART1_RXD: track 34.3 -> 35.8 mm
- net VDD_EXT: track 51.1 -> 52.2 mm
- net UART1_TXD: track 35.5 -> 36.6 mm
- net CD: track 24.1 -> 25.2 mm
- net SIM_PWRKEY: track 60.5 -> 61.5 mm
- net Net-(J1-Pin_2): track 11.8 -> 12.8 mm
- net SIM_VDD: track 28.6 -> 29.4 mm
- net Net-(D1-IO1): track 38.2 -> 38.9 mm
