File: Wireless modbus/Produktion/Modbus_master.kicad_sch (KiCad schematic)
At the start: 76 parts, among them J1 Screw_Terminal_01x03, J2 SIM8066-6-1-14-01-A, J3 Conn_Coaxial, J4 Screw_Terminal_01x04, J5 AVR-ISP-6, J6 Conn_01x04_Pin, Q1 BC847CW, Q2 BC847CW, Q3 BC847CW, Q4 BC847CW, Q5 BC847CW, SW1 TL3305AF260QG, U1 ATmega2560-16A, U2 SP485EN-L/TR, U3 L7805, U4 SIM7080G, U5 LSF0204PW-Q100J, Y1 ABM3B-8.000MHZ-10-1-U-T

Commit message: Ændring i print
Parts:
- removed Q1, Q2, Q3: BC847CW, Package_TO_SOT_SMD:SOT-323_SC-70, symbol Transistor_BJT:BC847W
- removed R11, R14, R18: 1K, Resistor_SMD:R_0402_1005Metric, symbol Device:R
- added C17: 1uF, Capacitor_SMD:C_0402_1005Metric, symbol Device:C_Small
- added IC1: LoRa-E5, LoRaE5, symbol SamacSys_Parts:LoRa-E5
Connections:
- net GND: now also C17.1, IC1.14 (GND_2), IC1.16 (GND_3), IC1.2 (GND_1), IC1.22 (GND_4)
- net LED_BLUE: now also R17.2
- net LED_GREEN: now also R16.1
- net LED_RED: now also R15.1
- net RF_ANT: now also IC1.15 (RFIO)
- net VCC_3.6: now also C17.2, IC1.1 (VCC)
- net LoraTX: now reaches U1.63 (PJ0)
- net LoraTX: now also IC1.10 (PB6)
- net LoraRX: now reaches U1.64 (PJ1)
- net LoraRX: now also IC1.9 (PB7)
- net DTR_E: no longer names the net of U1.51 (PG0)
- net DTR_E: no longer U5.11 (B3)
- net SIM_DTR: no longer names the net of U4.6 (UART1_DTR)
- net SIM_DTR: no longer U5.4 (A3)
Other:
- moved on the sheet: D10, D3, D7, D8, J5, Q4, R15, R16, R17, R20, R23, R25

Commit message: Ændring
Parts:
- added C18, C19: NC, Capacitor_SMD:C_0402_1005Metric, symbol Device:C_Small
- added L1: 0R, Resistor_SMD:R_0402_1005Metric, symbol Device:L
- C1, C2, C3, C4, C5: JLCPART# (none) -> C526997
- C10: JLCPART# (none) -> C161258
- C11, C12, C14, C6, C7, C8, C9: JLCPART# (none) -> C56392
- C15: JLCPART# (none) -> C326568
- C16: JLCPART# (none) -> C76661
- C17: value 1uF -> 4.7uF; JLCPART# (none) -> C2858031
- D1: JLCPART# (none) -> C87908
- D3: renamed from D7; value GREEN -> GREEN LED; JLCPART# (none) -> C965805
- D4: renamed from D2; JLCPART# (none) -> C282388
- D5: JLCPART# (none) -> C282388
- D6: renamed from D8; JLCPART# (none) -> C435833
- D7: renamed from D10; value YELLOW -> YELLOW LED; JLCPART# (none) -> C965802
- D8: renamed from D6; JLCPART# (none) -> C282388
- D9: JLCPART# (none) -> C1972978
- renumbered D3 to D2, J6 to J3, J3 to J4, J4 to J5, J5 to J6, Q5 to Q1, Q4 to Q2, R8 to R10, R32 to R11, R5 to R12, R9 to R13, R10 to R14, R30 to R18, R31 to R19, R12 to R20, R13 to R21, R20 to R22, R19 to R24, R21 to R26, R22 to R27, R24 to R28, R26 to R29, R27 to R30, R28 to R5, R29 to R6, R33 to R8, R6 to R9
Connections:
- net GND: now also C18.1, C19.1
- net RF_ANT: now also C18.2, L1.1; no longer J4.1 (In)
- new net: C19.2, J4.1 (In), L1.2
Other:
- moved on the sheet: D6, J4

Commit message: Ændring
Parts:
- removed D2: UHD111A-FKA, LED_SMD_RGB:LED_RGB_1_1_mm, symbol Device:LED_BGRA
- added D2: NH-B2020RGBA-HF, NHB2020RGBAHF, symbol SamacSys_Parts:NH-B2020RGBA-HF
- J2: JLCPART# (none) -> C381071
- J4: JLCPART# (none) -> C434808
- Q1, Q2: JLCPART# (none) -> C75567
- R1, R11, R12, R13, R14, R18, R19, R21, R26, R27, R29, R30, R5, R6, R7, R8, R9: JLCPART# (none) -> C25744
- R10: JLCPART# (none) -> C25792
- R15: JLCPART# (none) -> C25113
- R16, R17: JLCPART# (none) -> C44933
- R2, R3, R4: JLCPART# (none) -> C25092
- R20: JLCPART# (none) -> C25765
- R22, R23, R25: JLCPART# (none) -> C11702
- R24: JLCPART# (none) -> C560547
- R28: JLCPART# (none) -> C25764
- SW1: JLCPART# (none) -> C2886902
- U1: JLCPART# (none) -> C22460
- U2: JLCPART# (none) -> C6855
- U4: JLCPART# (none) -> C2943992
- U5: JLCPART# (none) -> C202288
- Y1: JLCPART# (none) -> C276420
Connections:
- net VCC_5: now also D2.3 (COM_A)
- net at R17.1: now also D2.2 (K_BLUE)
- net at R16.2: now also D2.4 (K_GREEN)
- net at R15.2: now also D2.1 (K_RED)
Other:
- moved on the sheet: D3, R15, R16, R17, R22

Commit message: Ændring
Parts:
- J2: value SIM8066-6-1-14-01-A -> XKNANO-113
Connections:
- net SS: no longer names the net of U1.19 (PB0)
- no-connect marks 0 -> 128
Changed lines of the file:
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@@
   (junction (at 196.215 307.34) (diameter 0) (color 0 0 0 0)
   )
+  (no_connect (at 162.56 94.615))
+  (no_connect (at 45.085 230.505))
+  (no_connect (at 213.36 114.935))
+  (no_connect (at 85.725 281.305))
+  (no_connect (at 45.085 212.725))
+  (no_connect (at 45.085 253.365))
+  (no_connect (at 313.69 194.31))
+  (no_connect (at 283.21 207.01))
+  (no_connect (at 162.56 112.395))
+  (no_connect (at 162.56 86.995))
+  (no_connect (at 85.725 271.145))
+  (no_connect (at 85.725 304.165))
+  (no_connect (at 293.37 173.99))
+  (no_connect (at 45.085 296.545))
+  (no_connect (at 45.085 189.865))
+  (no_connect (at 275.59 123.825))
+  (no_connect (at 45.085 197.485))
+  (no_connect (at 85.725 294.005))
+  (no_connect (at 85.725 197.485))
+  (no_connect (at 213.36 109.855))
+  (no_connect (at 85.725 296.545))
+  (no_connect (at 45.085 250.825))
+  (no_connect (at 84.455 105.41))
+  (no_connect (at 162.56 114.935))
+  (no_connect (at 45.085 283.845))
+  (no_connect (at 45.085 225.425))
+  (no_connect (at 85.725 220.345))
+  (no_connect (at 45.085 235.585))
+  (no_connect (at 303.53 173.99))
+  (no_connect (at 45.085 281.305))
+  (no_connect (at 213.36 102.235))
+  (no_connect (at 162.56 137.795))
+  (no_connect (at 85.725 210.185))
+  (no_connect (at 45.085 202.565))
+  (no_connect (at 298.45 173.99))
+  (no_connect (at 213.36 84.455))
+  (no_connect (at 295.91 121.285))
+  (no_connect (at 85.725 212.725))
+  (no_connect (at 67.31 111.125))
+  (no_connect (at 85.725 260.985))
+  (no_connect (at 213.36 71.755))
+  (no_connect (at 85.725 189.865))
+  (no_connect (at 45.085 220.345))
+  (no_connect (at 283.21 199.39))
+  (no_connect (at 283.21 201.93))
+  (no_connect (at 85.725 192.405))
+  (no_connect (at 85.725 187.325))
+  (no_connect (at 290.83 173.99))
+  (no_connect (at 313.69 191.77))
+  (no_connect (at 45.085 273.685))
+  (no_connect (at 213.36 112.395))
+  (no_connect (at 300.99 173.99))
+  (no_connect (at 45.085 299.085))
+  (no_connect (at 213.36 140.335))
+  (no_connect (at 45.085 233.045))
+  (no_connect (at 85.725 276.225))
+  (no_connect (at 213.36 135.255))
+  (no_connect (at 85.725 255.905))
+  (no_connect (at 283.21 204.47))
+  (no_connect (at 85.725 283.845))
+  (no_connect (at 162.56 84.455))
+  (no_connect (at 295.91 123.825))
+  (no_connect (at 162.56 89.535))
+  (no_connect (at 300.99 224.79))
+  (no_connect (at 213.36 92.075))
+  (no_connect (at 162.56 79.375))
+  (no_connect (at 213.36 94.615))
+  (no_connect (at 45.085 215.265))
+  (no_connect (at 45.085 276.225))
+  (no_connect (at 85.725 306.705))
+  (no_connect (at 45.085 294.005))
+  (no_connect (at 295.91 173.99))
+  (no_connect (at 85.725 238.125))
+  (no_connect (at 85.725 266.065))
+  (no_connect (at 313.69 199.39))
+  (no_connect (at 45.085 210.185))
+  (no_connect (at 162.56 76.835))
+  (no_connect (at 162.56 107.315))
+  (no_connect (at 85.725 222.885))
+  (no_connect (at 45.085 288.925))
+  (no_connect (at 45.085 248.285))
+  (no_connect (at 45.085 271.145))
+  (no_connect (at 213.36 86.995))
+  (no_connect (at 313.69 201.93))
+  (no_connect (at 45.085 227.965))
+  (no_connect (at 85.725 235.585))
+  (no_connect (at 85.725 215.265))
+  (no_connect (at 313.69 196.85))
+  (no_connect (at 275.59 121.285))
+  (no_connect (at 85.725 233.045))
+  (no_connect (at 213.36 130.175))
+  (no_connect (at 45.085 207.645))
+  (no_connect (at 85.725 230.505))
+  (no_connect (at 162.56 71.755))
+  (no_connect (at 45.085 260.985))
+  (no_connect (at 213.36 117.475))
+  (no_connect (at 213.36 104.775))
+  (no_connect (at 85.725 273.685))
+  (no_connect (at 45.085 205.105))
+  (no_connect (at 45.085 255.905))
+  (no_connect (at 45.085 222.885))
+  (no_connect (at 85.725 207.645))
+  (no_connect (at 213.36 125.095))
+  (no_connect (at 85.725 301.625))
+  (no_connect (at 85.725 291.465))
+  (no_connect (at 45.085 258.445))
+  (no_connect (at 162.56 135.255))
+  (no_connect (at 162.56 92.075))
+  (no_connect (at 303.53 224.79))
+  (no_connect (at 85.725 253.365))
+  (no_connect (at 162.56 104.775))
+  (no_connect (at 45.085 278.765))
+  (no_connect (at 213.36 137.795))
+  (no_connect (at 45.085 238.125))
+  (no_connect (at 290.83 224.79))
+  (no_connect (at 213.36 122.555))
+  (no_connect (at 85.725 225.425))
+  (no_connect (at 45.085 200.025))
+  (no_connect (at 213.36 99.695))
+  (no_connect (at 283.21 196.85))
+  (no_connect (at 85.725 258.445))
+  (no_connect (at 85.725 278.765))
+  (no_connect (at 298.45 224.79))
+  (no_connect (at 45.085 301.625))
+  (no_connect (at 85.725 227.965))
+  (no_connect (at 213.36 127.635))
+  (no_connect (at 85.725 299.085))
+  (no_connect (at 85.725 268.605))
   (wire (pts (xy 33.655 184.785) (xy 45.085 184.785))
     (stroke (width 0) (type default))
@@
     )
   )
-  (global_label "SS" (shape input) (at 85.725 197.485 0) (fields_autoplaced)
-    (effects (font (size 1.27 1.27)) (justify left))
-    (property "Intersheetrefs" "${INTERSHEET_REFS}" (at 90.5571 197.4056 0)
-      (effects (font (size 1.27 1.27)) (justify left) hide)
-    )
-  )
   (global_label "RF_ANT" (shape input) (at 216.535 79.375 0) (fields_autoplaced)
     (effects (font (size 1.27 1.27)) (justify left))
@@
       (effects (font (size 1.27 1.27)))
     )
-    (property "Value" "SIM8066-6-1-14-01-A" (at 99.695 90.805 0)
+    (property "Value" "XKNANO-113" (at 99.695 90.805 0)
       (effects (font (size 1.27 1.27)))
     )

Commit message: Ændring
Parts:
- added D10: GS1M-LTP, Diode_SMD:D_SMA, symbol Diode:US1G
Connections:
- net VCC_3.6 renamed +3.3V
- net +3.3V: now also D10.1 (K); no longer D6.1 (K)
- new net: D10.2 (A), D6.1 (K)
Other:
- moved on the sheet: D6
Changed lines of the file:
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@@
     (stroke (width 0) (type default))
   )
-  (wire (pts (xy 218.44 176.53) (xy 226.695 176.53))
+  (wire (pts (xy 212.725 176.53) (xy 217.17 176.53))
     (stroke (width 0) (type default))
   )
@@
     (stroke (width 0) (type default))
   )
-  (wire (pts (xy 201.93 176.53) (xy 210.82 176.53))
+  (wire (pts (xy 201.93 176.53) (xy 205.105 176.53))
     (stroke (width 0) (type default))
   )
@@
     (stroke (width 0) (type default))
   )
+  (wire (pts (xy 224.79 176.53) (xy 226.695 176.53))
+    (stroke (width 0) (type default))
+  )
   (wire (pts (xy 173.99 209.55) (xy 176.53 209.55))
     (stroke (width 0) (type default))
@@
     )
   )
+  (symbol (lib_id "Diode:US1G") (at 220.98 176.53 180) (unit 1)
+    (in_bom yes) (on_board yes) (dnp no) (fields_autoplaced)
+    (property "Reference" "D10" (at 220.98 171.45 0)
+      (effects (font (size 1.27 1.27)))
+    )
+    (property "Value" "GS1M-LTP" (at 220.98 173.99 0)
+      (effects (font (size 1.27 1.27)))
+    )
+    (property "Footprint" "Diode_SMD:D_SMA" (at 220.98 172.085 0)
+      (effects (font (size 1.27 1.27)) hide)
+    )
+    (property "Datasheet" "https://www.mouser.dk/datasheet/2/258/GS1A_L_7eGS1M_L_DO_214AC_-2634344.pdf" (at 220.98 176.53 0)
+      (effects (font (size 1.27 1.27)) hide)
+    )
+    (property "Sim.Device" "D" (at 220.98 176.53 0)
+      (effects (font (size 1.27 1.27)) hide)
+    )
+    (property "Sim.Pins" "1=K 2=A" (at 220.98 176.53 0)
+      (effects (font (size 1.27 1.27)) hide)
+    )
+    (property "Manufacturer_Name" "Micro Commercial Components (MCC)" (at 220.98 176.53 0)
+      (effects (font (size 1.27 1.27)) hide)
+    )
+    (property "Manufacturer_Part_Number" "GS1M-LTP" (at 220.98 176.53 0)
+      (effects (font (size 1.27 1.27)) hide)
+    )
+    (property "Mouser Price/Stock" "0,15" (at 220.98 176.53 0)
+      (effects (font (size 1.27 1.27)) hide)
+    )
+    (property "Description" "" (at 220.98 176.53 0)
+      (effects (font (size 1.27 1.27)) hide)
+    )
+    (property "JLCPART#" "C435833" (at 220.98 176.53 0)
+      (effects (font (size 1.27 1.27)) hide)
+    )
+    (pin "1")
+    (pin "2")
+    (instances
+      (project "Modbus_master"
+        (path "/7751fb88-c92a-4fc4-933d-a75f17492f83"
+          (reference "D10") (unit 1)
+        )
+      )
+    )
+  )
   (symbol (lib_id "power:GND") (at 162.56 184.15 0) (unit 1)
     (in_bom yes) (on_board yes) (dnp no)
@@
     )
   )
+  (symbol (lib_id "power:+3.3V") (at 226.695 176.53 270) (unit 1)
+    (in_bom yes) (on_board yes) (dnp no) (fields_autoplaced)
+    (property "Reference" "#PWR039" (at 222.885 176.53 0)
+      (effects (font (size 1.27 1.27)) hide)
+    )
+    (property "Value" "+3.3V" (at 230.505 176.53 90)
+      (effects (font (size 1.27 1.27)) (justify left))
+    )
+    (property "Footprint" "" (at 226.695 176.53 0)
+      (effects (font (size 1.27 1.27)) hide)
+    )
+    (property "Datasheet" "" (at 226.695 176.53 0)
+      (effects (font (size 1.27 1.27)) hide)
+    )
+    (pin "1")
+    (instances
+      (project "Modbus_master"
+        (path "/7751fb88-c92a-4fc4-933d-a75f17492f83"
+          (reference "#PWR039") (unit 1)
+        )
+      )
+    )
+  )
   (symbol (lib_id "power:GND") (at 156.21 313.69 0) (unit 1)
     (in_bom yes) (on_board yes) (dnp no) (fields_autoplaced)
@@
     )
   )
-  (symbol (lib_id "power:VCC") (at 226.695 176.53 270) (unit 1)
-    (in_bom yes) (on_board yes) (dnp no) (fields_autoplaced)
-    (property "Reference" "#PWR039" (at 225.425 184.15 0)
-      (effects (font (size 1.27 1.27)) hide)
-    )
-    (property "Value" "+3.6V" (at 224.155 172.72 90)
-      (effects (font (size 1.27 1.27)) (justify left))
-    )
-    (property "Footprint" "" (at 226.695 176.53 0)
-      (effects (font (size 1.27 1.27)) hide)
-    )
-    (property "Datasheet" "" (at 226.695 176.53 0)
-      (effects (font (size 1.27 1.27)) hide)
-    )
-    (pin "3")
-    (instances
-      (project "Modbus_master"
-        (path "/7751fb88-c92a-4fc4-933d-a75f17492f83"
-          (reference "#PWR039") (unit 1)
-        )
-      )
-    )
-  )
   (symbol (lib_id "power:GND") (at 198.12 327.025 0) (unit 1)
     (in_bom yes) (on_board yes) (dnp no) (fields_autoplaced)
@@
     )
   )
+  (symbol (lib_id "power:+3.3V") (at 278.765 187.96 0) (unit 1)
+    (in_bom yes) (on_board yes) (dnp no) (fields_autoplaced)
+    (property "Reference" "#PWR042" (at 278.765 191.77 0)
+      (effects (font (size 1.27 1.27)) hide)
+    )
+    (property "Value" "+3.3V" (at 278.765 183.515 0)
+      (effects (font (size 1.27 1.27)))
+    )
+    (property "Footprint" "" (at 278.765 187.96 0)
+      (effects (font (size 1.27 1.27)) hide)
+    )
+    (property "Datasheet" "" (at 278.765 187.96 0)
+      (effects (font (size 1.27 1.27)) hide)
+    )
+    (pin "1")
+    (instances
+      (project "Modbus_master"
+        (path "/7751fb88-c92a-4fc4-933d-a75f17492f83"
+          (reference "#PWR042") (unit 1)
+        )
+      )
+    )
+  )
   (symbol (lib_id "Device:L") (at 133.35 308.61 90) (unit 1)
     (in_bom yes) (on_board yes) (dnp no) (fields_autoplaced)
@@
     )
   )
-  (symbol (lib_id "power:VCC") (at 278.765 187.96 0) (unit 1)
-    (in_bom yes) (on_board yes) (dnp no) (fields_autoplaced)
-    (property "Reference" "#PWR046" (at 286.385 189.23 0)
-      (effects (font (size 1.27 1.27)) hide)
-    )
-    (property "Value" "+3.6V" (at 278.765 182.88 0)
-      (effects (font (size 1.27 1.27)))
-    )
-    (property "Footprint" "" (at 278.765 187.96 0)
-      (effects (font (size 1.27 1.27)) hide)
-    )
-    (property "Datasheet" "" (at 278.765 187.96 0)
-      (effects (font (size 1.27 1.27)) hide)
-    )
-    (pin "3")
-    (instances
-      (project "Modbus_master"
-        (path "/7751fb88-c92a-4fc4-933d-a75f17492f83"
-          (reference "#PWR046") (unit 1)
-        )
-      )
-    )
-  )
   (symbol (lib_name "VCC_2") (lib_id "power:VCC") (at 172.72 224.79 0) (unit 1)
     (in_bom yes) (on_board yes) (dnp no) (fields_autoplaced)
@@
     )
   )
-  (symbol (lib_id "power:VCC") (at 260.35 54.61 0) (unit 1)
-    (in_bom yes) (on_board yes) (dnp no) (fields_autoplaced)
-    (property "Reference" "#PWR042" (at 267.97 55.88 0)
-      (effects (font (size 1.27 1.27)) hide)
-    )
-    (property "Value" "+3.6V" (at 260.35 51.435 0)
-      (effects (font (size 1.27 1.27)))
-    )
-    (property "Footprint" "" (at 260.35 54.61 0)
-      (effects (font (size 1.27 1.27)) hide)
-    )
-    (property "Datasheet" "" (at 260.35 54.61 0)
-      (effects (font (size 1.27 1.27)) hide)
-    )
-    (pin "3")
-    (instances
-      (project "Modbus_master"
-        (path "/7751fb88-c92a-4fc4-933d-a75f17492f83"
-          (reference "#PWR042") (unit 1)
-        )
-      )
-    )
-  )
-  (symbol (lib_id "Diode:US1G") (at 214.63 176.53 180) (unit 1)
+  (symbol (lib_id "Diode:US1G") (at 208.915 176.53 180) (unit 1)
     (in_bom yes) (on_board yes) (dnp no) (fields_autoplaced)
-    (property "Reference" "D6" (at 214.63 171.45 0)
+    (property "Reference" "D6" (at 208.915 171.45 0)
       (effects (font (size 1.27 1.27)))
     )
-    (property "Value" "GS1M-LTP" (at 214.63 173.99 0)
+    (property "Value" "GS1M-LTP" (at 208.915 173.99 0)
       (effects (font (size 1.27 1.27)))
     )
-    (property "Footprint" "Diode_SMD:D_SMA" (at 214.63 172.085 0)
+    (property "Footprint" "Diode_SMD:D_SMA" (at 208.915 172.085 0)
       (effects (font (size 1.27 1.27)) hide)
     )
-    (property "Datasheet" "https://www.mouser.dk/datasheet/2/258/GS1A_L_7eGS1M_L_DO_214AC_-2634344.pdf" (at 214.63 176.53 0)
+    (property "Datasheet" "https://www.mouser.dk/datasheet/2/258/GS1A_L_7eGS1M_L_DO_214AC_-2634344.pdf" (at 208.915 176.53 0)
       (effects (font (size 1.27 1.27)) hide)
     )
-    (property "Sim.Device" "D" (at 214.63 176.53 0)
+    (property "Sim.Device" "D" (at 208.915 176.53 0)
       (effects (font (size 1.27 1.27)) hide)
     )
-    (property "Sim.Pins" "1=K 2=A" (at 214.63 176.53 0)
+    (property "Sim.Pins" "1=K 2=A" (at 208.915 176.53 0)
       (effects (font (size 1.27 1.27)) hide)
     )
-    (property "Manufacturer_Name" "Micro Commercial Components (MCC)" (at 214.63 176.53 0)
+    (property "Manufacturer_Name" "Micro Commercial Components (MCC)" (at 208.915 176.53 0)
       (effects (font (size 1.27 1.27)) hide)
     )
-    (property "Manufacturer_Part_Number" "GS1M-LTP" (at 214.63 176.53 0)
+    (property "Manufacturer_Part_Number" "GS1M-LTP" (at 208.915 176.53 0)
       (effects (font (size 1.27 1.27)) hide)
     )
-    (property "Mouser Price/Stock" "0,15" (at 214.63 176.53 0)
+    (property "Mouser Price/Stock" "0,15" (at 208.915 176.53 0)
       (effects (font (size 1.27 1.27)) hide)
     )
-    (property "Description" "" (at 214.63 176.53 0)
+    (property "Description" "" (at 208.915 176.53 0)
       (effects (font (size 1.27 1.27)) hide)
     )
-    (property "JLCPART#" "C435833" (at 214.63 176.53 0)
+    (property "JLCPART#" "C435833" (at 208.915 176.53 0)
       (effects (font (size 1.27 1.27)) hide)
     )
@@
         )
       )
+    )
+  )
+  (symbol (lib_id "power:+3.3V") (at 260.35 54.61 0) (unit 1)
+    (in_bom yes) (on_board yes) (dnp no) (fields_autoplaced)
+    (property "Reference" "#PWR054" (at 260.35 58.42 0)
+      (effects (font (size 1.27 1.27)) hide)
+    )
+    (property "Value" "+3.3V" (at 260.35 50.165 0)
+      (effects (font (size 1.27 1.27)))
+    )
+    (property "Footprint" "" (at 260.35 54.61 0)
+      (effects (font (size 1.27 1.27)) hide)
+    )
+    (property "Datasheet" "" (at 260.35 54.61 0)
+      (effects (font (size 1.27 1.27)) hide)
+    )
+    (pin "1")
+    (instances
+      (project "Modbus_master"
+        (path "/7751fb88-c92a-4fc4-933d-a75f17492f83"
+          (reference "#PWR054") (unit 1)
+        )
+      )

Commit message: Ændring
Other:
- moved on the sheet: C17, C18, C19, IC1, J4, L1

Commit message: Ændring
Other:
- moved on the sheet: C17, C18, C19, IC1, J4, L1
